File: onigaku.sch (KiCad schematic (older format))
At the start: 225 parts, among them U1 nice_nano

Commit message: wip
Parts:
- removed D0, D? (x71): LTST-A683CEGBW, symbol cherry_mx:LTST-A683CEGBW
- removed D_16, D_31, D_32, D_33, D_59, D_68, D_69, D_70: D, Diode_SMD:D_SOD-123, symbol Device:D_Small
- removed F?: 500mA, symbol Device:Polyfuse_Small
- removed J?: USB_C_Receptacle_USB2.0, symbol Connector:USB_C_Receptacle_USB2.0
- removed K_14, K_15, K_16, K_31, K_32, K_33, K_59, K_68, K_69, K_70: KEYSW, MX_Alps_Hybrid:MX-1U-NoLED, symbol MX_Alps_Hybrid:MX-NoLED
- removed Q?: BS107, Package_TO_SOT_THT:TO-92_Inline, symbol Transistor_FET:BS107
- removed R? (x2): 5.1k, symbol Device:R_Small
- removed U1: nice_nano, symbol nice_nano:nice_nano
- removed U?: pro_micro_pinout, symbol nice_nano:pro_micro_pinout
- removed U?: Cherry_MX_RGB, symbol cherry_mx:Cherry_MX_RGB
- removed U_KEYS, U_LEDS: proton_c, symbol qmk_hardware:proton_c
- added C?: 0.47uF, symbol Device:C
- added C?: 22uF, symbol ktype:C_Small_Pol
- added C? (x3): 0.47uF, symbol ktype:C_Small
- added C? (x3): 0.1uF, symbol ktype:C_Small
- added J1_L1: MJ-4PP-9, kbd:MJ-4PP-9_1side, symbol foostan_kbd:MJ-4PP-9
- added J2_L1, J4: OLED, kbd:OLED_1side, symbol Connector_Generic:Conn_01x04
- added J3: MJ-4PP-9, kbd:MJ-4PP-9, symbol kbd:MJ-4PP-9
- added LED0, LED1, LED10, LED11, LED12, LED13, LED2, LED20, LED21, LED22, LED23, LED24, LED25, LED26, LED27, LED28, LED29, LED3, LED30, LED31, LED32, LED33, LED34, LED35, LED36, LED37, LED38, LED39, LED4, LED40, LED41, LED42, LED43, LED44, LED45, LED46, LED48, LED49, LED5, LED50, LED51, LED52, LED53, LED54, LED55, LED56, LED57, LED58, LED59, LED6, LED60, LED61, LED62, LED63, LED64, LED65, LED66, LED67, LED7, LED73, LED74, LED75, LED8, LED9: YS-SK6812MINI-E, kbd:YS-SK6812MINI-E, symbol foostan_kbd:YS-SK6812MINI-E
- added LED14, LED15, LED16, LED17, LED18, LED19, LED47, LED68, LED69, LED70, LED71, LED72: WS2812B, kbd:LED_WS2812B-PLCC4, symbol LED:WS2812B
- added R2: 500ohm, symbol Device:R
- added R?: 13k, symbol ktype:R_Small
- added R? (x2): 1k, symbol ktype:R_Small
- added R? (x2): 100k, symbol ktype:R_Small
- added RSW1, RSW2: SW_PUSH, kbd:ResetSW_1side, symbol kbd:SW_PUSH
- added SW_57: KEYSW, kbd:CherryMX_Hotswap_2.75u_North, symbol MX_Alps_Hybrid:MX-NoLED
- added SW_62: KEYSW, kbd:CherryMX_Hotswap_1.25u_North, symbol MX_Alps_Hybrid:MX-NoLED
- added U1: ProMicro, kbd:ProMicro_v3, symbol foostan_kbd:ProMicro
- added U2: ProMicro, kbd:ProMicro_v3, symbol kbd:ProMicro
- added U?: IS31FL3733, symbol ktype:IS31FL3733
- D_0, D_1, D_10, D_11, D_12, D_13, D_14, D_15, D_17, D_18, D_19, D_2, D_20, D_21, D_22, D_23, D_24, D_25, D_26, D_27, D_28, D_29, D_3, D_30, D_34, D_35, D_36, D_37, D_38, D_39, D_4, D_40, D_41, D_42, D_43, D_44, D_45, D_46, D_47, D_48, D_49, D_5, D_50, D_51, D_52, D_53, D_54, D_55, D_56, D_57, D_58, D_6, D_60, D_61, D_62, D_63, D_64, D_65, D_66, D_67, D_7, D_8, D_9: footprint Diode_SMD:D_SOD-123 -> kbd:D3_SMD_v2
- R1: value 100 Ohm -> 500ohm
- SW_0: renamed from K_0; footprint MX_Alps_Hybrid:MX-1U-NoLED -> kbd:CherryMX_Hotswap
- SW_1: renamed from K_1; footprint MX_Alps_Hybrid:MX-1U-NoLED -> kbd:CherryMX_Hotswap
- SW_10: renamed from K_20; footprint MX_Alps_Hybrid:MX-1U-NoLED -> kbd:CherryMX_Hotswap
- SW_11: renamed from K_21; footprint MX_Alps_Hybrid:MX-1U-NoLED -> kbd:CherryMX_Hotswap
- SW_12: renamed from K_22; footprint MX_Alps_Hybrid:MX-1U-NoLED -> kbd:CherryMX_Hotswap
- SW_13: renamed from K_34; footprint MX_Alps_Hybrid:MX-1.75U-NoLED -> kbd:CherryMX_Hotswap_1.75u
- SW_14: renamed from K_35; footprint MX_Alps_Hybrid:MX-1U-NoLED -> kbd:CherryMX_Hotswap
- SW_15: renamed from K_36; footprint MX_Alps_Hybrid:MX-1U-NoLED -> kbd:CherryMX_Hotswap
- SW_16: renamed from K_37; footprint MX_Alps_Hybrid:MX-1U-NoLED -> kbd:CherryMX_Hotswap
- SW_17: renamed from K_38; footprint MX_Alps_Hybrid:MX-1U-NoLED -> kbd:CherryMX_Hotswap
- SW_18: renamed from K_39; footprint MX_Alps_Hybrid:MX-1U-NoLED -> kbd:CherryMX_Hotswap
- SW_19: renamed from K_47; footprint MX_Alps_Hybrid:MX-2.25U-NoLED -> kbd:CherryMX_Hotswap_2.25u_North
- SW_2: renamed from K_2; footprint MX_Alps_Hybrid:MX-1U-NoLED -> kbd:CherryMX_Hotswap
- SW_20: renamed from K_48; footprint MX_Alps_Hybrid:MX-1U-NoLED -> kbd:CherryMX_Hotswap
- SW_21: renamed from K_49; footprint MX_Alps_Hybrid:MX-1U-NoLED -> kbd:CherryMX_Hotswap
- SW_22: renamed from K_50; footprint MX_Alps_Hybrid:MX-1U-NoLED -> kbd:CherryMX_Hotswap
- SW_23: renamed from K_51; footprint MX_Alps_Hybrid:MX-1U-NoLED -> kbd:CherryMX_Hotswap
- SW_24: renamed from K_52; footprint MX_Alps_Hybrid:MX-1U-NoLED -> kbd:CherryMX_Hotswap
- SW_25: renamed from K_60; footprint MX_Alps_Hybrid:MX-1.25U-NoLED -> kbd:CherryMX_Hotswap_1.25u_North
- SW_26: renamed from K_61; footprint MX_Alps_Hybrid:MX-1.25U-NoLED -> kbd:CherryMX_Hotswap_1.25u_North
- SW_27: renamed from K_62; footprint MX_Alps_Hybrid:MX-1.25U-NoLED -> kbd:CherryMX_Hotswap_1.25u_North
- SW_28: renamed from K_63; footprint MX_Alps_Hybrid:MX-6.25U-NoLED -> kbd:CherryMX_Hotswap_2.25u_North
- SW_29: renamed from K_7; footprint MX_Alps_Hybrid:MX-1U-NoLED -> kbd:CherryMX_Hotswap
- SW_3: renamed from K_3; footprint MX_Alps_Hybrid:MX-1U-NoLED -> kbd:CherryMX_Hotswap
- SW_30: renamed from K_8; footprint MX_Alps_Hybrid:MX-1U-NoLED -> kbd:CherryMX_Hotswap
- SW_31: renamed from K_9; footprint MX_Alps_Hybrid:MX-1U-NoLED -> kbd:CherryMX_Hotswap
- SW_32: renamed from K_10; footprint MX_Alps_Hybrid:MX-1U-NoLED -> kbd:CherryMX_Hotswap
- SW_33: renamed from K_11; footprint MX_Alps_Hybrid:MX-1U-NoLED -> kbd:CherryMX_Hotswap
- SW_34: renamed from K_12; footprint MX_Alps_Hybrid:MX-1U-NoLED -> kbd:CherryMX_Hotswap
- SW_35: renamed from K_13; footprint MX_Alps_Hybrid:MX-2U-NoLED -> kbd:CherryMX_Hotswap
- SW_36: renamed from K_23; footprint MX_Alps_Hybrid:MX-1U-NoLED -> kbd:CherryMX_Hotswap
- SW_37: renamed from K_24; footprint MX_Alps_Hybrid:MX-1U-NoLED -> kbd:CherryMX_Hotswap
- SW_38: renamed from K_25; footprint MX_Alps_Hybrid:MX-1U-NoLED -> kbd:CherryMX_Hotswap
- SW_39: renamed from K_26; footprint MX_Alps_Hybrid:MX-1U-NoLED -> kbd:CherryMX_Hotswap
- SW_4: renamed from K_4; footprint MX_Alps_Hybrid:MX-1U-NoLED -> kbd:CherryMX_Hotswap
- SW_40: renamed from K_27; footprint MX_Alps_Hybrid:MX-1U-NoLED -> kbd:CherryMX_Hotswap
- SW_41: renamed from K_28; footprint MX_Alps_Hybrid:MX-1U-NoLED -> kbd:CherryMX_Hotswap
- SW_42: renamed from K_29; footprint MX_Alps_Hybrid:MX-1U-NoLED -> kbd:CherryMX_Hotswap
- SW_43: renamed from K_30; footprint MX_Alps_Hybrid:MX-1.5U-NoLED -> kbd:CherryMX_Hotswap_1.5u
- SW_44: renamed from K_40; footprint MX_Alps_Hybrid:MX-1U-NoLED -> kbd:CherryMX_Hotswap
- SW_45: renamed from K_41; footprint MX_Alps_Hybrid:MX-1U-NoLED -> kbd:CherryMX_Hotswap
- SW_46: renamed from K_42; footprint MX_Alps_Hybrid:MX-1U-NoLED -> kbd:CherryMX_Hotswap
- SW_47: renamed from K_43; footprint MX_Alps_Hybrid:MX-1U-NoLED -> kbd:CherryMX_Hotswap
- SW_48: renamed from K_44; footprint MX_Alps_Hybrid:MX-1U-NoLED -> kbd:CherryMX_Hotswap
- SW_49: renamed from K_45; footprint MX_Alps_Hybrid:MX-1U-NoLED -> kbd:CherryMX_Hotswap
- SW_5: renamed from K_5; footprint MX_Alps_Hybrid:MX-1U-NoLED -> kbd:CherryMX_Hotswap
- SW_50: renamed from K_46; footprint MX_Alps_Hybrid:MX-2.25U-NoLED -> kbd:CherryMX_Hotswap_2.25u_North
- SW_51: renamed from K_53; footprint MX_Alps_Hybrid:MX-1U-NoLED -> kbd:CherryMX_Hotswap
- SW_52: renamed from K_54; footprint MX_Alps_Hybrid:MX-1U-NoLED -> kbd:CherryMX_Hotswap
- SW_53: renamed from K_55; footprint MX_Alps_Hybrid:MX-1U-NoLED -> kbd:CherryMX_Hotswap
- SW_54: renamed from K_56; footprint MX_Alps_Hybrid:MX-1U-NoLED -> kbd:CherryMX_Hotswap
- SW_55: renamed from K_57; footprint MX_Alps_Hybrid:MX-1U-NoLED -> kbd:CherryMX_Hotswap
- SW_56: renamed from K_58; footprint MX_Alps_Hybrid:MX-2.75U-NoLED -> kbd:CherryMX_Hotswap_2.75u_North
- SW_58: renamed from K_64; footprint MX_Alps_Hybrid:MX-1.25U-NoLED -> kbd:CherryMX_Hotswap_1.25u_North
- SW_59: renamed from K_65; footprint MX_Alps_Hybrid:MX-1.25U-NoLED -> kbd:CherryMX_Hotswap_1.25u_North
- SW_6: renamed from K_6; footprint MX_Alps_Hybrid:MX-1U-NoLED -> kbd:CherryMX_Hotswap
- SW_60: renamed from K_66; footprint MX_Alps_Hybrid:MX-1.25U-NoLED -> kbd:CherryMX_Hotswap_1.25u_North
- SW_61: renamed from K_67; footprint MX_Alps_Hybrid:MX-1.25U-NoLED -> kbd:CherryMX_Hotswap_1.25u_North
- SW_7: renamed from K_17; footprint MX_Alps_Hybrid:MX-1.5U-NoLED -> kbd:CherryMX_Hotswap_1.5u
- SW_8: renamed from K_18; footprint MX_Alps_Hybrid:MX-1U-NoLED -> kbd:CherryMX_Hotswap
- SW_9: renamed from K_19; footprint MX_Alps_Hybrid:MX-1U-NoLED -> kbd:CherryMX_Hotswap
Connections:
- net labels added: GNDA, INTB, LED_L, LED_R, SCL_L, SCL_R, SDA_L, SDA_R, SDB, VDD, VSS, col0_L, col0_R, col1_L, col1_R, col2_L, col2_R, col3_L, col3_R, col4_L, col4_R, col5_L, col5_R, col6_L, col6_R, col7_R, data_L, data_R, reset_L, reset_R, row0_L, row0_R, row1_L, row1_R, row2_L, row2_R, row3_L, row3_R, row4_L, row4_R
- net labels removed: +5V, D+, D-, PWM, col0, col1, col10, col11, col12, col13, col14, col15, col16, col17, col2, col3, col4, col5, col6, col7, col8, col9, row0, row1, row2, row3, row4
- wire segments 490 -> 676
- no-connect marks 0 -> 8
Other:
- moved on the sheet: D_0, D_1, D_10, D_11, D_12, D_13, D_17, D_18, D_19, D_2, D_20, D_21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

Commit message: wip
Parts:
- removed C?: 0.47uF, symbol Device:C
- removed C?: 22uF, symbol ktype:C_Small_Pol
- removed C? (x3): 0.47uF, symbol ktype:C_Small
- removed C? (x3): 0.1uF, symbol ktype:C_Small
- removed J2_L1, J4: OLED, kbd:OLED_1side, symbol Connector_Generic:Conn_01x04
- removed J3: MJ-4PP-9, kbd:MJ-4PP-9, symbol kbd:MJ-4PP-9
- removed LED0, LED1, LED10, LED11, LED12, LED13, LED2, LED20, LED21, LED22, LED23, LED24, LED25, LED26, LED27, LED28, LED29, LED3, LED30, LED31, LED32, LED33, LED34, LED35, LED36, LED37, LED38, LED39, LED4, LED40, LED41, LED42, LED43, LED44, LED45, LED46, LED48, LED49, LED5, LED50, LED51, LED52, LED53, LED54, LED55, LED56, LED57, LED58, LED59, LED6, LED60, LED61, LED62, LED63, LED64, LED65, LED66, LED67, LED7, LED73, LED74, LED75, LED8, LED9: YS-SK6812MINI-E, kbd:YS-SK6812MINI-E, symbol foostan_kbd:YS-SK6812MINI-E
- removed LED14, LED15, LED16, LED17, LED18, LED19, LED47, LED68, LED69, LED70, LED71, LED72: WS2812B, kbd:LED_WS2812B-PLCC4, symbol LED:WS2812B
- removed R1, R2: 500ohm, symbol Device:R
- removed R?: 13k, symbol ktype:R_Small
- removed R? (x2): 1k, symbol ktype:R_Small
- removed R? (x2): 100k, symbol ktype:R_Small
- removed U?: IS31FL3733, symbol ktype:IS31FL3733
- added C? (x2): 22uF, lib.pretty:SMD-7343-Pol, symbol K-Type:C_Small_Pol
- added C? (x6): 0.1uF, lib.pretty:SMD-0402, symbol K-Type:C_Small
- added C? (x8): 0.47uF, lib.pretty:SMD-0402, symbol K-Type:C_Small
- added D? (x57): LED_GRBA, symbol Device:LED_GRBA
- added J1_L?: MJ-4PP-9, kbd:MJ-4PP-9_1side, symbol foostan_kbd:MJ-4PP-9
- added MH1, MH2, MH3, MH4, MH5, MH6, MH7, MH8: 1PIN, lib.pretty:1PAD, symbol K-Type:1PIN
- added R? (x2): 20k, lib.pretty:SMD-0402, symbol K-Type:R_Small
- added R? (x2): 100k, lib.pretty:SMD-0402, symbol K-Type:R_Small
- added R? (x4): 1k, lib.pretty:SMD-0402, symbol K-Type:R_Small
- added R? (x4): 10k, symbol Device:R_Small
- added U3, U4: IS31FL3733, lib.pretty:QFN-48-6mm-vias, symbol K-Type:IS31FL3733
Connections:
- net labels added: +5V, Col1, Col10, Col2, Col3, Col4, Col5, Col6, Col7, Col8, Col9, LD1_CS1, LD1_CS10, LD1_CS11, LD1_CS12, LD1_CS13, LD1_CS14, LD1_CS15, LD1_CS16, LD1_CS2, LD1_CS3, LD1_CS4, LD1_CS5, LD1_CS6, LD1_CS7, LD1_CS8, LD1_CS9, LD1_SW1, LD1_SW10, LD1_SW11, LD1_SW12, LD1_SW2, LD1_SW3, LD1_SW4, LD1_SW5, LD1_SW6, LD1_SW7, LD1_SW8, LD1_SW9, LD2_CS1, LD2_CS10, LD2_CS11, LD2_CS12, LD2_CS13, LD2_CS14, LD2_CS15, LD2_CS16, LD2_CS2, LD2_CS3, LD2_CS4, LD2_CS5, LD2_CS6, LD2_CS7, LD2_CS8, LD2_CS9, Row1, Row10, Row2, Row3, Row4, Row5, Row6, Row7, Row8, Row9, SYNC
- net labels removed: GNDA, INTB, LED_L, LED_R, SDB, VSS, data_L
- wire segments 676 -> 1322
- no-connect marks 8 -> 7
Other:
- note added: "Ctrl, Win, Fnc, Alt, Spacebar"
- note added: "Note: We remap the pins of the LED a bit for simplicity reasons:\n\nDatasheet: 1=G, 2=R, 3=B, 4=CA\n\nRemap in the footprint: 1=CA, 2=R, 3=G, 4=B"
- note added: "SLAVE @ 0xA1 (See IS31FL3733 datasheet)"
- moved on the sheet: D_0, D_1, D_10, D_11, D_12, D_13, D_14, D_15, D_17, D_18, D_19, D_2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

Commit message: sorted out matrix, upgraded to elite-c, and added underglow leds
Parts:
- removed MH1, MH2, MH3, MH4, MH5, MH6, MH7, MH8: 1PIN, lib.pretty:1PAD, symbol K-Type:1PIN
- removed U1: ProMicro, kbd:ProMicro_v3, symbol foostan_kbd:ProMicro
- removed U2: ProMicro, kbd:ProMicro_v3, symbol kbd:ProMicro
- added D? (x12): WS2812B, LED_SMD:LED_WS2812B_PLCC4_5.0x5.0mm_P3.2mm, symbol LED:WS2812B
- added U1, U2: elite-c, symbol nice_nano:elite-c
- R? (x4): value 1k -> 4.7k
- gave numbers to parts that had none: 1
Connections:
- net labels added: BACKLIGHT_LED_L, BACKLIGHT_LED_R, L_CS1, L_CS10, L_CS11, L_CS12, L_CS13, L_CS14, L_CS15, L_CS16, L_CS2, L_CS3, L_CS4, L_CS5, L_CS6, L_CS7, L_CS8, L_CS9, L_SW07, L_SW08, L_SW09, L_SW10, L_SW11, L_SW12, R_CS1, R_CS10, R_CS11, R_CS12, R_CS13, R_CS14, R_CS15, R_CS16, R_CS2, R_CS3, R_CS4, R_CS5, R_CS6, R_CS7, R_CS8, R_CS9, R_SW07, R_SW08, R_SW09, R_SW10, R_SW11, R_SW12
- net labels removed: Col1, Col10, Col2, Col3, Col4, Col5, Col6, Col7, Col8, Col9, LD1_CS1, LD1_CS10, LD1_CS11, LD1_CS12, LD1_CS13, LD1_CS14, LD1_CS15, LD1_CS16, LD1_CS2, LD1_CS3, LD1_CS4, LD1_CS5, LD1_CS6, LD1_CS7, LD1_CS8, LD1_CS9, LD1_SW1, LD1_SW10, LD1_SW11, LD1_SW12, LD1_SW2, LD1_SW3, LD1_SW4, LD1_SW5, LD1_SW6, LD1_SW7, LD1_SW8, LD1_SW9, LD2_CS1, LD2_CS10, LD2_CS11, LD2_CS12, LD2_CS13, LD2_CS14, LD2_CS15, LD2_CS16, LD2_CS2, LD2_CS3, LD2_CS4, LD2_CS5, LD2_CS6, LD2_CS7, LD2_CS8, LD2_CS9, Row1, Row10, Row2, Row3, Row4, Row5, Row6, Row7, Row8, Row9, VDD, data_R
- wire segments 1322 -> 847
- no-connect marks 7 -> 25
Other:
- note added: "7, 8, 9, 0, -, +, bckspace"
- note added: "Esc, 1, 2, 3, 4, 5, 6"
- note added: "MASTER @ 0xA0"
- note added: "Tab, q, w, e, r, t"
- note added: "cpslck, a, s"
- note added: "d, f, g"
- note added: "h"
- note added: "j, k, l, m, ;, ', enter"
- note added: "shift, z, x, c, v, b"
- note added: "space, alt, fn, win, ctrl"
- note added: "y, u, i, o, p, [, ], \"
- note removed: "Note: We remap the pins of the LED a bit for simplicity reasons:\n\nDatasheet: 1=G, 2=R, 3=B, 4=CA\n\nRemap in the footprint: 1=CA, 2=R, 3=G, 4=B"
- moved on the sheet: C?, D?, D_0, D_1, D_10, D_11, D_12, D_13, D_14, D_15, D_17, D_18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

Commit message: continuing WIP
Parts:
- removed C? (x2): 22uF, lib.pretty:SMD-7343-Pol, symbol K-Type:C_Small_Pol
- removed C? (x6): 0.1uF, lib.pretty:SMD-0402, symbol K-Type:C_Small
- removed C? (x8): 0.47uF, lib.pretty:SMD-0402, symbol K-Type:C_Small
- removed D? (x57): LED_GRBA, symbol Device:LED_GRBA
- removed D? (x12): WS2812B, LED_SMD:LED_WS2812B_PLCC4_5.0x5.0mm_P3.2mm, symbol LED:WS2812B
- removed D_0: D, kbd:D3_SMD_v2, symbol Device:D_Small
- removed J1_L1, J1_L2: MJ-4PP-9, kbd:MJ-4PP-9_1side, symbol foostan_kbd:MJ-4PP-9
- removed R? (x2): 20k, lib.pretty:SMD-0402, symbol K-Type:R_Small
- removed R? (x2): 100k, lib.pretty:SMD-0402, symbol K-Type:R_Small
- removed R? (x4): 4.7k, lib.pretty:SMD-0402, symbol K-Type:R_Small
- removed R? (x4): 10k, symbol Device:R_Small
- removed RSW2: SW_PUSH, kbd:ResetSW_1side, symbol kbd:SW_PUSH
- removed U1, U2: elite-c, symbol nice_nano:elite-c
- removed U3, U4: IS31FL3733, lib.pretty:QFN-48-6mm-vias, symbol K-Type:IS31FL3733
- added D_8: D, kbd:D3_SMD_v2, symbol Device:D_Small
- added J1: MJ-4PP-9, onigaku:MJ-4PP-9_1side, symbol kbd:MJ-4PP-9
- added J2: MJ-4PP-9, onigaku:MJ-4PP-9, symbol kbd:MJ-4PP-9
- added LED1, LED10, LED11, LED12, LED13, LED14, LED15, LED16, LED17, LED18, LED19, LED2, LED20, LED21, LED22, LED23, LED24, LED25, LED26, LED27, LED28, LED29, LED3, LED30, LED31, LED32, LED33, LED34, LED35, LED36, LED37, LED38, LED39, LED4, LED40, LED41, LED42, LED43, LED44, LED45, LED46, LED47, LED48, LED49, LED5, LED50, LED51, LED52, LED53, LED54, LED55, LED56, LED57, LED58, LED59, LED6, LED60, LED61, LED62, LED63, LED64, LED65, LED66, LED67, LED68, LED69, LED7, LED70, LED71, LED72, LED73, LED74, LED75, LED76, LED77, LED78, LED79, LED8, LED9: YS-SK6812MINI-E, onigaku:YS-SK6812MINI-E, symbol kbd:YS-SK6812MINI-E
- added RSW1: SW_PUSH, onigaku:ResetSW, symbol kbd:SW_PUSH
- added U1, U2: elite-c, keebio:Elite-C, symbol onigaku:elite-c
- RSW2: renamed from RSW1; footprint kbd:ResetSW_1side -> onigaku:ResetSW_1side
- SW_1: renamed from SW_29; footprint kbd:CherryMX_Hotswap -> onigaku:CherryMX_Hotswap
- SW_10: renamed from SW_2; footprint kbd:CherryMX_Hotswap -> onigaku:CherryMX_Hotswap
- SW_11: renamed from SW_3; footprint kbd:CherryMX_Hotswap -> onigaku:CherryMX_Hotswap
- SW_12: renamed from SW_4; footprint kbd:CherryMX_Hotswap -> onigaku:CherryMX_Hotswap
- SW_13: renamed from SW_5; footprint kbd:CherryMX_Hotswap -> onigaku:CherryMX_Hotswap
- SW_14: renamed from SW_6; footprint kbd:CherryMX_Hotswap -> onigaku:CherryMX_Hotswap
- SW_15: renamed from SW_36; footprint kbd:CherryMX_Hotswap -> onigaku:CherryMX_Hotswap
- SW_16: renamed from SW_37; footprint kbd:CherryMX_Hotswap -> onigaku:CherryMX_Hotswap
- SW_17: renamed from SW_38; footprint kbd:CherryMX_Hotswap -> onigaku:CherryMX_Hotswap
- SW_18: renamed from SW_39; footprint kbd:CherryMX_Hotswap -> onigaku:CherryMX_Hotswap
- SW_19: renamed from SW_40; footprint kbd:CherryMX_Hotswap -> onigaku:CherryMX_Hotswap
- SW_2: renamed from SW_30; footprint kbd:CherryMX_Hotswap -> onigaku:CherryMX_Hotswap
- SW_20: renamed from SW_41; footprint kbd:CherryMX_Hotswap -> onigaku:CherryMX_Hotswap
- SW_21: renamed from SW_42; footprint kbd:CherryMX_Hotswap -> onigaku:CherryMX_Hotswap
- SW_22: renamed from SW_43; footprint kbd:CherryMX_Hotswap_1.5u -> onigaku:CherryMX_Hotswap
- SW_23: renamed from SW_7; footprint kbd:CherryMX_Hotswap_1.5u -> onigaku:CherryMX_Hotswap
- SW_24: renamed from SW_8; footprint kbd:CherryMX_Hotswap -> onigaku:CherryMX_Hotswap
- SW_25: renamed from SW_9; footprint kbd:CherryMX_Hotswap -> onigaku:CherryMX_Hotswap
- SW_26: renamed from SW_10; footprint kbd:CherryMX_Hotswap -> onigaku:CherryMX_Hotswap
- SW_27: renamed from SW_11; footprint kbd:CherryMX_Hotswap -> onigaku:CherryMX_Hotswap
- SW_28: renamed from SW_12; footprint kbd:CherryMX_Hotswap -> onigaku:CherryMX_Hotswap
- SW_29: renamed from SW_44; footprint kbd:CherryMX_Hotswap -> onigaku:CherryMX_Hotswap
- SW_3: renamed from SW_31; footprint kbd:CherryMX_Hotswap -> onigaku:CherryMX_Hotswap
- SW_30: renamed from SW_45; footprint kbd:CherryMX_Hotswap -> onigaku:CherryMX_Hotswap
- SW_31: renamed from SW_46; footprint kbd:CherryMX_Hotswap -> onigaku:CherryMX_Hotswap
- SW_32: renamed from SW_47; footprint kbd:CherryMX_Hotswap -> onigaku:CherryMX_Hotswap
- SW_33: renamed from SW_48; footprint kbd:CherryMX_Hotswap -> onigaku:CherryMX_Hotswap
- SW_34: renamed from SW_49; footprint kbd:CherryMX_Hotswap -> onigaku:CherryMX_Hotswap
- SW_35: renamed from SW_50; footprint kbd:CherryMX_Hotswap_2.25u_North -> onigaku:CherryMX_Hotswap
- SW_36: renamed from SW_13; footprint kbd:CherryMX_Hotswap_1.75u -> onigaku:CherryMX_Hotswap
- SW_37: renamed from SW_14; footprint kbd:CherryMX_Hotswap -> onigaku:CherryMX_Hotswap
- SW_38: renamed from SW_15; footprint kbd:CherryMX_Hotswap -> onigaku:CherryMX_Hotswap
- SW_39: renamed from SW_16; footprint kbd:CherryMX_Hotswap -> onigaku:CherryMX_Hotswap
- SW_4: renamed from SW_32; footprint kbd:CherryMX_Hotswap -> onigaku:CherryMX_Hotswap
- SW_40: renamed from SW_17; footprint kbd:CherryMX_Hotswap -> onigaku:CherryMX_Hotswap
- SW_41: renamed from SW_18; footprint kbd:CherryMX_Hotswap -> onigaku:CherryMX_Hotswap
- SW_42: renamed from SW_51; footprint kbd:CherryMX_Hotswap -> onigaku:CherryMX_Hotswap
- SW_43: renamed from SW_52; footprint kbd:CherryMX_Hotswap -> onigaku:CherryMX_Hotswap
- SW_44: renamed from SW_53; footprint kbd:CherryMX_Hotswap -> onigaku:CherryMX_Hotswap
- SW_45: renamed from SW_54; footprint kbd:CherryMX_Hotswap -> onigaku:CherryMX_Hotswap
- SW_46: renamed from SW_55; footprint kbd:CherryMX_Hotswap -> onigaku:CherryMX_Hotswap
- SW_47: renamed from SW_56; footprint kbd:CherryMX_Hotswap_2.75u_North -> onigaku:CherryMX_Hotswap_2.75u_North
- SW_48: renamed from SW_19; footprint kbd:CherryMX_Hotswap_2.25u_North -> onigaku:CherryMX_Hotswap_2.25u_North
- SW_49: renamed from SW_20; footprint kbd:CherryMX_Hotswap -> onigaku:CherryMX_Hotswap
- SW_5: renamed from SW_33; footprint kbd:CherryMX_Hotswap -> onigaku:CherryMX_Hotswap
- SW_50: renamed from SW_21; footprint kbd:CherryMX_Hotswap -> onigaku:CherryMX_Hotswap
- SW_51: renamed from SW_22; footprint kbd:CherryMX_Hotswap -> onigaku:CherryMX_Hotswap
- SW_52: renamed from SW_23; footprint kbd:CherryMX_Hotswap -> onigaku:CherryMX_Hotswap
- SW_53: renamed from SW_24; footprint kbd:CherryMX_Hotswap -> onigaku:CherryMX_Hotswap
- SW_54: renamed from SW_57; footprint kbd:CherryMX_Hotswap_2.75u_North -> onigaku:CherryMX_Hotswap_2.75u_North
- SW_55: renamed from SW_58; footprint kbd:CherryMX_Hotswap_1.25u_North -> onigaku:CherryMX_Hotswap_1.25u_North
- SW_56: renamed from SW_59; footprint kbd:CherryMX_Hotswap_1.25u_North -> onigaku:CherryMX_Hotswap_1.25u_North
- SW_57: renamed from SW_60; footprint kbd:CherryMX_Hotswap_1.25u_North -> onigaku:CherryMX_Hotswap_1.25u_North
- SW_58: renamed from SW_61; footprint kbd:CherryMX_Hotswap_1.25u_North -> onigaku:CherryMX_Hotswap_1.25u_North
- SW_59: renamed from SW_25; footprint kbd:CherryMX_Hotswap_1.25u_North -> onigaku:CherryMX_Hotswap_1.25u_North
- SW_6: renamed from SW_34; footprint kbd:CherryMX_Hotswap -> onigaku:CherryMX_Hotswap
- SW_60: renamed from SW_26; footprint kbd:CherryMX_Hotswap_1.25u_North -> onigaku:CherryMX_Hotswap_1.25u_North
- SW_61: renamed from SW_62; footprint kbd:CherryMX_Hotswap_1.25u_North -> onigaku:CherryMX_Hotswap_1.25u_North
- SW_62: renamed from SW_27; footprint kbd:CherryMX_Hotswap_1.25u_North -> onigaku:CherryMX_Hotswap_1.25u_North
- SW_63: renamed from SW_28; footprint kbd:CherryMX_Hotswap_2.25u_North -> onigaku:CherryMX_Hotswap_2.25u_North
- SW_7: renamed from SW_35; footprint kbd:CherryMX_Hotswap -> onigaku:CherryMX_Hotswap
- SW_8: renamed from SW_0; footprint kbd:CherryMX_Hotswap -> onigaku:CherryMX_Hotswap
- SW_9: renamed from SW_1; footprint kbd:CherryMX_Hotswap -> onigaku:CherryMX_Hotswap
- renumbered D_7 to D_1, D_2 to D_10, D_3 to D_11, D_4 to D_12, D_5 to D_13, D_6 to D_14, D_23 to D_15, D_24 to D_16, D_25 to D_17, D_26 to D_18, D_27 to D_19, D_8 to D_2, D_28 to D_20, D_29 to D_21, D_30 to D_22, D_17 to D_23, D_18 to D_24, D_19 to D_25, D_20 to D_26, D_21 to D_27, D_22 to D_28, D_40 to D_29, D_9 to D_3, D_41 to D_30, D_42 to D_31, D_43 to D_32, D_44 to D_33, D_45 to D_34, D_46 to D_35, D_34 to D_36, D_35 to D_37, D_36 to D_38, D_37 to D_39, D_10 to D_4, D_38 to D_40, D_39 to D_41, D_53 to D_42, D_54 to D_43, D_55 to D_44, D_56 to D_45, D_57 to D_46, D_58 to D_47, D_47 to D_48, D_48 to D_49, D_11 to D_5, D_49 to D_50, D_50 to D_51, D_51 to D_52, D_52 to D_53, D_14 to D_54, D_64 to D_55, D_65 to D_56, D_66 to D_57, D_67 to D_58, D_60 to D_59, D_12 to D_6, D_61 to D_60, D_15 to D_61, D_13 to D_7, D_1 to D_9
Connections:
- net BACKLIGHT_LED_L: now also LED5.4 (DIN), U1.~ (A5/F1)
- net BACKLIGHT_LED_R: now also LED1.4 (DIN)
- net GND: now also J1.B, J2.B, LED1.1 (VDD), LED10.1 (VDD), LED11.1 (VDD), LED12.1 (VDD), LED13.1 (VDD), LED14.1 (VDD), LED15.1 (VDD), LED16.1 (VDD), LED17.3 (VSS), LED18.3 (VSS), LED19.3 (VSS), LED2.1 (VDD), LED20.3 (VSS), LED21.3 (VSS), LED22.3 (VSS), LED24.3 (VSS), LED25.3 (VSS), LED26.3 (VSS), LED27.3 (VSS), LED28.3 (VSS), LED29.3 (VSS), LED3.1 (VDD), LED31.3 (VSS), LED32.3 (VSS), LED34.3 (VSS), LED35.3 (VSS), LED36.3 (VSS), LED37.3 (VSS), LED39.3 (VSS), LED4.1 (VDD), LED40.3 (VSS), LED41.3 (VSS), LED42.3 (VSS), LED43.3 (VSS), LED45.3 (VSS), LED46.3 (VSS), LED47.3 (VSS), LED48.3 (VSS), LED49.3 (VSS), LED5.1 (VDD), LED50.3 (VSS), LED51.3 (VSS), LED52.3 (VSS), LED53.3 (VSS), LED54.3 (VSS), LED55.3 (VSS), LED56.3 (VSS), LED58.3 (VSS), LED59.3 (VSS), LED6.1 (VDD), LED60.3 (VSS), LED61.3 (VSS), LED62.3 (VSS), LED63.3 (VSS), LED64.3 (VSS), LED65.3 (VSS), LED66.3 (VSS), LED67.3 (VSS), LED68.3 (VSS), LED7.1 (VDD), LED70.3 (VSS), LED71.3 (VSS), LED72.3 (VSS), LED75.3 (VSS), LED76.3 (VSS), LED77.3 (VSS), LED78.3 (VSS), LED8.1 (VDD), LED9.1 (VDD), RSW1.2, U1.23 (GND), U1.3 (GND), U1.4 (GND), U2.23 (GND), U2.3 (GND), U2.4 (GND)
- net VCC: now also J1.A, J2.A, LED1.3 (VSS), LED10.3 (VSS), LED11.3 (VSS), LED12.3 (VSS), LED13.3 (VSS), LED14.3 (VSS), LED15.3 (VSS), LED16.3 (VSS), LED17.1 (VDD), LED18.1 (VDD), LED19.1 (VDD), LED2.3 (VSS), LED20.1 (VDD), LED21.1 (VDD), LED22.1 (VDD), LED23.1 (VDD), LED24.1 (VDD), LED25.1 (VDD), LED26.1 (VDD), LED27.1 (VDD), LED28.1 (VDD), LED29.1 (VDD), LED3.3 (VSS), LED30.1 (VDD), LED31.1 (VDD), LED32.1 (VDD), LED34.1 (VDD), LED35.1 (VDD), LED36.1 (VDD), LED37.1 (VDD), LED38.1 (VDD), LED39.1 (VDD), LED4.3 (VSS), LED40.1 (VDD), LED41.1 (VDD), LED42.1 (VDD), LED43.1 (VDD), LED44.1 (VDD), LED45.1 (VDD), LED46.1 (VDD), LED47.1 (VDD), LED48.1 (VDD), LED49.1 (VDD), LED5.3 (VSS), LED50.1 (VDD), LED51.1 (VDD), LED52.1 (VDD), LED53.1 (VDD), LED54.1 (VDD), LED55.1 (VDD), LED56.1 (VDD), LED57.1 (VDD), LED58.1 (VDD), LED59.1 (VDD), LED6.3 (VSS), LED60.1 (VDD), LED61.1 (VDD), LED62.1 (VDD), LED63.1 (VDD), LED64.1 (VDD), LED65.1 (VDD), LED66.1 (VDD), LED67.1 (VDD), LED68.1 (VDD), LED69.1 (VDD), LED7.3 (VSS), LED70.1 (VDD), LED71.1 (VDD), LED72.1 (VDD), LED73.1 (VDD), LED74.1 (VDD), LED75.1 (VDD), LED76.1 (VDD), LED77.1 (VDD), LED78.1 (VDD), LED79.1 (VDD), LED8.3 (VSS), LED9.3 (VSS), U1.21 (VCC), U2.21 (VCC)
- net col0_L: now also U1.20 (F4/D21/A3)
- net col0_R: now also U2.11 (D8/A8/B4), U2.20 (F4/D21/A3)
- net col1_L: now also U1.19 (F5/D20/A2)
- net col1_R: now also U2.19 (F5/D20/A2)
- net col2_L: now also U1.18 (F6/D19/A1)
- net col2_R: now also U2.18 (F6/D19/A1)
- net col3_L: now also U1.17 (F7/D18/A0)
- net col3_R: now also U2.17 (F7/D18/A0)
- net col4_L: now also U1.16 (B1/D16/SCLK)
- net col4_R: now also U2.16 (B1/D16/SCLK)
- net col5_L: now also U1.15 (B3/D14/MISO)
- net col5_R: now also U2.15 (B3/D14/MISO)
- net col6_L: now also U1.14 (B2/D16/MOSI)
- net col6_R: now also U2.14 (B2/D16/MOSI)
- net col7_R: now also U2.13 (B6/D10/A10)
- net reset_L: now also U1.22 (RST)
- net reset_R: now also RSW1.1, U2.22 (RST)
- net row0_L: now also D_8.1 (K), U1.7 (D4/A6/D4)
- net row0_R: now also U2.7 (D4/A6/D4)
- net row1_L: now also U1.8 (D12/C6)
- net row1_R: now also U2.8 (D12/C6)
- net row2_L: now also U1.9 (D6/A7/D7)
- net row2_R: now also U2.9 (D6/A7/D7)
- net row3_L: now also U1.10 (D7/E6)
- net row3_R: now also U2.10 (D7/E6)
- net row4_L: now also U1.11 (D8/A8/B4)
- net at SW_8.2 (ROW): now also D_8.2 (A)
- new net: LED25.2 (DOUT), LED64.4 (DIN)
- new net: LED25.4 (DIN), LED26.2 (DOUT)
- new net: LED26.4 (DIN), LED40.2 (DOUT)
- new net: LED27.2 (DOUT), LED41.4 (DIN)
- new net: LED27.4 (DIN), LED28.2 (DOUT)
- new net: LED28.4 (DIN), LED42.2 (DOUT)
- new net: LED29.2 (DOUT), LED43.4 (DIN)
- new net: LED29.4 (DIN), LED30.2 (DOUT)
- new net: LED30.3 (VSS), LED44.3 (VSS), LED57.3 (VSS), LED69.3 (VSS), LED79.3 (VSS)
- new net: LED30.4 (DIN), LED44.2 (DOUT)
- new net: LED40.4 (DIN), LED53.2 (DOUT)
- new net: LED41.2 (DOUT), LED54.4 (DIN)
- new net: LED42.4 (DIN), LED55.2 (DOUT)
- new net: LED43.2 (DOUT), LED56.4 (DIN)
- new net: LED44.4 (DIN), LED57.2 (DOUT)
- new net: LED53.4 (DIN), LED65.2 (DOUT)
- new net: LED54.2 (DOUT), LED66.4 (DIN)
- new net: LED55.4 (DIN), LED67.2 (DOUT)
- new net: LED56.2 (DOUT), LED68.4 (DIN)
- new net: LED57.4 (DIN), LED69.2 (DOUT)
- new net: LED67.4 (DIN), LED68.2 (DOUT)
- new net: LED24.4 (DIN), LED39.2 (DOUT)
- new net: LED39.4 (DIN), LED52.2 (DOUT)
- new net: LED52.4 (DIN), LED75.2 (DOUT)
- new net: LED75.4 (DIN), LED76.2 (DOUT)
- new net: LED64.2 (DOUT), LED76.4 (DIN)
- new net: LED65.4 (DIN), LED77.2 (DOUT)
- new net: LED77.4 (DIN), LED78.2 (DOUT)
- new net: LED13.2 (DOUT), LED79.4 (DIN)
- new net: LED5.2 (DOUT), LED6.4 (DIN)
- new net: LED6.2 (DOUT), LED7.4 (DIN)
- new net: LED7.2 (DOUT), LED8.4 (DIN)
- new net: LED16.4 (DIN), LED8.2 (DOUT)
- new net: LED15.4 (DIN), LED16.2 (DOUT)
- new net: LED14.4 (DIN), LED15.2 (DOUT)
- new net: LED19.2 (DOUT), LED33.4 (DIN)
- new net: LED19.4 (DIN), LED20.2 (DOUT)
- new net: LED20.4 (DIN), LED34.2 (DOUT)
- new net: LED21.2 (DOUT), LED35.4 (DIN)
- new net: LED21.4 (DIN), LED22.2 (DOUT)
- new net: LED22.4 (DIN), LED36.2 (DOUT)
- new net: LED23.2 (DOUT), LED37.4 (DIN)
- new net: LED23.3 (VSS), LED38.3 (VSS), LED74.3 (VSS)
- new net: LED23.4 (DIN), LED38.2 (DOUT)
- new net: LED34.4 (DIN), LED48.2 (DOUT)
- new net: LED35.2 (DOUT), LED49.4 (DIN)
- new net: LED36.4 (DIN), LED50.2 (DOUT)
- new net: LED37.2 (DOUT), LED51.4 (DIN)
- new net: LED38.4 (DIN), LED74.2 (DOUT)
- new net: LED48.4 (DIN), LED61.2 (DOUT)
- new net: LED49.2 (DOUT), LED62.4 (DIN)
- new net: LED51.2 (DOUT), LED63.4 (DIN)
- new net: LED17.4 (DIN), LED18.2 (DOUT)
- new net: LED18.4 (DIN), LED32.2 (DOUT)
- new net: LED32.4 (DIN), LED46.2 (DOUT)
- new net: LED46.4 (DIN), LED59.2 (DOUT)
- new net: LED47.2 (DOUT), LED60.4 (DIN)
- new net: LED33.2 (DOUT), LED47.4 (DIN)
- new net: LED61.4 (DIN), LED71.2 (DOUT)
- new net: LED71.4 (DIN), LED72.2 (DOUT)
- new net: LED74.4 (DIN), LED9.2 (DOUT)
- new net: LED59.4 (DIN), LED60.2 (DOUT)
- new net: LED63.2 (DOUT), LED73.4 (DIN)
- new net: LED1.2 (DOUT), LED2.4 (DIN)
- new net: LED12.4 (DIN), LED4.2 (DOUT)
- new net: LED3.2 (DOUT), LED4.4 (DIN)
- new net: LED11.4 (DIN), LED12.2 (DOUT)
- new net: LED10.4 (DIN), LED11.2 (DOUT)
- new net: LED2.2 (DOUT), LED3.4 (DIN)
- new net: LED17.2 (DOUT), LED31.4 (DIN)
- new net: LED31.2 (DOUT), LED45.4 (DIN)
- new net: LED45.2 (DOUT), LED58.4 (DIN)
- new net: LED58.2 (DOUT), LED70.4 (DIN)
- new net data_L: J1.D, U1.2 (RX/D0/D2)
- new net data_R: J2.D, U2.2 (RX/D0/D2)
- no-connect marks 25 -> 3
Other:
- note removed: "7, 8, 9, 0, -, +, bckspace"
- note removed: "Ctrl, Win, Fnc, Alt, Spacebar"
- note removed: "Esc, 1, 2, 3, 4, 5, 6"
- note removed: "MASTER @ 0xA0"
- note removed: "SLAVE @ 0xA1 (See IS31FL3733 datasheet)"
- note removed: "Tab, q, w, e, r, t"
- note removed: "cpslck, a, s"
- note removed: "d, f, g"
- note removed: "h"
- note removed: "j, k, l, m, ;, ', enter"
- note removed: "shift, z, x, c, v, b"
- note removed: "space, alt, fn, win, ctrl"
- note removed: "y, u, i, o, p, [, ], \"
- moved on the sheet: D_1, D_10, D_11, D_12, D_13, D_14, D_15, D_16, D_17, D_18, D_19, D_2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

Commit message: lined up rgb leds, WIP on adding bypass capacitors
Parts:
- removed U1, U2: elite-c, keebio:Elite-C, symbol onigaku:elite-c
- added 0.1uF (x5): C_Small, symbol Device:C_Small
- added C? (x18): 0.1uF, symbol Device:C_Small
- added LED80, LED81, LED82, LED83, LED84, LED85, LED86, LED87: YS-SK6812MINI-E, kbd:YS-SK6812MINI-E_underglow, symbol kbd:YS-SK6812MINI-E
- added OL1, OL2: OLED, kbd:OLED_v2, symbol kbd:OLED
- added R1, R2: 500, Resistor_SMD:R_0805_2012Metric_Pad1.20x1.40mm_HandSolder, symbol Device:R_Small
- added U1, U2: Elite-C, keebio:Elite-C, symbol keebio:Elite-C
- J1: footprint onigaku:MJ-4PP-9_1side -> kbd:MJ-4PP-9_1side
- J2: footprint onigaku:MJ-4PP-9 -> kbd:MJ-4PP-9_1side
- LED1, LED10, LED11, LED12, LED13, LED14, LED15, LED16, LED2, LED3, LED4, LED5, LED6, LED7, LED8, LED9: footprint onigaku:YS-SK6812MINI-E -> kbd:YS-SK6812MINI-E_underglow
- LED17, LED18, LED19, LED20, LED21, LED22, LED23, LED24, LED25, LED26, LED27, LED28, LED29, LED30, LED31, LED32, LED33, LED34, LED35, LED36, LED37, LED38, LED39, LED40, LED41, LED42, LED43, LED44, LED45, LED46, LED47, LED48, LED49, LED50, LED51, LED52, LED53, LED54, LED55, LED56, LED57, LED58, LED59, LED60, LED61, LED62, LED63, LED64, LED65, LED66, LED67, LED68, LED69, LED70, LED71, LED72, LED73, LED74, LED75, LED76, LED77, LED78, LED79: footprint onigaku:YS-SK6812MINI-E -> kbd:YS-SK6812MINI-E
- RSW1: footprint onigaku:ResetSW -> Button_Switch_SMD:SW_SPST_TL3342
- RSW2: footprint onigaku:ResetSW_1side -> Button_Switch_SMD:SW_SPST_TL3342
- SW_1, SW_10, SW_11, SW_12, SW_13, SW_14, SW_15, SW_16, SW_17, SW_18, SW_19, SW_2, SW_20, SW_21, SW_24, SW_25, SW_26, SW_27, SW_28, SW_29, SW_3, SW_30, SW_31, SW_32, SW_33, SW_34, SW_37, SW_38, SW_39, SW_4, SW_40, SW_41, SW_42, SW_43, SW_44, SW_45, SW_46, SW_49, SW_5, SW_50, SW_51, SW_52, SW_53, SW_6, SW_8, SW_9: footprint onigaku:CherryMX_Hotswap -> kbd:CherryMX_Hotswap
- SW_22, SW_23: footprint onigaku:CherryMX_Hotswap -> kbd:CherryMX_Hotswap_1.5u
- SW_35: footprint onigaku:CherryMX_Hotswap -> kbd:CherryMX_Hotswap_2.25u_North
- SW_36: footprint onigaku:CherryMX_Hotswap -> kbd:CherryMX_Hotswap_1.75u
- SW_47, SW_54: footprint onigaku:CherryMX_Hotswap_2.75u_North -> kbd:CherryMX_Hotswap_2.75u_North
- SW_48, SW_63: footprint onigaku:CherryMX_Hotswap_2.25u_North -> kbd:CherryMX_Hotswap_2.25u_North
- SW_55, SW_56, SW_57, SW_58, SW_59, SW_60, SW_61, SW_62: footprint onigaku:CherryMX_Hotswap_1.25u_North -> kbd:CherryMX_Hotswap_1.25u_North
- SW_7: footprint onigaku:CherryMX_Hotswap -> kbd:CherryMX_Hotswap_2u_North
Connections:
- net BACKLIGHT_LED_L: now also R2.1; no longer LED5.4 (DIN)
- net BACKLIGHT_LED_R: now also R1.1; no longer LED1.4 (DIN)
- net GND: now also LED1.3 (VSS), LED10.3 (VSS), LED11.3 (VSS), LED12.3 (VSS), LED13.3 (VSS), LED14.3 (VSS), LED15.3 (VSS), LED16.3 (VSS), LED2.3 (VSS), LED23.3 (VSS), LED3.3 (VSS), LED30.3 (VSS), LED38.3 (VSS), LED4.3 (VSS), LED44.3 (VSS), LED5.3 (VSS), LED57.3 (VSS), LED6.3 (VSS), LED69.3 (VSS), LED7.3 (VSS), LED74.3 (VSS), LED79.3 (VSS), LED8.3 (VSS), LED9.3 (VSS), 0.1uF.2, 0.1uF.2, 0.1uF.2, 0.1uF.2, 0.1uF.2, C?.1, C?.2, C?.2, C?.2, C?.2, C?.2, C?.2, C?.2, C?.2, C?.2, C?.2, C?.2, C?.2, LED80.3 (VSS), LED81.3 (VSS), LED84.3 (VSS), LED85.3 (VSS), OL1.4 (GND), OL2.4 (GND), U1.2 (RX1/PD2), U1.24 (B0), U1.3 (GND), U2.2 (RX1/PD2), U2.24 (B0), U2.3 (GND); no longer LED1.1 (VDD), LED10.1 (VDD), LED11.1 (VDD), LED12.1 (VDD), LED13.1 (VDD), LED14.1 (VDD), LED15.1 (VDD), LED16.1 (VDD), LED2.1 (VDD), LED3.1 (VDD), LED4.1 (VDD), LED5.1 (VDD), LED6.1 (VDD), LED7.1 (VDD), LED8.1 (VDD), LED9.1 (VDD)
- net VCC: now also LED1.1 (VDD), LED10.1 (VDD), LED11.1 (VDD), LED12.1 (VDD), LED13.1 (VDD), LED14.1 (VDD), LED15.1 (VDD), LED16.1 (VDD), LED2.1 (VDD), LED3.1 (VDD), LED4.1 (VDD), LED5.1 (VDD), LED6.1 (VDD), LED7.1 (VDD), LED8.1 (VDD), LED9.1 (VDD), 0.1uF.1, 0.1uF.1, 0.1uF.1, 0.1uF.1, 0.1uF.1, C?.1, C?.1, C?.1, C?.1, C?.1, C?.1, C?.1, C?.1, C?.1, C?.1, C?.1, C?.1, C?.1, C?.1, C?.1, C?.1, C?.1, C?.2, LED80.1 (VDD), LED81.1 (VDD), LED82.1 (VDD), LED83.1 (VDD), LED84.1 (VDD), LED85.1 (VDD), LED86.1 (VDD), LED87.1 (VDD), U1.22 (RST), U2.22 (RST); no longer LED1.3 (VSS), LED10.3 (VSS), LED11.3 (VSS), LED12.3 (VSS), LED13.3 (VSS), LED14.3 (VSS), LED15.3 (VSS), LED16.3 (VSS), LED2.3 (VSS), LED3.3 (VSS), LED4.3 (VSS), LED5.3 (VSS), LED6.3 (VSS), LED7.3 (VSS), LED8.3 (VSS), LED9.3 (VSS)
- net col0_L: now also U1.21 (VCC)
- net col0_R: now also SW_54.1 (COL), U2.21 (VCC); no longer D_54.1 (K), D_55.1 (K), D_56.1 (K), D_57.1 (K), D_58.1 (K)
- net col1_L: now also U1.20 (A3/PF4)
- net col1_R: now also U2.20 (A3/PF4)
- net col2_L: now also U1.19 (A2/PF5)
- net col2_R: now also U2.19 (A2/PF5)
- net col3_L: now also U1.18 (A1/PF6)
- net col3_R: now also U2.18 (A1/PF6)
- net col4_L: now also U1.17 (A0/PF7)
- net col4_R: now also U2.17 (A0/PF7)
- net col5_L: now also U1.16 (15/PB1)
- net col5_R: now also U2.16 (15/PB1)
- net col6_L: now also U1.15 (14/PB3)
- net col6_R: now also U2.15 (14/PB3)
- net col7_R: now also U2.14 (16/PB2)
- net data_L: now also U1.1 (TX0/PD3)
- net data_R: now also U2.1 (TX0/PD3)
- net reset_L: now also U1.23 (GND)
- net reset_R: now also U2.23 (GND)
- net row0_L: now also U1.6 (3/PD0)
- net row0_R: now also U2.6 (3/PD0)
- net row1_L: now also U1.7 (4/PD4)
- net row1_R: now also U2.7 (4/PD4)
- net row2_L: now also U1.8 (5/PC6)
- net row2_R: now also U2.8 (5/PC6)
- net row3_L: now also U1.9 (6/PD7)
- net row3_R: now also U2.9 (6/PD7)
- net row4_L: now also U1.10 (7/PE6)
- net at LED69.4 (DIN): now also LED79.2 (DOUT)
- net at LED16.4 (DIN): now also LED86.2 (DOUT); no longer LED8.2 (DOUT)
- net at LED14.2 (DOUT): now also LED13.4 (DIN)
- net at LED12.4 (DIN): now also LED84.2 (DOUT); no longer LED4.2 (DOUT)
- net at LED10.2 (DOUT): now also LED9.4 (DIN)
- new net: LED83.2 (DOUT), LED87.4 (DIN)
- new net: C?.2, C?.2, C?.2, C?.2, C?.2, LED82.3 (VSS), LED83.3 (VSS), LED86.3 (VSS), LED87.3 (VSS)
- new net: LED82.2 (DOUT), LED83.4 (DIN)
- new net: LED86.4 (DIN), LED87.2 (DOUT)
- new net: LED8.2 (DOUT), LED82.4 (DIN)
- new net: LED81.2 (DOUT), LED85.4 (DIN)
- new net: LED80.2 (DOUT), LED81.4 (DIN)
- new net: LED84.4 (DIN), LED85.2 (DOUT)
- new net: LED4.2 (DOUT), LED80.4 (DIN)
- new net: LED5.4 (DIN), R2.2
- new net: LED1.4 (DIN), R1.2
- new net 5V+: OL1.3 (VCC), OL2.3 (VCC)
- new net SCL_L: OL2.2 (SCL), U1.5 (2/PD1)
- new net SCL_R: OL1.2 (SCL), U2.5 (2/PD1)
- new net SDA_L: OL2.1 (SDA), U1.4 (GND)
- new net SDA_R: OL1.1 (SDA), U2.4 (GND)
- new net row4_R: D_54.1 (K), D_55.1 (K), D_56.1 (K), D_57.1 (K), D_58.1 (K), U2.10 (7/PE6)
Other:
- moved on the sheet: D_1, D_10, D_11, D_12, D_13, D_14, D_15, D_16, D_17, D_18, D_19, D_2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
