File: onigaku.sch (KiCad schematic (older format))
At the start: 246 parts, among them J1 MJ-4PP-9, J2 MJ-4PP-9, U1 Elite-C, U2 Elite-C

Commit message: rearranged leds, moved caps, adjusting size of keyboard
Parts:
- removed 0.1uF (x5): C_Small, symbol Device:C_Small
- added C13, C14, C15, C16, C17, C23, C24, C25, C26, C27, C28, C29, C30, C31, C32, C33, C34, C35, C36, C37, C38, C39, C40, C41, C42, C43, C44, C45, C46, C47, C48, C49, C50, C51, C52, C53, C54, C55, C56, C57, C58, C59, C60, C61, C62, C63, C64, C65, C66, C67, C68, C69, C70, C71, C72, C73, C74, C75, C76, C77, C78, C79, C80, C82, C83, C84, C85, C86, C87: 0.1uF, Capacitor_SMD:C_0603_1608Metric_Pad1.08x0.95mm_HandSolder, symbol Device:C_Small
- added R3, R4: 500, Resistor_SMD:R_0805_2012Metric_Pad1.20x1.40mm_HandSolder, symbol Device:R_Small
- C1, C10, C11, C12, C18, C19, C2, C20, C21, C22, C3, C4, C5, C6, C7, C8, C81, C9: renamed from C?; footprint (none) -> Capacitor_SMD:C_0603_1608Metric_Pad1.08x0.95mm_HandSolder
- renumbered LED8 to LED10, LED82 to LED11, LED83 to LED12, LED9 to LED13, LED10 to LED14, LED11 to LED15, LED12 to LED16, LED84 to LED17, LED85 to LED18, LED13 to LED19, LED14 to LED20, LED15 to LED21, LED16 to LED22, LED86 to LED23, LED87 to LED24, LED17 to LED25, LED18 to LED26, LED19 to LED27, LED20 to LED28, LED21 to LED29, LED22 to LED30, LED23 to LED31, LED24 to LED32, LED25 to LED33, LED26 to LED34, LED27 to LED35, LED28 to LED36, LED29 to LED37, LED30 to LED38, LED31 to LED39, LED32 to LED40, LED33 to LED41, LED34 to LED42, LED35 to LED43, LED36 to LED44, LED37 to LED45, LED38 to LED46, LED39 to LED47, LED40 to LED48, LED41 to LED49, LED80 to LED5, LED42 to LED50, LED43 to LED51, LED44 to LED52, LED45 to LED53, LED46 to LED54, LED47 to LED55, LED48 to LED56, LED49 to LED57, LED50 to LED58, LED51 to LED59, LED81 to LED6, LED52 to LED60, LED53 to LED61, LED54 to LED62, LED55 to LED63, LED56 to LED64, LED57 to LED65, LED58 to LED66, LED59 to LED67, LED60 to LED68, LED61 to LED69, LED5 to LED7, LED62 to LED70, LED63 to LED71, LED64 to LED72, LED65 to LED73, LED66 to LED74, LED67 to LED75, LED68 to LED76, LED69 to LED77, LED70 to LED78, LED71 to LED79, LED6 to LED8, LED72 to LED80, LED73 to LED81, LED74 to LED82, LED75 to LED83, LED76 to LED84, LED77 to LED85, LED78 to LED86, LED79 to LED87, LED7 to LED9, U2 to U1, U1 to U2
Connections:
- net BACKLIGHT_LED_L: now also U2.29 (F0)
- net BACKLIGHT_LED_R: now also U1.25 (B7)
- net GND: now also C10.2, C12.2, C21.2, C22.2, C9.2, LED11.3 (VSS), LED12.3 (VSS), LED23.3 (VSS), LED24.3 (VSS), U2.23 (GND), U2.4 (GND), C30.1, C31.1, C32.1, C33.1, C34.1, C35.1, C36.2, C45.1, C46.1, C47.1, C48.1, C49.1, C57.1, C58.1, C59.1, C60.1, C61.1, C68.1, C69.1, C70.1, C71.1, C72.1, C78.1, C79.1, C80.1, C82.1, C83.1, C84.1, C85.1, C87.2; no longer C1.2, C11.2, C2.2, C3.2, C4.2, C5.2, J2.B, LED1.3 (VSS), LED13.3 (VSS), LED14.3 (VSS), LED15.3 (VSS), LED16.3 (VSS), LED17.3 (VSS), LED18.3 (VSS), LED2.3 (VSS), LED25.3 (VSS), LED26.3 (VSS), LED27.3 (VSS), LED28.3 (VSS), LED29.3 (VSS), LED3.3 (VSS), LED30.3 (VSS), LED31.3 (VSS), LED39.3 (VSS), LED4.3 (VSS), LED40.3 (VSS), LED42.3 (VSS), LED43.3 (VSS), LED44.3 (VSS), LED45.3 (VSS), LED46.3 (VSS), LED5.3 (VSS), LED53.3 (VSS), LED54.3 (VSS), LED55.3 (VSS), LED56.3 (VSS), LED57.3 (VSS), LED58.3 (VSS), LED59.3 (VSS), LED6.3 (VSS), LED66.3 (VSS), LED67.3 (VSS), LED68.3 (VSS), LED69.3 (VSS), LED70.3 (VSS), LED71.3 (VSS), LED78.3 (VSS), LED79.3 (VSS), LED80.3 (VSS), LED82.3 (VSS), OL1.4 (GND), RSW1.2, U1.2 (RX1/PD2), U1.24 (B0), U1.3 (GND), U2.2 (RX1/PD2), U2.24 (B0)
- net SCL_L: now also U2.6 (3/PD0); no longer U2.5 (2/PD1)
- net SCL_R: now also U1.6 (3/PD0); no longer U1.5 (2/PD1)
- net SDA_L: now also U2.5 (2/PD1); no longer U2.4 (GND)
- net SDA_R: now also U1.5 (2/PD1); no longer U1.4 (GND)
- net VCC: now also OL2.3 (VCC), U2.21 (VCC), C30.2, C31.2, C32.2, C33.2, C34.2, C35.2, C36.1, C45.2, C46.2, C47.2, C48.2, C49.2, C57.2, C58.2, C59.2, C60.2, C61.2, C68.2, C69.2, C70.2, C71.2, C72.2, C78.2, C79.2, C80.2, C82.2, C83.2, C84.2, C85.2, C87.1; no longer C1.1, C11.1, C2.1, C3.1, C4.1, C5.1, J2.A, LED1.1 (VDD), LED13.1 (VDD), LED14.1 (VDD), LED15.1 (VDD), LED16.1 (VDD), LED17.1 (VDD), LED18.1 (VDD), LED2.1 (VDD), LED25.1 (VDD), LED26.1 (VDD), LED27.1 (VDD), LED28.1 (VDD), LED29.1 (VDD), LED3.1 (VDD), LED30.1 (VDD), LED31.1 (VDD), LED39.1 (VDD), LED4.1 (VDD), LED40.1 (VDD), LED42.1 (VDD), LED43.1 (VDD), LED44.1 (VDD), LED45.1 (VDD), LED46.1 (VDD), LED5.1 (VDD), LED53.1 (VDD), LED54.1 (VDD), LED55.1 (VDD), LED56.1 (VDD), LED57.1 (VDD), LED58.1 (VDD), LED59.1 (VDD), LED6.1 (VDD), LED66.1 (VDD), LED67.1 (VDD), LED68.1 (VDD), LED69.1 (VDD), LED70.1 (VDD), LED71.1 (VDD), LED78.1 (VDD), LED79.1 (VDD), LED80.1 (VDD), LED81.1 (VDD), LED82.1 (VDD), U1.22 (RST), U2.22 (RST)
- net col0_L: now also U2.20 (A3/PF4); no longer U2.21 (VCC)
- net col0_R: now also U1.20 (A3/PF4); no longer U1.21 (VCC)
- net col1_L: now also U2.19 (A2/PF5); no longer U2.20 (A3/PF4)
- net col1_R: now also U1.19 (A2/PF5); no longer U1.20 (A3/PF4)
- net col2_L: now also U2.18 (A1/PF6); no longer U2.19 (A2/PF5)
- net col2_R: now also U1.18 (A1/PF6); no longer U1.19 (A2/PF5)
- net col3_L: now also U2.17 (A0/PF7); no longer U2.18 (A1/PF6)
- net col3_R: now also U1.17 (A0/PF7); no longer U1.18 (A1/PF6)
- net col4_L: now also U2.16 (15/PB1); no longer U2.17 (A0/PF7)
- net col4_R: now also U1.16 (15/PB1); no longer U1.17 (A0/PF7)
- net col5_L: now also U2.15 (14/PB3); no longer U2.16 (15/PB1)
- net col5_R: now also U1.15 (14/PB3); no longer U1.16 (15/PB1)
- net col6_L: now also U2.14 (16/PB2); no longer U2.15 (14/PB3)
- net col6_R: now also U1.14 (16/PB2); no longer U1.15 (14/PB3)
- net col7_R: now also U1.13 (10/PB6); no longer U1.14 (16/PB2)
- net data_L: now also U2.2 (RX1/PD2); no longer U2.1 (TX0/PD3)
- net data_R: now also U1.2 (RX1/PD2); no longer U1.1 (TX0/PD3)
- net reset_L: now also U2.22 (RST); no longer U2.23 (GND)
- net reset_R: now also U1.22 (RST); no longer U1.23 (GND)
- net row0_L: now also U2.7 (4/PD4); no longer U2.6 (3/PD0)
- net row0_R: now also U1.7 (4/PD4); no longer U1.6 (3/PD0)
- net row1_L: now also U2.8 (5/PC6); no longer U2.7 (4/PD4)
- net row1_R: now also U1.8 (5/PC6); no longer U1.7 (4/PD4)
- net row2_L: now also U2.9 (6/PD7); no longer U2.8 (5/PC6)
- net row2_R: now also U1.9 (6/PD7); no longer U1.8 (5/PC6)
- net row3_L: now also U2.10 (7/PE6); no longer U2.9 (6/PD7)
- net row3_R: now also U1.10 (7/PE6); no longer U1.9 (6/PD7)
- net row4_L: now also U2.11 (8/PB4); no longer U2.10 (7/PE6)
- net row4_R: now also U1.11 (8/PB4); no longer U1.10 (7/PE6)
- net at LED33.4 (DIN): now also LED32.2 (DOUT); no longer LED34.2 (DOUT)
- net at LED35.4 (DIN): now also LED34.2 (DOUT); no longer LED36.2 (DOUT)
- net at LED37.4 (DIN): now also LED36.2 (DOUT); no longer LED38.2 (DOUT)
- net at LED75.4 (DIN): no longer LED76.2 (DOUT)
- net at LED84.2 (DOUT): now also LED85.4 (DIN); no longer LED83.4 (DIN)
- net at LED86.2 (DOUT): no longer LED85.4 (DIN)
- net at LED86.4 (DIN): now also LED74.2 (DOUT)
- net at LED87.4 (DIN): now also LED76.2 (DOUT); no longer LED19.2 (DOUT)
- net at LED6.2 (DOUT): no longer LED18.4 (DIN)
- net at R1.2: now also LED18.4 (DIN); no longer LED1.4 (DIN)
- net LED_L: now reaches U2.12 (9/PB5)
- net LED_L: now also R4.2
- net LED_R: now reaches U1.12 (9/PB5)
- net LED_R: now also R3.2
- net at LED58.4 (DIN): now also LED81.2 (DOUT)
- net at LED82.4 (DIN): now also R3.1; no longer LED13.2 (DOUT)
- net VDD: now reaches LED41.1 (VDD)
- net VDD: now also C1.1, C11.1, C2.1, C3.1, C4.1, C5.1, J2.A, LED1.1 (VDD), LED13.1 (VDD), LED14.1 (VDD), LED15.1 (VDD), LED16.1 (VDD), LED17.1 (VDD), LED18.1 (VDD), LED2.1 (VDD), LED25.1 (VDD), LED26.1 (VDD), LED27.1 (VDD), LED28.1 (VDD), LED29.1 (VDD), LED3.1 (VDD), LED30.1 (VDD), LED31.1 (VDD), LED39.1 (VDD), LED4.1 (VDD), LED40.1 (VDD), LED42.1 (VDD), LED43.1 (VDD), LED44.1 (VDD), LED45.1 (VDD), LED46.1 (VDD), LED5.1 (VDD), LED53.1 (VDD), LED54.1 (VDD), LED55.1 (VDD), LED56.1 (VDD), LED57.1 (VDD), LED58.1 (VDD), LED59.1 (VDD), LED6.1 (VDD), LED66.1 (VDD), LED67.1 (VDD), LED68.1 (VDD), LED69.1 (VDD), LED70.1 (VDD), LED71.1 (VDD), LED78.1 (VDD), LED79.1 (VDD), LED80.1 (VDD), LED81.1 (VDD), LED82.1 (VDD), OL1.3 (VCC), U1.21 (VCC), C13.1, C14.1, C15.1, C16.1, C17.1, C23.2, C24.2, C25.2, C26.2, C27.2, C28.2, C29.2, C37.2, C38.2, C39.2, C40.2, C41.2, C42.2, C43.2, C44.1, C50.2, C51.2, C52.2, C53.2, C54.2, C55.2, C56.2, C62.2, C63.2, C64.2, C65.2, C66.2, C67.2, C73.2, C74.2, C75.2, C76.2, C77.1, C86.1
- net GNDA: now reaches LED41.3 (VSS)
- net GNDA: now also C1.2, C11.2, C2.2, C3.2, C4.2, C5.2, J2.B, LED1.3 (VSS), LED13.3 (VSS), LED14.3 (VSS), LED15.3 (VSS), LED16.3 (VSS), LED17.3 (VSS), LED18.3 (VSS), LED2.3 (VSS), LED25.3 (VSS), LED26.3 (VSS), LED27.3 (VSS), LED28.3 (VSS), LED29.3 (VSS), LED3.3 (VSS), LED30.3 (VSS), LED31.3 (VSS), LED39.3 (VSS), LED4.3 (VSS), LED40.3 (VSS), LED42.3 (VSS), LED43.3 (VSS), LED44.3 (VSS), LED45.3 (VSS), LED46.3 (VSS), LED5.3 (VSS), LED53.3 (VSS), LED54.3 (VSS), LED55.3 (VSS), LED56.3 (VSS), LED57.3 (VSS), LED58.3 (VSS), LED59.3 (VSS), LED6.3 (VSS), LED66.3 (VSS), LED67.3 (VSS), LED68.3 (VSS), LED69.3 (VSS), LED70.3 (VSS), LED71.3 (VSS), LED78.3 (VSS), LED79.3 (VSS), LED80.3 (VSS), LED81.3 (VSS), LED82.3 (VSS), OL1.4 (GND), RSW1.2, U1.23 (GND), U1.3 (GND), U1.4 (GND), C13.2, C14.2, C15.2, C16.2, C17.2, C23.1, C24.1, C25.1, C26.1, C27.1, C28.1, C29.1, C37.1, C38.1, C39.1, C40.1, C41.1, C42.1, C43.1, C44.2, C50.1, C51.1, C52.1, C53.1, C54.1, C55.1, C56.1, C62.1, C63.1, C64.1, C65.1, C66.1, C67.1, C73.1, C74.1, C75.1, C76.1, C77.2, C86.2
- net at LED70.2 (DOUT): now also LED80.4 (DIN)
- removed net 5V+: OL1.3 (VCC), OL2.3 (VCC)
- new net: LED83.4 (DIN), R4.1
- new net: LED1.4 (DIN), LED13.2 (DOUT)
- no-connect marks 3 -> 19
Other:
- moved on the sheet: C1, C11, C2, C3, C4, C5, C81, U1, U2
