File: onigaku.sch (KiCad schematic (older format))
At the start: 312 parts, among them J1 MJ-4PP-9, J2 MJ-4PP-9, U1 Elite-C, U2 Elite-C

Commit message: right side routed
Connections:
- net at LED6.2 (DOUT): now also LED1.4 (DIN)
- net at LED6.4 (DIN): now also LED13.2 (DOUT); no longer LED5.2 (DOUT)
- net at LED14.4 (DIN): now also LED5.2 (DOUT); no longer LED15.2 (DOUT)
- net at LED13.4 (DIN): now also LED15.2 (DOUT); no longer LED14.2 (DOUT)
Other:
- moved on the sheet: LED13, LED14, LED6
Changed lines of the file:
@@
 L kbd:YS-SK6812MINI-E LED14
 U 1 1 63340FE4
+P 21700 7900
+F 0 "LED14" H 22044 7930 29  0000 L CNN
+F 1 "YS-SK6812MINI-E" H 22044 7871 29  0000 L CNN
+F 2 "kbd:YS-SK6812MINI-E_underglow" H 21800 7650 50  0001 C CNN
+F 3 "" H 21800 7650 50  0001 C CNN
+	1    21700 7900
+	1    0    0    -1
+$EndComp
+Connection ~ 18650 9000
+$Comp
+L kbd:YS-SK6812MINI-E LED13
+U 1 1 63340FEE
 P 18650 8700
-F 0 "LED14" H 18994 8730 29  0000 L CNN
+F 0 "LED13" H 18994 8730 29  0000 L CNN
 F 1 "YS-SK6812MINI-E" H 18994 8671 29  0000 L CNN
 F 2 "kbd:YS-SK6812MINI-E_underglow" H 18750 8450 50  0001 C CNN
 F 3 "" H 18750 8450 50  0001 C CNN
 	1    18650 8700
-	-1   0    0    1
-$EndComp
-Connection ~ 18650 9000
-$Comp
-L kbd:YS-SK6812MINI-E LED13
-U 1 1 63340FEE
-P 17850 8700
-F 0 "LED13" H 18194 8730 29  0000 L CNN
-F 1 "YS-SK6812MINI-E" H 18194 8671 29  0000 L CNN
-F 2 "kbd:YS-SK6812MINI-E_underglow" H 17950 8450 50  0001 C CNN
-F 3 "" H 17950 8450 50  0001 C CNN
-	1    17850 8700
 	-1   0    0    1
 $EndComp
@@
 L kbd:YS-SK6812MINI-E LED6
 U 1 1 6137ED36
-P 21700 7900
-F 0 "LED6" H 22044 7930 29  0000 L CNN
-F 1 "YS-SK6812MINI-E" H 22044 7871 29  0000 L CNN
-F 2 "kbd:YS-SK6812MINI-E_underglow" H 21800 7650 50  0001 C CNN
-F 3 "" H 21800 7650 50  0001 C CNN
-	1    21700 7900
-	1    0    0    -1
-$EndComp
-$Comp
+P 17850 8700
+F 0 "LED6" H 18194 8730 29  0000 L CNN
+F 1 "YS-SK6812MINI-E" H 18194 8671 29  0000 L CNN
+F 2 "kbd:YS-SK6812MINI-E_underglow" H 17950 8450 50  0001 C CNN
+F 3 "" H 17950 8450 50  0001 C CNN
+	1    17850 8700
+	-1   0    0    1
+$EndComp
+$Comp

Commit message: wiring up oleds and trs. starting left side
Connections:
- net col0_L: now also U2.14 (16/PB2); no longer U2.20 (A3/PF4)
- net col1_L: now also U2.15 (14/PB3); no longer U2.19 (A2/PF5)
- net col2_L: now also U2.16 (15/PB1); no longer U2.18 (A1/PF6)
- net col4_L: now also U2.18 (A1/PF6); no longer U2.16 (15/PB1)
- net col5_L: now also U2.19 (A2/PF5); no longer U2.15 (14/PB3)
- net col6_L: now also U2.20 (A3/PF4); no longer U2.14 (16/PB2)
Changed lines of the file:
@@
 Text GLabel 9900 2025 0    50   Input ~ 0
 row4_L
-Text GLabel 11300 1425 2    50   Input ~ 0
+Text GLabel 11300 2025 2    50   Input ~ 0
 col0_L
-Text GLabel 11300 1525 2    50   Input ~ 0
+Text GLabel 11300 1925 2    50   Input ~ 0
 col1_L
-Text GLabel 11300 1625 2    50   Input ~ 0
+Text GLabel 11300 1825 2    50   Input ~ 0
 col2_L
 Text GLabel 11300 1725 2    50   Input ~ 0
 col3_L
-Text GLabel 11300 1825 2    50   Input ~ 0
+Text GLabel 11300 1625 2    50   Input ~ 0
 col4_L
-Text GLabel 11300 2025 2    50   Input ~ 0
+Text GLabel 11300 1425 2    50   Input ~ 0
 col6_L
 Wire Wire Line
@@
 	17300 5150 17300 6150
 Connection ~ 17300 5150
-Text GLabel 11300 1925 2    50   Input ~ 0
+Text GLabel 11300 1525 2    50   Input ~ 0
 col5_L
 Wire Wire Line

Commit message: created more traces on left, all grounds first pass
Connections:
- net at LED75.4 (DIN): now also LED85.2 (DOUT)
- net at LED84.2 (DOUT): now also LED86.4 (DIN); no longer LED85.4 (DIN)
- net at LED73.4 (DIN): now also LED86.2 (DOUT); no longer LED85.2 (DOUT)
- net at LED74.2 (DOUT): now also LED85.4 (DIN); no longer LED86.4 (DIN)
Other:
- moved on the sheet: LED85, LED86
Changed lines of the file:
@@
 $EndComp
 $Comp
-L kbd:YS-SK6812MINI-E LED85
-U 1 1 61059800
-P 4075 13625
-F 0 "LED85" H 4419 13655 29  0000 L CNN
-F 1 "YS-SK6812MINI-E" H 4419 13596 29  0000 L CNN
-F 2 "kbd:YS-SK6812MINI-E" H 4175 13375 50  0001 C CNN
-F 3 "" H 4175 13375 50  0001 C CNN
-	1    4075 13625
-	0    -1   -1   0
-$EndComp
-$Comp
 L kbd:YS-SK6812MINI-E LED87
 U 1 1 61059818
@@
 Wire Wire Line
 	4925 12475 4925 12225
-$Comp
-L kbd:YS-SK6812MINI-E LED86
-U 1 1 61059806
-P 4925 13625
-F 0 "LED86" H 5269 13655 29  0000 L CNN
-F 1 "YS-SK6812MINI-E" H 5269 13596 29  0000 L CNN
-F 2 "kbd:YS-SK6812MINI-E" H 5025 13375 50  0001 C CNN
-F 3 "" H 5025 13375 50  0001 C CNN
-	1    4925 13625
-	0    1    1    0
-$EndComp
 Connection ~ 7775 12775
 Wire Wire Line
@@
 	17550 8700 17550 7900
 Connection ~ 17850 7600
+$Comp
+L kbd:YS-SK6812MINI-E LED85
+U 1 1 61059800
+P 4925 13625
+F 0 "LED85" H 5269 13655 29  0000 L CNN
+F 1 "YS-SK6812MINI-E" H 5269 13596 29  0000 L CNN
+F 2 "kbd:YS-SK6812MINI-E" H 5025 13375 50  0001 C CNN
+F 3 "" H 5025 13375 50  0001 C CNN
+	1    4925 13625
+	0    1    1    0
+$EndComp
+$Comp
+L kbd:YS-SK6812MINI-E LED86
+U 1 1 61059806
+P 4075 13625
+F 0 "LED86" H 4419 13655 29  0000 L CNN
+F 1 "YS-SK6812MINI-E" H 4419 13596 29  0000 L CNN
+F 2 "kbd:YS-SK6812MINI-E" H 4175 13375 50  0001 C CNN
+F 3 "" H 4175 13375 50  0001 C CNN
+	1    4075 13625
+	0    -1   -1   0
+$EndComp
+Wire Wire Line
+	4925 13925 4925 13950
 $EndSCHEMATC

Commit message: adding fill areas
Parts:
- removed C19, C9: 0.1uF, Capacitor_SMD:C_0603_1608Metric_Pad1.08x0.95mm_HandSolder, symbol Device:C_Small
- removed LED11, LED20: YS-SK6812MINI-E, kbd:YS-SK6812MINI-E_underglow, symbol kbd:YS-SK6812MINI-E
Connections:
- net at LED12.2 (DOUT): no longer LED24.4 (DIN)
- net at LED12.4 (DIN): now also LED19.2 (DOUT)
- net at LED24.2 (DOUT): now also LED19.4 (DIN); no longer LED23.4 (DIN)
- net at LED23.2 (DOUT): now also LED24.4 (DIN); no longer LED22.4 (DIN)
- net at LED10.2 (DOUT): now also LED21.4 (DIN)
- net at LED22.2 (DOUT): now also LED23.4 (DIN); no longer LED21.4 (DIN)
- net at LED21.2 (DOUT): now also LED22.4 (DIN)
Other:
- moved on the sheet: C10, C12, C18, C20, C21, C22, LED12, LED19, LED21, LED22, LED23, LED24

Commit message: rewiring to make traces more readable
Connections:
- net GND: now also C30.2, C31.2, C34.2, C35.2, C57.2, C58.2, C59.2, C60.2, C61.2, C68.2, C69.2, C70.2, C71.2, C72.2, C79.2, C80.2, C82.2, C84.2, C85.2; no longer C30.1, C31.1, C34.1, C35.1, C57.1, C58.1, C59.1, C60.1, C61.1, C68.1, C69.1, C70.1, C71.1, C72.1, C79.1, C80.1, C82.1, C84.1, C85.1, LED72.3 (VSS), LED73.3 (VSS), LED74.3 (VSS), LED75.3 (VSS), LED76.3 (VSS), LED77.3 (VSS)
- net VCC: now also C30.1, C31.1, C34.1, C35.1, C57.1, C58.1, C59.1, C60.1, C61.1, C68.1, C69.1, C70.1, C71.1, C72.1, C79.1, C80.1, C82.1, C84.1, C85.1, LED72.3 (VSS), LED73.3 (VSS), LED74.3 (VSS), LED75.3 (VSS), LED76.3 (VSS), LED77.3 (VSS); no longer C30.2, C31.2, C34.2, C35.2, C57.2, C58.2, C59.2, C60.2, C61.2, C68.2, C69.2, C70.2, C71.2, C72.2, C79.2, C80.2, C82.2, C84.2, C85.2, LED63.1 (VDD)
- net at LED33.2 (DOUT): now also LED34.4 (DIN); no longer LED72.4 (DIN)
- net at LED48.2 (DOUT): now also LED47.4 (DIN); no longer LED34.4 (DIN)
- net at LED35.2 (DOUT): now also LED36.4 (DIN); no longer LED49.4 (DIN)
- net at LED50.2 (DOUT): now also LED49.4 (DIN); no longer LED36.4 (DIN)
- net at LED37.2 (DOUT): now also LED38.4 (DIN); no longer LED51.4 (DIN)
- net at LED38.2 (DOUT): now also LED52.4 (DIN)
- net at LED52.2 (DOUT): now also LED51.4 (DIN); no longer LED38.4 (DIN)
- net at LED48.4 (DIN): now also LED49.2 (DOUT); no longer LED61.2 (DOUT)
- net at LED62.4 (DIN): no longer LED49.2 (DOUT)
- net at LED50.4 (DIN): now also LED51.2 (DOUT); no longer LED63.2 (DOUT)
- net at LED64.4 (DIN): no longer LED51.2 (DOUT)
- net at LED65.2 (DOUT): no longer LED52.4 (DIN)
- net at LED61.4 (DIN): now also LED60.2 (DOUT); no longer LED73.2 (DOUT)
- net at LED62.2 (DOUT): now also LED63.4 (DIN); no longer LED74.4 (DIN)
- net at LED75.2 (DOUT): now also LED74.4 (DIN); no longer LED63.4 (DIN)
- net at LED64.2 (DOUT): no longer LED76.4 (DIN)
- net at LED65.4 (DIN): no longer LED77.2 (DOUT)
- net at LED75.4 (DIN): now also LED76.2 (DOUT); no longer LED85.2 (DOUT)
- net at LED87.4 (DIN): now also LED85.2 (DOUT); no longer LED76.2 (DOUT)
- net at LED77.4 (DIN): no longer LED87.2 (DOUT)
- net at LED32.4 (DIN): now also R4.1; no longer LED47.2 (DOUT)
- net at LED60.4 (DIN): now also LED47.2 (DOUT); no longer LED83.2 (DOUT)
- net at LED84.4 (DIN): now also LED83.2 (DOUT); no longer LED72.2 (DOUT)
- net at LED85.4 (DIN): now also LED86.2 (DOUT); no longer LED74.2 (DOUT)
- net at LED73.4 (DIN): now also LED74.2 (DOUT); no longer LED86.2 (DOUT)
- net at LED83.4 (DIN): now also LED72.2 (DOUT); no longer R4.1
- new net: LED76.4 (DIN), LED77.2 (DOUT)
- new net: LED72.4 (DIN), LED73.2 (DOUT)
Other:
- moved on the sheet: C30, C31, C32, C33, C34, C35, C36, C45, C46, C47, C48, C49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

Commit message: left side redone. wip on right side and whether or not to add nav section
Parts:
- removed D_16, D_33, D_59: D, kbd:D3_SMD_v2, symbol Device:D_Small
- added C? (x2): 0.1uF, Capacitor_SMD:C_0603_1608Metric_Pad1.08x0.95mm_HandSolder, symbol Device:C_Small
- added D_14, D_15, D_16, D_31, D_32, D_33, D_59, D_68, D_69, D_70: D, Diode_SMD:D_SOD-123, symbol Device:D_Small
- added D_16, D_33, D_59: D, kbd:D3_SMD_v2, symbol Device:D_Small
- added K_14, K_15, K_16, K_31, K_32, K_33, K_59, K_68, K_69, K_70: KEYSW, MX_Alps_Hybrid:MX-1U-NoLED, symbol MX_Alps_Hybrid:MX-NoLED
- added LED? (x10): YS-SK6812MINI-E, kbd:YS-SK6812MINI-E, symbol kbd:YS-SK6812MINI-E
Connections:
- net GND: now also LED72.3 (VSS), LED73.3 (VSS), LED74.3 (VSS), LED75.3 (VSS), LED76.3 (VSS), LED77.3 (VSS)
- net GNDA: no longer C23.1, C24.1, C25.1, C26.1, C27.1, C28.1, C29.1, C37.1, C38.1, C39.1, C40.1, C41.1, C42.1, C43.1, C44.2, C50.1, C51.1, C52.1, C53.1, C54.1, C55.1, C56.1, C62.1, C63.1, C64.1, C65.1, C66.1, C67.1, C73.1, C74.1, C75.1, C76.1, C77.2, LED25.3 (VSS), LED26.3 (VSS), LED27.3 (VSS), LED28.3 (VSS), LED29.3 (VSS), LED30.3 (VSS), LED31.3 (VSS), LED39.3 (VSS), LED40.3 (VSS), LED41.3 (VSS), LED42.3 (VSS), LED43.3 (VSS), LED44.3 (VSS), LED45.3 (VSS), LED46.3 (VSS), LED53.3 (VSS), LED54.3 (VSS), LED55.3 (VSS), LED56.3 (VSS), LED57.3 (VSS), LED58.3 (VSS), LED59.3 (VSS), LED66.3 (VSS), LED67.3 (VSS), LED68.3 (VSS), LED69.3 (VSS), LED70.3 (VSS), LED71.3 (VSS), LED78.3 (VSS), LED79.3 (VSS), LED80.3 (VSS), LED81.3 (VSS), LED82.3 (VSS)
- net VCC: now also LED63.1 (VDD); no longer LED72.3 (VSS), LED73.3 (VSS), LED74.3 (VSS), LED75.3 (VSS), LED76.3 (VSS), LED77.3 (VSS)
- net VDD: now also LED29.4 (DIN), LED30.2 (DOUT), LED31.2 (DOUT), LED43.2 (DOUT), LED44.4 (DIN), LED45.2 (DOUT), LED46.4 (DIN), LED57.4 (DIN), LED58.2 (DOUT), LED59.4 (DIN), LED70.2 (DOUT), LED71.2 (DOUT), LED80.2 (DOUT), LED81.2 (DOUT); no longer C23.2, C26.2, C27.2, C28.2, C37.2, C38.2, C39.2, C40.2, C50.2, C51.2, C52.2, C53.2, C62.2, C63.2, C64.2, C65.2, C73.2, C74.2, C77.1, LED25.1 (VDD), LED26.1 (VDD), LED27.1 (VDD), LED28.1 (VDD), LED29.1 (VDD), LED30.1 (VDD), LED31.1 (VDD), LED39.1 (VDD), LED40.1 (VDD), LED41.1 (VDD), LED42.1 (VDD), LED43.1 (VDD), LED44.1 (VDD), LED45.1 (VDD), LED46.1 (VDD), LED53.1 (VDD), LED54.1 (VDD), LED55.1 (VDD), LED56.1 (VDD), LED57.1 (VDD), LED58.1 (VDD), LED59.1 (VDD), LED66.1 (VDD), LED67.1 (VDD), LED68.1 (VDD), LED69.1 (VDD), LED70.1 (VDD), LED71.1 (VDD), LED78.1 (VDD), LED79.1 (VDD), LED80.1 (VDD), LED81.1 (VDD), LED82.1 (VDD)
- net row0_R: now also D_14.1 (K), D_15.1 (K), D_16.1 (K)
- net row1_R: now also D_16.1 (K), D_31.1 (K), D_32.1 (K), D_33.1 (K)
- net row2_R: now also D_33.1 (K)
- net row3_R: now also D_59.1 (K)
- net row4_L: now also D_59.1 (K)
- net row4_R: now also D_68.1 (K), D_69.1 (K), D_70.1 (K)
- net at SW_16.2 (ROW): now also D_16.2 (A)
- net at SW_33.2 (ROW): now also D_33.2 (A)
- net at LED61.2 (DOUT): now also LED62.4 (DIN)
- net at LED63.2 (DOUT): now also LED64.4 (DIN)
- net at LED64.2 (DOUT): now also LED65.4 (DIN)
- net at LED65.2 (DOUT): now also LED77.4 (DIN)
- net at SW_59.2 (ROW): now also D_59.2 (A)
- net col8_R: now reaches U1.27 (C7)
- net col8_R: now also K_14.1 (COL), K_31.1 (COL), K_68.1 (COL)
- net col9_R: now reaches U1.28 (F1)
- net col9_R: now also K_15.1 (COL), K_32.1 (COL), K_59.1 (COL), K_69.1 (COL)
- net col10_R: now reaches U1.29 (F0)
- net col10_R: now also K_16.1 (COL), K_33.1 (COL), K_70.1 (COL)
- net at LED27.2 (DOUT): now also C26.1; no longer LED41.4 (DIN)
- net at LED27.4 (DIN): now also C39.2, C52.2, C65.2, LED41.2 (DOUT), LED55.4 (DIN), LED68.2 (DOUT); no longer LED28.2 (DOUT)
- net at LED28.4 (DIN): no longer LED42.2 (DOUT)
- net at LED29.2 (DOUT): no longer LED43.4 (DIN)
- net at LED30.4 (DIN): now also C25.1; no longer LED44.2 (DOUT)
- net at LED45.4 (DIN): now also C43.1, C56.1, LED59.2 (DOUT); no longer LED31.2 (DOUT)
- net at LED31.4 (DIN), LED46.2 (DOUT): now also C29.1, C44.2
- net at LED42.4 (DIN), LED56.2 (DOUT): now also C40.2, C53.2, C62.2, C74.2, LED28.2 (DOUT), LED69.4 (DIN), LED79.4 (DIN)
- net at LED82.2 (DOUT): now also C77.2; no longer LED46.4 (DIN)
- net at LED56.4 (DIN): no longer LED69.2 (DOUT)
- net at LED57.2 (DOUT): no longer LED70.4 (DIN)
- net at LED58.4 (DIN): now also C55.1, LED44.2 (DOUT); no longer LED81.2 (DOUT)
- net at LED71.4 (DIN): no longer LED59.2 (DOUT)
- net at LED25.4 (DIN), LED26.2 (DOUT): now also C23.2, C26.2, C27.2, C28.2, C37.2, C38.2, C50.2, C51.2, C63.2, C64.2, C73.2, LED39.2 (DOUT), LED40.4 (DIN), LED53.4 (DIN), LED54.2 (DOUT), LED66.2 (DOUT), LED67.4 (DIN), LED78.2 (DOUT)
- net at LED26.4 (DIN): now also C28.1; no longer LED40.2 (DOUT)
- net at LED54.4 (DIN): no longer LED67.2 (DOUT)
- net at LED55.2 (DOUT): no longer LED68.4 (DIN)
- net at LED79.2 (DOUT): no longer LED69.4 (DIN)
- net at LED82.4 (DIN): now also C77.1; no longer R3.1
- net at LED81.4 (DIN): no longer LED71.2 (DOUT)
- net at LED80.4 (DIN): no longer LED70.2 (DOUT)
- net at LED25.2 (DOUT): now also C27.1; no longer LED39.4 (DIN)
- net at LED53.2 (DOUT): no longer LED66.4 (DIN)
- net at LED78.4 (DIN): no longer LED66.2 (DOUT)
- new net: D_14.2 (A), K_14.2 (ROW)
- new net: D_15.2 (A), K_15.2 (ROW)
- new net: D_16.2 (A), K_16.2 (ROW)
- new net: D_31.2 (A), K_31.2 (ROW)
- new net: D_32.2 (A), K_32.2 (ROW)
- new net: D_33.2 (A), K_33.2 (ROW)
- new net: D_59.2 (A), K_59.2 (ROW)
- new net: LED27.1 (VDD), LED41.1 (VDD)
- new net: LED28.1 (VDD), LED42.1 (VDD)
- new net: LED29.1 (VDD), LED43.1 (VDD)
- new net: LED29.3 (VSS), LED30.3 (VSS)
- new net: LED30.1 (VDD), LED44.1 (VDD)
- new net: LED31.1 (VDD), LED46.1 (VDD)
- new net: LED31.3 (VSS), LED45.1 (VDD)
- new net: LED42.3 (VSS), LED56.3 (VSS)
- new net: LED43.3 (VSS), LED57.3 (VSS)
- new net: LED44.3 (VSS), LED58.3 (VSS)
- new net: LED45.3 (VSS), LED59.3 (VSS)
- new net: LED56.1 (VDD), LED69.1 (VDD)
- new net: LED57.1 (VDD), LED70.1 (VDD)
- new net: LED59.1 (VDD), LED71.1 (VDD)
- new net: LED26.1 (VDD), LED40.1 (VDD)
- new net: LED25.3 (VSS), LED26.3 (VSS)
- new net: LED40.3 (VSS), LED54.3 (VSS)
- new net: LED54.1 (VDD), LED67.1 (VDD)
- new net: LED55.1 (VDD), LED68.1 (VDD)
- new net: LED41.3 (VSS), LED55.3 (VSS)
- new net: LED69.3 (VSS), LED79.1 (VDD)
- new net: LED79.3 (VSS), LED80.3 (VSS)
- new net: LED67.3 (VSS), LED68.3 (VSS)
- new net: LED71.3 (VSS), LED81.1 (VDD)
- new net: LED70.3 (VSS), LED80.1 (VDD)
- new net: LED25.1 (VDD), LED39.1 (VDD)
- new net: LED39.3 (VSS), LED53.3 (VSS)
- new net: LED53.1 (VDD), LED66.1 (VDD)
- new net: LED66.3 (VSS), LED78.1 (VDD)
- new net: D_68.2 (A), K_68.2 (ROW)
- new net: C?.1, LED?.4 (DIN)
- new net: C?.2, LED?.2 (DOUT), LED?.2 (DOUT)
- new net: LED?.1 (VDD), LED?.3 (VSS)
- new net: C?.1, LED?.4 (DIN), LED?.4 (DIN)
- new net: D_69.2 (A), K_69.2 (ROW)
- new net: D_70.2 (A), K_70.2 (ROW)
- no-connect marks 18 -> 14
Other:
- moved on the sheet: C1, C10, C11, C12, C13, C14, C15, C16, C17, C18, C2, C20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

Commit message: redid entire left side
Parts:
- removed D_14, D_15, D_16, D_31, D_59, D_68, D_69: D, Diode_SMD:D_SOD-123, symbol Device:D_Small
- removed D_14, D_15, D_31, D_59: D, kbd:D3_SMD_v2, symbol Device:D_Small
- removed LED? (x3): YS-SK6812MINI-E, kbd:YS-SK6812MINI-E, symbol kbd:YS-SK6812MINI-E
- added C88, C89, C90, C91, C92, C93, C94, C95: 0.1uF, Capacitor_SMD:C_0603_1608Metric_Pad1.08x0.95mm_HandSolder, symbol Device:C_Small
- added D_14, D_15, D_31, D_59, D_64, D_65, D_66, D_67, D_70, D_71, D_72: D, kbd:D3_SMD_v2, symbol Device:D_Small
- added LED92, LED94, LED95: YS-SK6812MINI-E, kbd:YS-SK6812MINI-E, symbol kbd:YS-SK6812MINI-E
- D_68: renamed from D_32; footprint Diode_SMD:D_SOD-123 -> kbd:D3_SMD_v2
- D_69: renamed from D_33; footprint Diode_SMD:D_SOD-123 -> kbd:D3_SMD_v2
- D_73: renamed from D_70; footprint Diode_SMD:D_SOD-123 -> kbd:D3_SMD_v2
- K_14, K_15, K_16, K_31, K_32, K_33, K_59, K_68, K_69, K_70: footprint MX_Alps_Hybrid:MX-1U-NoLED -> kbd:CherryMX_Hotswap
- gave numbers to parts that had none: 9
Connections:
- net GND: now also C19.1, C23.2, C24.1, C25.2, C26.1, C27.2, C28.2, C29.2, C37.1, C38.2, C39.1, C40.2, C41.1, C42.2, C43.1, C44.1, C50.1, C51.2, C52.1, C53.2, C54.2, C55.1, C56.2, C62.2, C63.1, C64.2, C65.1, C66.2, C67.1, C73.1, C74.1, C75.2, C76.1, C77.1, C9.1, LED11.3 (VSS), LED20.3 (VSS), LED25.3 (VSS), LED26.3 (VSS), LED27.3 (VSS), LED28.3 (VSS), LED29.3 (VSS), LED30.3 (VSS), LED31.3 (VSS), LED39.3 (VSS), LED40.3 (VSS), LED41.1 (VDD), LED42.3 (VSS), LED43.3 (VSS), LED44.3 (VSS), LED45.3 (VSS), LED46.3 (VSS), LED53.3 (VSS), LED54.3 (VSS), LED55.3 (VSS), LED56.3 (VSS), LED57.3 (VSS), LED58.3 (VSS), LED59.3 (VSS), LED66.3 (VSS), LED67.3 (VSS), LED68.3 (VSS), LED69.3 (VSS), LED70.3 (VSS), LED71.3 (VSS), LED78.3 (VSS), LED79.3 (VSS), LED80.3 (VSS), LED81.3 (VSS), LED82.3 (VSS), LED88.3 (VSS), LED89.3 (VSS), LED90.3 (VSS), LED91.3 (VSS), LED93.3 (VSS), C88.1, C89.1, C90.1, C91.1, C92.1, C93.1, C94.1, C95.1, LED92.3 (VSS), LED94.3 (VSS), LED95.3 (VSS)
- net VCC: now also C19.2, C23.1, C24.2, C25.1, C26.2, C27.1, C28.1, C29.1, C37.2, C38.1, C39.2, C40.1, C41.2, C42.1, C43.2, C44.2, C50.2, C51.1, C52.2, C53.1, C54.1, C55.2, C56.1, C62.1, C63.2, C64.1, C65.2, C66.1, C67.2, C73.2, C74.2, C75.1, C76.2, C77.2, C9.2, LED11.1 (VDD), LED20.1 (VDD), LED25.1 (VDD), LED26.1 (VDD), LED27.1 (VDD), LED28.1 (VDD), LED29.1 (VDD), LED30.1 (VDD), LED31.1 (VDD), LED39.1 (VDD), LED40.1 (VDD), LED41.3 (VSS), LED42.1 (VDD), LED43.1 (VDD), LED44.1 (VDD), LED45.1 (VDD), LED46.1 (VDD), LED53.1 (VDD), LED54.1 (VDD), LED55.1 (VDD), LED56.1 (VDD), LED57.1 (VDD), LED58.1 (VDD), LED59.1 (VDD), LED66.1 (VDD), LED67.1 (VDD), LED68.1 (VDD), LED69.1 (VDD), LED70.1 (VDD), LED71.1 (VDD), LED78.1 (VDD), LED79.1 (VDD), LED80.1 (VDD), LED81.1 (VDD), LED82.1 (VDD), LED88.1 (VDD), LED89.1 (VDD), LED90.1 (VDD), LED91.1 (VDD), LED93.1 (VDD), C88.2, C89.2, C90.2, C91.2, C92.2, C93.2, C94.2, C95.2, LED92.1 (VDD), LED94.1 (VDD), LED95.1 (VDD)
- net VDD: no longer C24.2, C25.2, C29.2, C41.2, C42.2, C43.2, C44.1, C54.2, C55.2, C56.2, C66.2, C67.2, C75.2, C76.2, LED29.4 (DIN), LED30.2 (DOUT), LED31.2 (DOUT), LED43.2 (DOUT), LED44.4 (DIN), LED45.2 (DOUT), LED46.4 (DIN), LED57.4 (DIN), LED58.2 (DOUT), LED59.4 (DIN), LED70.2 (DOUT), LED71.2 (DOUT), LED80.2 (DOUT), LED81.2 (DOUT)
- net col0_L: now also U2.20 (A3/PF4); no longer U2.14 (16/PB2)
- net col1_L: now also U2.19 (A2/PF5); no longer U2.15 (14/PB3)
- net col2_L: now also U2.18 (A1/PF6); no longer U2.16 (15/PB1)
- net col4_L: now also U2.16 (15/PB1); no longer U2.18 (A1/PF6)
- net col5_L: now also U2.15 (14/PB3); no longer U2.19 (A2/PF5)
- net col6_L: now also U2.14 (16/PB2); no longer U2.20 (A3/PF4)
- net row0_L: now also D_14.1 (K)
- net row0_R: now also D_64.1 (K), D_65.1 (K), D_66.1 (K)
- net row1_R: now also D_15.1 (K), D_67.1 (K)
- net row2_R: now also D_31.1 (K)
- net row3_R: now also D_70.1 (K)
- net row4_L: now also D_59.1 (K)
- net row4_R: now also D_71.1 (K), D_72.1 (K)
- net at K_14.2 (ROW): now also D_64.2 (A)
- net at K_15.2 (ROW): now also D_65.2 (A)
- net at K_16.2 (ROW): now also D_66.2 (A)
- net at SW_15.2 (ROW): now also D_15.2 (A)
- net at K_31.2 (ROW): now also D_67.2 (A)
- net at SW_31.2 (ROW): now also D_31.2 (A)
- net at K_59.2 (ROW): now also D_70.2 (A)
- net at LED33.4 (DIN): now also LED72.2 (DOUT); no longer LED32.2 (DOUT)
- net at LED34.2 (DOUT): now also LED48.4 (DIN); no longer LED35.4 (DIN)
- net at LED36.2 (DOUT): now also LED50.4 (DIN); no longer LED37.4 (DIN)
- net at LED48.2 (DOUT): now also LED61.4 (DIN); no longer LED47.4 (DIN)
- net at LED49.2 (DOUT): now also LED35.4 (DIN); no longer LED48.4 (DIN)
- net at LED49.4 (DIN): now also LED62.2 (DOUT); no longer LED50.2 (DOUT)
- net at LED51.2 (DOUT): now also LED37.4 (DIN); no longer LED50.4 (DIN)
- net at LED51.4 (DIN): now also LED64.2 (DOUT); no longer LED52.2 (DOUT)
- net at LED61.2 (DOUT): now also LED73.4 (DIN); no longer LED62.4 (DIN)
- net at LED60.2 (DOUT): now also LED83.4 (DIN); no longer LED61.4 (DIN)
- net at LED63.4 (DIN): now also LED50.2 (DOUT); no longer LED62.2 (DOUT)
- net at LED63.2 (DOUT): now also LED75.4 (DIN); no longer LED64.4 (DIN)
- net at LED65.4 (DIN): now also LED52.2 (DOUT); no longer LED64.2 (DOUT)
- net at LED75.2 (DOUT): now also LED76.4 (DIN); no longer LED74.4 (DIN)
- net at LED76.2 (DOUT): now also LED64.4 (DIN); no longer LED75.4 (DIN)
- net at LED77.2 (DOUT): now also LED87.4 (DIN); no longer LED76.4 (DIN)
- net at SW_14.2 (ROW): now also D_14.2 (A)
- net at LED84.2 (DOUT): now also LED72.4 (DIN); no longer LED86.4 (DIN)
- net at LED85.2 (DOUT): now also LED74.4 (DIN); no longer LED87.4 (DIN)
- net at LED73.2 (DOUT): now also LED86.4 (DIN); no longer LED72.4 (DIN)
- net at LED74.2 (DOUT): now also LED62.4 (DIN); no longer LED73.4 (DIN)
- net at LED27.2 (DOUT): now also LED41.2 (DOUT); no longer C26.1
- net at LED28.4 (DIN): now also LED42.2 (DOUT)
- net at LED29.2 (DOUT): now also LED43.4 (DIN)
- net at LED30.4 (DIN): now also LED44.2 (DOUT); no longer C25.1
- net at LED31.4 (DIN), LED46.2 (DOUT): no longer C29.1, C44.2
- net at LED56.4 (DIN): now also LED69.2 (DOUT)
- net at LED57.2 (DOUT): now also LED70.4 (DIN)
- net at LED26.4 (DIN): now also LED40.2 (DOUT); no longer C28.1
- net at LED54.4 (DIN): now also LED67.2 (DOUT)
- net at LED55.2 (DOUT): now also LED68.4 (DIN)
- net at LED79.2 (DOUT): now also LED69.4 (DIN)
- net at LED82.2 (DOUT): now also LED46.4 (DIN); no longer C77.2
- net at LED82.4 (DIN): now also LED93.2 (DOUT); no longer C77.1
- net at LED41.4 (DIN): now also LED55.4 (DIN)
- net at LED71.4 (DIN): now also LED59.2 (DOUT)
- net at LED81.4 (DIN): now also LED71.2 (DOUT)
- net at LED80.4 (DIN): now also LED70.2 (DOUT)
- net at LED25.2 (DOUT): now also LED39.4 (DIN); no longer C27.1
- net at LED53.2 (DOUT): now also LED66.4 (DIN)
- net at LED78.4 (DIN): now also LED66.2 (DOUT)
- net at R3.1: now also LED88.4 (DIN)
- net at K_68.2 (ROW): now also D_71.2 (A)
- net at LED11.2 (DOUT): now also LED89.4 (DIN)
- net at LED11.4 (DIN): now also LED20.2 (DOUT)
- net at LED20.4 (DIN): now also LED90.2 (DOUT)
- net at LED88.2 (DOUT): now also LED91.4 (DIN)
- net at LED89.2 (DOUT): now also LED93.4 (DIN)
- net at LED90.4 (DIN): now also LED92.2 (DOUT)
- net at LED91.2 (DOUT): now also LED95.4 (DIN)
- net at K_69.2 (ROW): now also D_72.2 (A)
- net at SW_59.2 (ROW): now also D_59.2 (A)
- new net: LED32.2 (DOUT), LED47.4 (DIN)
- new net: LED27.4 (DIN), LED28.2 (DOUT)
- new net: LED45.2 (DOUT), LED59.4 (DIN)
- new net: LED31.2 (DOUT), LED45.4 (DIN)
- new net: LED42.4 (DIN), LED56.2 (DOUT)
- new net: LED43.2 (DOUT), LED57.4 (DIN)
- new net: LED44.4 (DIN), LED58.2 (DOUT)
- new net: LED58.4 (DIN), LED81.2 (DOUT)
- new net: LED40.4 (DIN), LED54.2 (DOUT)
- new net: LED79.4 (DIN), LED80.2 (DOUT)
- new net: LED25.4 (DIN), LED26.2 (DOUT)
- new net: LED39.2 (DOUT), LED53.4 (DIN)
- new net: LED67.4 (DIN), LED68.2 (DOUT)
- new net: LED94.4 (DIN), LED95.2 (DOUT)
- new net: LED92.4 (DIN), LED94.2 (DOUT)
- new net: LED29.4 (DIN), LED30.2 (DOUT)
- now unconnected: LED78.2 (DOUT)
- no-connect marks 14 -> 15
Other:
- moved on the sheet: C11, C12, C13, C14, C15, C16, C17, C19, C23, C24, C25, C26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

Commit message: redoing right side, figuring out reset switch WIP
Parts:
- added C100, C101, C96, C97, C98, C99: 0.1uF, Capacitor_SMD:C_0603_1608Metric_Pad1.08x0.95mm_HandSolder, symbol Device:C_Small
- added LED100, LED101, LED96, LED97, LED98, LED99: YS-SK6812MINI-E, kbd:YS-SK6812MINI-E_underglow, symbol kbd:YS-SK6812MINI-E
- RSW1, RSW2: footprint Button_Switch_SMD:SW_SPST_TL3342 -> kbd:ResetSW_1side
Connections:
- net GNDA is gone; now on net GND: C1.2, C11.2, C13.2, C14.2, C15.2, C16.2, C17.2, C2.2, C3.2, C4.2, C5.2, C86.2, J2.B, LED1.3 (VSS), LED13.3 (VSS), LED14.3 (VSS), LED15.3 (VSS), LED16.3 (VSS), LED17.3 (VSS), LED18.3 (VSS), LED2.3 (VSS), LED3.3 (VSS), LED4.3 (VSS), LED5.3 (VSS), LED6.3 (VSS), OL1.4 (GND), RSW1.2, U1.23 (GND), U1.3 (GND), U1.4 (GND)
- net VDD is gone; now on net VCC: C1.1, C11.1, C13.1, C14.1, C15.1, C16.1, C17.1, C2.1, C3.1, C4.1, C5.1, C86.1, J2.A, LED1.1 (VDD), LED13.1 (VDD), LED14.1 (VDD), LED15.1 (VDD), LED16.1 (VDD), LED17.1 (VDD), LED18.1 (VDD), LED2.1 (VDD), LED3.1 (VDD), LED4.1 (VDD), LED5.1 (VDD), LED6.1 (VDD), OL1.3 (VCC), U1.21 (VCC)
- net GND: now also LED41.3 (VSS), C100.2, C96.2, C97.2, C98.2, C99.2, LED100.3 (VSS), LED101.3 (VSS), LED96.3 (VSS), LED97.3 (VSS), LED98.3 (VSS), LED99.3 (VSS); no longer LED41.1 (VDD)
- net VCC: now also LED41.1 (VDD), C100.1, C101.1, C96.1, C97.1, C98.1, C99.1, LED100.1 (VDD), LED101.1 (VDD), LED96.1 (VDD), LED97.1 (VDD), LED98.1 (VDD), LED99.1 (VDD); no longer LED41.3 (VSS)
- net at LED27.2 (DOUT): now also LED41.4 (DIN); no longer LED41.2 (DOUT)
- net at LED55.4 (DIN): now also LED41.2 (DOUT); no longer LED41.4 (DIN)
- net at LED18.4 (DIN): now also LED96.2 (DOUT); no longer R1.2
- net at LED14.2 (DOUT): now also LED97.4 (DIN)
- new net: LED96.4 (DIN), LED99.2 (DOUT)
- new net: LED97.2 (DOUT), LED98.4 (DIN)
- new net: LED101.4 (DIN), LED98.2 (DOUT)
- new net: LED100.2 (DOUT), LED99.4 (DIN)
- new net: LED100.4 (DIN), R1.2
Other:
- moved on the sheet: R1
