File: onigaku.sch (KiCad schematic (older format))
At the start: 360 parts, among them J1 MJ-4PP-9, J2 MJ-4PP-9, U1 Elite-C, U2 Elite-C

Commit message: wiring done, added more leds, figuring out best place for oled
Parts:
- added C102, C103: 0.1uF, Capacitor_SMD:C_0603_1608Metric_Pad1.08x0.95mm_HandSolder, symbol Device:C_Small
- added LED102, LED103: YS-SK6812MINI-E, kbd:YS-SK6812MINI-E_underglow, symbol kbd:YS-SK6812MINI-E
Connections:
- net GND: now also C101.2, C102.2, C103.2, LED102.3 (VSS), LED103.3 (VSS)
- net VCC: now also C102.1, C103.1, LED102.1 (VDD), LED103.1 (VDD)
- net col10_R: now also U1.27 (C7); no longer U1.29 (F0)
- net col8_R: now also U1.29 (F0); no longer U1.27 (C7)
- net at LED7.4 (DIN): now also LED102.2 (DOUT); no longer R2.2
- net at LED19.4 (DIN): now also LED103.2 (DOUT); no longer LED24.2 (DOUT)
- new net: LED102.4 (DIN), R2.2
- new net: LED103.4 (DIN), LED24.2 (DOUT)
Other:
- moved on the sheet: R2
Changed lines of the file:
@@
 L Device:R_Small R2
 U 1 1 604F8078
-P 2675 8250
-F 0 "R2" H 2705 8270 50  0000 L CNN
-F 1 "500" H 2705 8210 50  0000 L CNN
-F 2 "Resistor_SMD:R_0805_2012Metric_Pad1.20x1.40mm_HandSolder" H 2675 8250 50  0001 C CNN
-F 3 "~" H 2675 8250 50  0001 C CNN
-	1    2675 8250
+P 1575 8250
+F 0 "R2" H 1605 8270 50  0000 L CNN
+F 1 "500" H 1605 8210 50  0000 L CNN
+F 2 "Resistor_SMD:R_0805_2012Metric_Pad1.20x1.40mm_HandSolder" H 1575 8250 50  0001 C CNN
+F 3 "~" H 1575 8250 50  0001 C CNN
+	1    1575 8250
 	0    -1   -1   0
 $EndComp
 Wire Wire Line
-	2575 8250 2425 8250
+	1475 8250 1325 8250
 Wire Wire Line
-	2775 8250 2975 8250
+	1675 8250 2225 8250
 Wire Wire Line
 	17100 6350 17350 6350
@@
 L power:GND #PWR020
 U 1 1 604F80D7
-P 2600 8750
-F 0 "#PWR020" H 2600 8500 50  0001 C CNN
-F 1 "GND" H 2600 8600 50  0000 C CNN
-F 2 "" H 2600 8750 50  0001 C CNN
-F 3 "" H 2600 8750 50  0001 C CNN
-	1    2600 8750
+P 1500 8750
+F 0 "#PWR020" H 1500 8500 50  0001 C CNN
+F 1 "GND" H 1500 8600 50  0000 C CNN
+F 2 "" H 1500 8750 50  0001 C CNN
+F 3 "" H 1500 8750 50  0001 C CNN
+	1    1500 8750
 	1    0    0    -1
 $EndComp
 Wire Wire Line
-	2600 8750 2600 8650
+	1500 8750 1500 8650
 Wire Wire Line
 	7750 8650 7750 9350
@@
 	2925 8650 3275 8650
 Wire Wire Line
-	2600 8650 2925 8650
+	1500 8650 2175 8650
 Connection ~ 2925 8650
 Wire Wire Line
@@
 Connection ~ 2925 7950
 Wire Wire Line
-	2675 7950 2925 7950
+	1575 7950 2175 7950
 $Comp
 L Device:C_Small C87
@@
 L power:VCC #PWR0110
 U 1 1 604F805F
-P 2675 7950
-F 0 "#PWR0110" H 2675 7800 50  0001 C CNN
-F 1 "VCC" H 2675 8100 50  0000 C CNN
-F 2 "" H 2675 7950 50  0001 C CNN
-F 3 "" H 2675 7950 50  0001 C CNN
-	1    2675 7950
+P 1575 7950
+F 0 "#PWR0110" H 1575 7800 50  0001 C CNN
+F 1 "VCC" H 1575 8100 50  0000 C CNN
+F 2 "" H 1575 7950 50  0001 C CNN
+F 3 "" H 1575 7950 50  0001 C CNN
+	1    1575 7950
 	0    -1   -1   0
 $EndComp
@@
 Text GLabel 10450 2725 0    50   Input ~ 0
 BACKLIGHT_LED_L
-Text GLabel 2425 8250 0    50   Input ~ 0
+Text GLabel 1325 8250 0    50   Input ~ 0
 BACKLIGHT_LED_L
-NoConn ~ 3775 9050
 $Comp
 L Device:R_Small R4
@@
 	4850 9350 5225 9350
 Wire Wire Line
-	5150 9050 6100 9050
+	5150 9050 5300 9050
 Connection ~ 5225 9350
 Wire Wire Line
-	5225 9350 6400 9350
+	5225 9350 5600 9350
 Wire Wire Line
 	5225 9150 5225 8650
@@
 	25700 5800 22900 5800
 Connection ~ 22900 5800
-Text GLabel 14625 2650 3    50   Input ~ 0
+Text GLabel 14825 2650 3    50   Input ~ 0
 col8_R
 Text GLabel 14725 2650 3    50   Input ~ 0
 col9_R
-Text GLabel 14825 2650 3    50   Input ~ 0
+Text GLabel 14625 2650 3    50   Input ~ 0
 col10_R
 $Comp
@@
 Connection ~ 24000 8500
 Wire Wire Line
-	24000 8500 25175 8500
-Wire Wire Line
 	23625 8500 23625 9000
 Wire Wire Line
@@
 $EndComp
 Wire Wire Line
-	24375 8000 24375 8500
-Wire Wire Line
 	24000 7800 24375 7800
 Connection ~ 24000 7800
@@
 	0    1    1    0
 $EndComp
+Wire Wire Line
+	2525 7950 2925 7950
+Wire Wire Line
+	2525 8550 2525 8650
+Connection ~ 2525 8650
+Wire Wire Line
+	2525 8650 2925 8650
+$Comp
+L kbd:YS-SK6812MINI-E LED102
+U 1 1 603AAEBA
+P 2525 8250
+F 0 "LED102" H 2869 8280 29  0000 L CNN
+F 1 "YS-SK6812MINI-E" H 2869 8221 29  0000 L CNN
+F 2 "kbd:YS-SK6812MINI-E_underglow" H 2625 8000 50  0001 C CNN
+F 3 "" H 2625 8000 50  0001 C CNN
+	1    2525 8250
+	1    0    0    -1
+$EndComp
+Wire Wire Line
+	2175 8650 2525 8650
+Wire Wire Line
+	2175 8150 2175 8650
+Wire Wire Line
+	2175 7950 2525 7950
+$Comp
+L Device:C_Small C102
+U 1 1 603AAEC7
+P 2175 8050
+F 0 "C102" H 2185 8120 50  0000 L CNN
+F 1 "0.1uF" H 2185 7970 50  0000 L CNN
+F 2 "Capacitor_SMD:C_0603_1608Metric_Pad1.08x0.95mm_HandSolder" H 2175 8050 50  0001 C CNN
+F 3 "~" H 2175 8050 50  0001 C CNN
+	1    2175 8050
+	1    0    0    -1
+$EndComp
+Connection ~ 2525 7950
+Wire Wire Line
+	2825 8250 2975 8250
+Connection ~ 2175 7950
+Connection ~ 2175 8650
+$Comp
+L kbd:YS-SK6812MINI-E LED103
+U 1 1 60521656
+P 5600 9050
+F 0 "LED103" H 5944 9080 29  0000 L CNN
+F 1 "YS-SK6812MINI-E" H 5944 9021 29  0000 L CNN
+F 2 "kbd:YS-SK6812MINI-E_underglow" H 5700 8800 50  0001 C CNN
+F 3 "" H 5700 8800 50  0001 C CNN
+	1    5600 9050
+	-1   0    0    1
+$EndComp
+$Comp
+L Device:C_Small C103
+U 1 1 6052165C
+P 6000 9250
+F 0 "C103" H 6010 9320 50  0000 L CNN
+F 1 "0.1uF" H 6010 9170 50  0000 L CNN
+F 2 "Capacitor_SMD:C_0603_1608Metric_Pad1.08x0.95mm_HandSolder" H 6000 9250 50  0001 C CNN
+F 3 "~" H 6000 9250 50  0001 C CNN
+	1    6000 9250
+	-1   0    0    1
+$EndComp
+Wire Wire Line
+	5600 9350 6000 9350
+Connection ~ 6000 9350
+Wire Wire Line
+	6000 9150 6000 8650
+Wire Wire Line
+	6000 9350 6400 9350
+Wire Wire Line
+	5900 9050 6100 9050
+Wire Wire Line
+	3275 8750 3275 8650
+Connection ~ 5600 9350
+Wire Wire Line
+	5600 8750 5600 8650
+NoConn ~ 3775 9050
+Wire Wire Line
+	24000 8500 24375 8500
+Wire Wire Line
+	24375 8000 24375 8500
+Connection ~ 24375 8500
+Wire Wire Line
+	24375 8500 25175 8500
 $EndSCHEMATC

Commit message: wired up and still thinking
Parts:
- removed J1, J2: MJ-4PP-9, kbd:MJ-4PP-9_1side, symbol kbd:MJ-4PP-9
- added J1, J2: MJ-4PP-9, mj-4pp-9:MJ-4PP-9, symbol mj-4pp-9:MJ-4PP-9
- RSW1, RSW2: footprint kbd:ResetSW_1side -> Button_Switch_SMD:SW_SPST_TL3342
Connections:
- net GND: now also J1.2 (B), J2.2 (B)
- net VCC: now also J1.1 (A), J2.1 (A)
- net data_L: now also J2.4 (D)
- net data_R: now also J1.4 (D)
Changed lines of the file:
@@
 L power:GND #PWR015
 U 1 1 604F807D
-P 11325 4075
-F 0 "#PWR015" H 11325 3825 50  0001 C CNN
-F 1 "GND" H 11325 3925 50  0000 C CNN
-F 2 "" H 11325 4075 50  0001 C CNN
-F 3 "" H 11325 4075 50  0001 C CNN
-	1    11325 4075
-	-1   0    0    -1
+P 11625 3775
+F 0 "#PWR015" H 11625 3525 50  0001 C CNN
+F 1 "GND" H 11625 3625 50  0000 C CNN
+F 2 "" H 11625 3775 50  0001 C CNN
+F 3 "" H 11625 3775 50  0001 C CNN
+	1    11625 3775
+	1    0    0    -1
 $EndComp
-Wire Wire Line
-	11325 4075 11325 4025
 $Comp
 L kbd:SW_PUSH RSW2
@@
 F 0 "RSW2" H 10825 3335 50  0000 C CNN
 F 1 "SW_PUSH" H 10675 3145 50  0000 C CNN
-F 2 "kbd:ResetSW_1side" H 10675 3225 50  0001 C CNN
+F 2 "Button_Switch_SMD:SW_SPST_TL3342" H 10675 3225 50  0001 C CNN
 F 3 "" H 10675 3225 50  0000 C CNN
 	1    10675 3225
@@
 F 0 "RSW1" H 14800 3260 50  0000 C CNN
 F 1 "SW_PUSH" H 14650 3070 50  0000 C CNN
-F 2 "kbd:ResetSW_1side" H 14650 3150 50  0001 C CNN
+F 2 "Button_Switch_SMD:SW_SPST_TL3342" H 14650 3150 50  0001 C CNN
 F 3 "" H 14650 3150 50  0000 C CNN
 	1    14650 3150
@@
 Connection ~ 4350 5450
 Wire Wire Line
-	11425 4025 11325 4025
-Wire Wire Line
-	11425 3725 11425 3875
-Wire Wire Line
-	13825 4075 13925 4075
-Wire Wire Line
-	13825 3775 13825 3925
+	14225 4125 14325 4125
 Wire Wire Line
 	3575 8250 3775 8250
@@
 	5150 8250 5300 8250
 $Comp
-L kbd:MJ-4PP-9 J1
-U 1 1 5ACD605D
-P 11625 3975
-F 0 "J1" H 11625 4125 50  0000 C CNN
-F 1 "MJ-4PP-9" H 11625 3825 50  0000 C CNN
-F 2 "kbd:MJ-4PP-9_1side" H 11900 4150 50  0001 C CNN
-F 3 "" H 11900 4150 50  0001 C CNN
-	1    11625 3975
-	-1   0    0    -1
-$EndComp
-$Comp
 L kbd:YS-SK6812MINI-E LED33
 U 1 1 604F8029
@@
 $EndComp
 $Comp
-L kbd:MJ-4PP-9 J2
-U 1 1 604F805B
-P 13625 4025
-F 0 "J2" H 13625 4175 50  0000 C CNN
-F 1 "MJ-4PP-9" H 13625 3875 50  0000 C CNN
-F 2 "kbd:MJ-4PP-9_1side" H 13900 4200 50  0001 C CNN
-F 3 "" H 13900 4200 50  0001 C CNN
-	1    13625 4025
-	1    0    0    -1
-$EndComp
-$Comp
 L kbd:YS-SK6812MINI-E LED60
 U 1 1 60E11226
@@
 Text GLabel 13925 1250 0    50   Input ~ 0
 data_R
-Text GLabel 11425 3925 0    50   Input ~ 0
+Text GLabel 11975 3975 0    50   Input ~ 0
 data_L
 Text GLabel 9950 1325 0    50   Input ~ 0
@@
 NoConn ~ 13925 1150
 NoConn ~ 15325 1150
-Text GLabel 13825 3975 2    50   Input ~ 0
+Text GLabel 14225 3925 2    50   Input ~ 0
 data_R
-NoConn ~ 11425 3975
-NoConn ~ 13825 4025
+NoConn ~ 14225 4025
 $Comp
 L kbd:YS-SK6812MINI-E LED27
@@
 	15100 3150 14950 3150
 Wire Wire Line
-	11350 1525 11800 1525
-Wire Wire Line
-	11425 3725 11800 3725
-Wire Wire Line
-	11800 3725 11800 1525
-Connection ~ 11800 1525
+	11350 1525 11475 1525
+Connection ~ 11475 1525
 Wire Wire Line
-	11800 1525 12150 1525
+	11475 1525 12150 1525
 Wire Wire Line
 	16050 1450 15775 1450
@@
 	15775 1450 15775 3775
 Wire Wire Line
-	13825 3775 15775 3775
+	14225 3775 15775 3775
 Connection ~ 15775 1450
 Wire Wire Line
@@
 Connection ~ 13825 1450
 Wire Wire Line
-	13925 4125 13925 4075
+	14325 4175 14325 4125
 $Comp
 L power:PWR_FLAG #FLG0103
@@
 L power:GND #PWR0108
 U 1 1 6170662B
-P 13925 4125
-F 0 "#PWR0108" H 13925 3875 50  0001 C CNN
-F 1 "GND" H 13925 3975 50  0000 C CNN
-F 2 "" H 13925 4125 50  0001 C CNN
-F 3 "" H 13925 4125 50  0001 C CNN
-	1    13925 4125
+P 14325 4175
+F 0 "#PWR0108" H 14325 3925 50  0001 C CNN
+F 1 "GND" H 14325 4025 50  0000 C CNN
+F 2 "" H 14325 4175 50  0001 C CNN
+F 3 "" H 14325 4175 50  0001 C CNN
+	1    14325 4175
 	1    0    0    -1
 $EndComp
@@
 Wire Wire Line
 	24375 8500 25175 8500
+$Comp
+L mj-4pp-9:MJ-4PP-9 J2
+U 1 1 607CD277
+P 12525 3975
+F 0 "J2" H 12525 4275 50  0000 C CNN
+F 1 "MJ-4PP-9" H 12525 3625 50  0000 C CNN
+F 2 "mj-4pp-9:MJ-4PP-9" H 11925 3875 50  0001 C CNN
+F 3 "" H 11925 3875 50  0001 C CNN
+	1    12525 3975
+	-1   0    0    1
+$EndComp
+Wire Wire Line
+	11475 4125 11975 4125
+NoConn ~ 11975 3875
+Wire Wire Line
+	11475 1525 11475 4125
+Wire Wire Line
+	11625 3775 11975 3775
+$Comp
+L mj-4pp-9:MJ-4PP-9 J1
+U 1 1 60EC7D5C
+P 13675 3925
+F 0 "J1" H 13675 4225 50  0000 C CNN
+F 1 "MJ-4PP-9" H 13675 3575 50  0000 C CNN
+F 2 "mj-4pp-9:MJ-4PP-9" H 13075 3825 50  0001 C CNN
+F 3 "" H 13075 3825 50  0001 C CNN
+	1    13675 3925
+	1    0    0    -1
+$EndComp
 $EndSCHEMATC
