File: onigaku.kicad_pcb (KiCad board)
At the start: 2 copper layers, 355.7 x 103.2 mm, 209 parts, among them J1_L1 MJ-4PP-9, J2_L1 OLED, J3 MJ-4PP-9, J4 OLED, U1 ProMicro, U2 ProMicro

Commit message: continuing WIP
Parts:
- removed D_0, D_64, D_65, D_66, D_67: D, kbd:D3_SMD_v2
- removed the D_11 at (210.6, 10.0)
- removed the D_12 at (229.6, 10.0)
- removed the D_13 at (258.2, 10.0)
- removed the D_15 at (94.2, 86.2)
- removed the D_24 at (160.9, 29.1)
- removed the D_25 at (180.0, 29.1)
- removed the D_26 at (199.0, 29.1)
- removed the D_27 at (218.1, 29.1)
- removed the D_28 at (237.1, 29.1)
- removed the D_40 at (146.6, 48.1)
- removed the D_41 at (165.7, 48.1)
- removed the D_48 at (60.9, 67.2)
- removed the D_52 at (137.1, 67.2)
- removed the D_54 at (175.2, 67.2)
- removed J1_L1: MJ-4PP-9, kbd:MJ-4PP-9_1side
- removed J2_L1, J4: OLED, kbd:OLED_1side
- removed J3: MJ-4PP-9, kbd:MJ-4PP-9
- removed LED0: YS-SK6812MINI-E, kbd:YS-SK6812MINI-E
- removed the RSW2 at (115.9, 164.4)
- removed SW_0: KEYSW, kbd:CherryMX_Hotswap
- removed the SW_24 at (128.6, 66.7)
- removed the SW_37 at (152.4, 28.6)
- removed the SW_38 at (171.4, 28.6)
- removed the SW_39 at (190.5, 28.6)
- removed the SW_40 at (209.6, 28.6)
- removed the SW_41 at (228.6, 28.6)
- removed the SW_48 at (214.3, 47.6)
- removed the SW_49 at (233.4, 47.6)
- removed the SW_50 at (264.3, 47.6)
- removed the SW_51 at (147.6, 66.7)
- removed the SW_52 at (166.7, 66.7)
- removed the SW_59 at (226.2, 85.7)
- removed the SW_60 at (250.0, 85.7)
- removed the SW_61 at (273.8, 85.7)
- added D_16: D, onigaku:D3_SMD_v2, B.Cu at (167.9, 28.6)
- added D_17: D, onigaku:D3_SMD_v2, B.Cu at (186.9, 28.6)
- added D_18: D, onigaku:D3_SMD_v2, B.Cu at (206.0, 28.6)
- added D_19: D, onigaku:D3_SMD_v2, B.Cu at (225.0, 28.6)
- added D_20: D, onigaku:D3_SMD_v2, B.Cu at (244.1, 28.6)
- added D_21: D, onigaku:D3_SMD_v2, B.Cu at (263.1, 28.6)
- added D_22: D, onigaku:D3_SMD_v2, B.Cu at (291.7, 28.6)
- added D_3: D, onigaku:D3_SMD_v2, B.Cu at (201.2, 9.52)
- added D_31: D, onigaku:D3_SMD_v2, B.Cu at (212.5, 48.1)
- added D_32: D, onigaku:D3_SMD_v2, B.Cu at (231.6, 48.1)
- added D_33: D, onigaku:D3_SMD_v2, B.Cu at (250.6, 48.1)
- added D_34: D, onigaku:D3_SMD_v2, B.Cu at (269.7, 48.1)
- added D_35: D, onigaku:D3_SMD_v2, B.Cu at (312.5, 48.1)
- added D_4: D, onigaku:D3_SMD_v2, B.Cu at (220.2, 9.53)
- added D_47: D, onigaku:D3_SMD_v2, B.Cu at (279.5, 66.7)
- added D_49: D, onigaku:D3_SMD_v2, B.Cu at (44.8, 66.7)
- added D_5: D, onigaku:D3_SMD_v2, B.Cu at (239.2, 9.53)
- added D_6: D, onigaku:D3_SMD_v2, B.Cu at (258.3, 9.52)
- added D_60: D, onigaku:D3_SMD_v2, B.Cu at (27.9, 85.7)
- added J1: MJ-4PP-9, onigaku:MJ-4PP-9_1side, F.Cu at (332.2, 154.9)
- added J2: MJ-4PP-9, onigaku:MJ-4PP-9, F.Cu at (369.9, 116.6)
- added LED75: YS-SK6812MINI-E, onigaku:YS-SK6812MINI-E, F.Cu at (402.6, 156.8)
- added LED76: YS-SK6812MINI-E, onigaku:YS-SK6812MINI-E, F.Cu at (413.6, 147.2)
- added LED77: YS-SK6812MINI-E, onigaku:YS-SK6812MINI-E, F.Cu at (422.6, 137.6)
- added LED78: YS-SK6812MINI-E, onigaku:YS-SK6812MINI-E, F.Cu at (395.7, 166.5)
- added LED79: YS-SK6812MINI-E, onigaku:YS-SK6812MINI-E, F.Cu at (404.6, 161.7)
- added RSW1: SW_PUSH, onigaku:ResetSW, F.Cu at (369.3, 132.5)
- added SW_1: KEYSW, onigaku:CherryMX_Hotswap, F.Cu at (170.7, 9.53)
- added SW_16: KEYSW, onigaku:CherryMX_Hotswap, F.Cu at (180.2, 28.6)
- added SW_17: KEYSW, onigaku:CherryMX_Hotswap, F.Cu at (199.2, 28.6)
- added SW_18: KEYSW, onigaku:CherryMX_Hotswap, F.Cu at (218.3, 28.6)
- added SW_19: KEYSW, onigaku:CherryMX_Hotswap, F.Cu at (237.3, 28.6)
- added SW_2: KEYSW, onigaku:CherryMX_Hotswap, F.Cu at (189.7, 9.53)
- added SW_20: KEYSW, onigaku:CherryMX_Hotswap, F.Cu at (256.4, 28.6)
- added SW_21: KEYSW, onigaku:CherryMX_Hotswap, F.Cu at (275.4, 28.6)
- added SW_22: KEYSW, onigaku:CherryMX_Hotswap, F.Cu at (299.2, 28.6)
- added SW_3: KEYSW, onigaku:CherryMX_Hotswap, F.Cu at (208.8, 9.53)
- added SW_4: KEYSW, onigaku:CherryMX_Hotswap, F.Cu at (227.8, 9.53)
- added SW_5: KEYSW, onigaku:CherryMX_Hotswap, F.Cu at (246.9, 9.53)
- added SW_6: KEYSW, onigaku:CherryMX_Hotswap, F.Cu at (265.9, 9.53)
- added SW_7: KEYSW, onigaku:CherryMX_Hotswap, F.Cu at (294.5, 9.53)
- added SW_8: KEYSW, onigaku:CherryMX_Hotswap, F.Cu at (9.53, 9.53)
- D_1, D_10, D_2, D_29, D_30, D_42, D_43, D_44, D_45, D_46, D_53, D_55, D_56, D_57, D_58, D_61, D_62, D_63, D_7, D_8, D_9: footprint kbd:D3_SMD_v2 -> onigaku:D3_SMD_v2
- D_11: renamed from D_3; footprint kbd:D3_SMD_v2 -> onigaku:D3_SMD_v2
- D_12: renamed from D_4; footprint kbd:D3_SMD_v2 -> onigaku:D3_SMD_v2
- D_13: renamed from D_5; footprint kbd:D3_SMD_v2 -> onigaku:D3_SMD_v2
- D_14: renamed from D_6; footprint kbd:D3_SMD_v2 -> onigaku:D3_SMD_v2
- D_15: renamed from D_23; footprint kbd:D3_SMD_v2 -> onigaku:D3_SMD_v2
- D_23: renamed from D_17; footprint kbd:D3_SMD_v2 -> onigaku:D3_SMD_v2
- D_24: renamed from D_18; footprint kbd:D3_SMD_v2 -> onigaku:D3_SMD_v2
- D_25: renamed from D_19; footprint kbd:D3_SMD_v2 -> onigaku:D3_SMD_v2
- D_26: renamed from D_20; footprint kbd:D3_SMD_v2 -> onigaku:D3_SMD_v2
- D_27: renamed from D_21; footprint kbd:D3_SMD_v2 -> onigaku:D3_SMD_v2
- D_28: renamed from D_22; footprint kbd:D3_SMD_v2 -> onigaku:D3_SMD_v2
- D_36: renamed from D_34; footprint kbd:D3_SMD_v2 -> onigaku:D3_SMD_v2
- D_37: renamed from D_35; footprint kbd:D3_SMD_v2 -> onigaku:D3_SMD_v2
- D_38: renamed from D_36; footprint kbd:D3_SMD_v2 -> onigaku:D3_SMD_v2
- D_39: renamed from D_37; footprint kbd:D3_SMD_v2 -> onigaku:D3_SMD_v2
- D_40: renamed from D_38; footprint kbd:D3_SMD_v2 -> onigaku:D3_SMD_v2
- D_41: renamed from D_39; footprint kbd:D3_SMD_v2 -> onigaku:D3_SMD_v2
- D_48: renamed from D_47; footprint kbd:D3_SMD_v2 -> onigaku:D3_SMD_v2
- D_50: renamed from D_49; footprint kbd:D3_SMD_v2 -> onigaku:D3_SMD_v2
- D_51: renamed from D_50; footprint kbd:D3_SMD_v2 -> onigaku:D3_SMD_v2
- D_52: renamed from D_51; footprint kbd:D3_SMD_v2 -> onigaku:D3_SMD_v2
- D_54: renamed from D_14; footprint kbd:D3_SMD_v2 -> onigaku:D3_SMD_v2
- D_59: renamed from D_60; footprint kbd:D3_SMD_v2 -> onigaku:D3_SMD_v2
- LED1, LED10, LED11, LED12, LED13, LED2, LED20, LED21, LED22, LED23, LED24, LED25, LED26, LED27, LED28, LED29, LED3, LED30, LED31, LED32, LED33, LED34, LED35, LED36, LED37, LED38, LED39, LED4, LED40, LED41, LED42, LED43, LED44, LED45, LED46, LED48, LED49, LED5, LED50, LED51, LED52, LED53, LED54, LED55, LED56, LED57, LED58, LED59, LED6, LED60, LED61, LED62, LED63, LED64, LED65, LED66, LED67, LED7, LED73, LED74, LED8, LED9: footprint kbd:YS-SK6812MINI-E -> onigaku:YS-SK6812MINI-E
- LED14, LED15, LED16, LED17, LED18, LED19, LED47, LED68, LED69, LED70, LED71, LED72: value WS2812B -> YS-SK6812MINI-E; footprint kbd:LED_WS2812B-PLCC4 -> onigaku:YS-SK6812MINI-E
- RSW2: renamed from RSW1; footprint kbd:ResetSW_1side -> onigaku:ResetSW_1side
- SW_10: renamed from SW_2; footprint kbd:CherryMX_Hotswap -> onigaku:CherryMX_Hotswap
- SW_11: renamed from SW_3; footprint kbd:CherryMX_Hotswap -> onigaku:CherryMX_Hotswap
- SW_12: renamed from SW_4; footprint kbd:CherryMX_Hotswap -> onigaku:CherryMX_Hotswap
- SW_13: renamed from SW_5; footprint kbd:CherryMX_Hotswap -> onigaku:CherryMX_Hotswap
- SW_14: renamed from SW_6; footprint kbd:CherryMX_Hotswap -> onigaku:CherryMX_Hotswap
- SW_15: renamed from SW_36; footprint kbd:CherryMX_Hotswap -> onigaku:CherryMX_Hotswap
- SW_23: renamed from SW_7; footprint kbd:CherryMX_Hotswap_1.5u -> onigaku:CherryMX_Hotswap
- SW_24: renamed from SW_8; footprint kbd:CherryMX_Hotswap -> onigaku:CherryMX_Hotswap
- SW_25: renamed from SW_9; footprint kbd:CherryMX_Hotswap -> onigaku:CherryMX_Hotswap
- SW_26: renamed from SW_10; footprint kbd:CherryMX_Hotswap -> onigaku:CherryMX_Hotswap
- SW_27: renamed from SW_11; footprint kbd:CherryMX_Hotswap -> onigaku:CherryMX_Hotswap
- SW_28: renamed from SW_12; footprint kbd:CherryMX_Hotswap -> onigaku:CherryMX_Hotswap
- SW_29, SW_30, SW_31, SW_32, SW_33, SW_34, SW_35, SW_42, SW_44, SW_45, SW_46, SW_53: footprint kbd:CherryMX_Hotswap -> onigaku:CherryMX_Hotswap
- SW_37: renamed from SW_14; footprint kbd:CherryMX_Hotswap -> onigaku:CherryMX_Hotswap
- SW_38: renamed from SW_15; footprint kbd:CherryMX_Hotswap -> onigaku:CherryMX_Hotswap
- SW_39: renamed from SW_16; footprint kbd:CherryMX_Hotswap -> onigaku:CherryMX_Hotswap
- SW_40: renamed from SW_17; footprint kbd:CherryMX_Hotswap -> onigaku:CherryMX_Hotswap
- SW_41: renamed from SW_18; footprint kbd:CherryMX_Hotswap -> onigaku:CherryMX_Hotswap
- SW_43: footprint kbd:CherryMX_Hotswap_1.5u -> onigaku:CherryMX_Hotswap
- SW_47, SW_54: footprint kbd:CherryMX_Hotswap -> onigaku:CherryMX_Hotswap_2.75u_North
- SW_48: renamed from SW_19; footprint kbd:CherryMX_Hotswap_2.25u_North -> onigaku:CherryMX_Hotswap_2.25u_North
- SW_49: renamed from SW_20; footprint kbd:CherryMX_Hotswap -> onigaku:CherryMX_Hotswap
- SW_50: renamed from SW_21; footprint kbd:CherryMX_Hotswap -> onigaku:CherryMX_Hotswap
- SW_51: renamed from SW_22; footprint kbd:CherryMX_Hotswap -> onigaku:CherryMX_Hotswap
- SW_52: renamed from SW_23; footprint kbd:CherryMX_Hotswap -> onigaku:CherryMX_Hotswap
- SW_55: footprint kbd:CherryMX_Hotswap -> onigaku:CherryMX_Hotswap_1.25u_North
- SW_56, SW_57: footprint kbd:CherryMX_Hotswap_2.75u_North -> onigaku:CherryMX_Hotswap_1.25u_North
- SW_58: footprint kbd:CherryMX_Hotswap_1.25u_North -> onigaku:CherryMX_Hotswap_1.25u_North
- SW_59: renamed from SW_25; footprint kbd:CherryMX_Hotswap_1.25u_North -> onigaku:CherryMX_Hotswap_1.25u_North
- SW_60: renamed from SW_26; footprint kbd:CherryMX_Hotswap_1.25u_North -> onigaku:CherryMX_Hotswap_1.25u_North
- SW_61: renamed from SW_62; footprint kbd:CherryMX_Hotswap_1.25u_North -> onigaku:CherryMX_Hotswap_1.25u_North
- SW_62: renamed from SW_27; footprint kbd:CherryMX_Hotswap_1.25u_North -> onigaku:CherryMX_Hotswap_1.25u_North
- SW_63: renamed from SW_28; footprint kbd:CherryMX_Hotswap_2.25u_North -> onigaku:CherryMX_Hotswap_2.25u_North
- SW_9: renamed from SW_1; footprint kbd:CherryMX_Hotswap -> onigaku:CherryMX_Hotswap
- SW_e: renamed from SW_13; footprint kbd:CherryMX_Hotswap_1.75u -> onigaku:CherryMX_Hotswap
- U1, U2: value ProMicro -> elite-c; footprint kbd:ProMicro_v3 -> keebio:Elite-C
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Connections:
- D_1 pad 1: row0_L -> row0_R
- D_10 pad 1: row0_R -> row0_L
- D_2 pad 1: row0_L -> row0_R
- D_29 pad 1: row1_R -> row2_R
- D_30 pad 1: row1_R -> row2_R
- D_42 pad 1: row2_R -> row3_R
- D_43 pad 1: row2_R -> row3_R
- D_44 pad 1: row2_R -> row3_R
- D_45 pad 1: row2_R -> row3_R
- D_46 pad 1: row2_R -> row3_R
- D_53 pad 1: row3_R -> row3_L
- D_54 pad 2: Net-(D_14-Pad2) (its old number) -> Net-(D_54-Pad2)
- D_55 pad 1: row3_R -> col0_R
- D_56 pad 1: row3_R -> col0_R
- D_57 pad 1: row3_R -> col0_R
- D_58 pad 1: row3_R -> col0_R
- D_8 pad 1: row0_R -> row0_L
- D_9 pad 1: row0_R -> row0_L
- LED1 pad 2: Net-(LED0-Pad4) -> Net-(LED1-Pad2)
- LED1 pad 3: GND -> VCC
- LED1 pad 4: Net-(LED1-Pad4) -> BACKLIGHT_LED_R
- LED10 pad 3: GND -> VCC
- LED11 pad 2: Net-(LED11-Pad2) -> Net-(LED10-Pad4)
- LED11 pad 3: GND -> VCC
- LED11 pad 4: Net-(LED10-Pad2) -> Net-(LED11-Pad4)
- LED12 pad 2: Net-(LED12-Pad2) -> Net-(LED11-Pad4)
- LED12 pad 3: GND -> VCC
- LED13 pad 3: GND -> VCC
- LED14 pad 3: GND -> VCC
- LED15 pad 3: GND -> VCC
- LED16 pad 3: GND -> VCC
- LED16 pad 4: LED_L -> Net-(LED16-Pad4)
- LED17 pad 1: GND -> VCC
- LED17 pad 4: LED_R -> Net-(LED17-Pad4)
- LED18 pad 1: GND -> VCC
- LED18 pad 2: Net-(LED18-Pad2) -> Net-(LED17-Pad4)
- LED18 pad 4: Net-(LED17-Pad2) -> Net-(LED18-Pad4)
- LED19 pad 1: GND -> VCC
- LED19 pad 4: Net-(LED18-Pad2) -> Net-(LED19-Pad4)
- LED2 pad 3: GND -> VCC
- LED2 pad 4: Net-(LED2-Pad4) -> Net-(LED1-Pad2)
- LED20 pad 1: GND -> VCC
- LED20 pad 2: Net-(LED13-Pad4) -> Net-(LED19-Pad4)
- LED21 pad 1: GND -> VCC
- LED21 pad 4: Net-(LED12-Pad2) -> Net-(LED21-Pad4)
- LED22 pad 1: GND -> VCC
- LED22 pad 2: Net-(LED12-Pad4) -> Net-(LED21-Pad4)
- LED23 pad 1: GND -> VCC
- LED23 pad 3: GND -> Net-(LED23-Pad3)
- LED23 pad 4: Net-(LED11-Pad2) -> Net-(LED23-Pad4)
- LED24 pad 1: GND -> VCC
- LED24 pad 2: Net-(LED10-Pad4) -> Net-(LED24-Pad2)
- LED25 pad 1: GND -> VCC
- LED26 pad 1: GND -> VCC
- LED26 pad 2: Net-(LED26-Pad2) -> Net-(LED25-Pad4)
- LED27 pad 1: GND -> VCC
- LED28 pad 1: GND -> VCC
- LED28 pad 2: Net-(LED28-Pad2) -> Net-(LED27-Pad4)
- LED29 pad 1: GND -> VCC
- LED3 pad 2: Net-(LED2-Pad4) -> Net-(LED3-Pad2)
- LED3 pad 3: GND -> VCC
- LED3 pad 4: Net-(LED3-Pad4) -> Net-(LED2-Pad2)
- LED30 pad 1: GND -> VCC
- LED30 pad 2: Net-(LED30-Pad2) -> Net-(LED29-Pad4)
- LED30 pad 3: GND -> Net-(LED30-Pad3)
- LED31 pad 1: GND -> VCC
- LED31 pad 2: Net-(LED3-Pad4) -> Net-(LED31-Pad2)
- LED31 pad 4: Net-(LED31-Pad4) -> Net-(LED17-Pad2)
- LED32 pad 1: GND -> VCC
- LED32 pad 2: Net-(LED32-Pad2) -> Net-(LED18-Pad4)
- LED32 pad 3: Net-(LED32-Pad3) -> GND
- LED32 pad 4: Net-(LED2-Pad2) -> Net-(LED32-Pad4)
- LED33 pad 1: GND -> Net-(LED33-Pad1)
- LED33 pad 3: GND -> Net-(LED33-Pad3)
- LED33 pad 4: Net-(LED0-Pad2) -> Net-(LED19-Pad2)
- LED34 pad 1: GND -> VCC
- LED34 pad 2: Net-(LED34-Pad2) -> Net-(LED20-Pad4)
- LED34 pad 4: Net-(LED33-Pad2) -> Net-(LED34-Pad4)
- LED35 pad 1: GND -> VCC
- LED35 pad 2: Net-(LED1-Pad4) -> Net-(LED35-Pad2)
- LED35 pad 4: Net-(LED35-Pad4) -> Net-(LED21-Pad2)
- LED36 pad 1: GND -> VCC
- LED36 pad 2: Net-(LED36-Pad2) -> Net-(LED22-Pad4)
- LED36 pad 4: Net-(LED32-Pad2) -> Net-(LED36-Pad4)
- LED37 pad 1: GND -> VCC
- LED37 pad 2: Net-(LED31-Pad4) -> Net-(LED37-Pad2)
- LED37 pad 4: Net-(LED37-Pad4) -> Net-(LED23-Pad2)
- LED38 pad 1: GND -> VCC
- LED38 pad 2: Net-(LED38-Pad2) -> Net-(LED23-Pad4)
- LED38 pad 3: GND -> Net-(LED23-Pad3)
- LED38 pad 4: Net-(LED30-Pad2) -> Net-(LED38-Pad4)
- LED39 pad 1: GND -> VCC
- LED39 pad 2: Net-(LED29-Pad4) -> Net-(LED24-Pad4)
- LED4 pad 2: Net-(LED30-Pad4) -> Net-(LED12-Pad4)
- LED4 pad 3: GND -> VCC
- LED4 pad 4: Net-(LED4-Pad4) -> Net-(LED3-Pad2)
- LED40 pad 1: GND -> VCC
- LED40 pad 2: Net-(LED40-Pad2) -> Net-(LED26-Pad4)
- LED40 pad 4: Net-(LED28-Pad2) -> Net-(LED40-Pad4)
- LED41 pad 1: GND -> VCC
- LED42 pad 1: GND -> VCC
- LED42 pad 2: Net-(LED42-Pad2) -> Net-(LED28-Pad4)
- LED42 pad 4: Net-(LED25-Pad2) -> Net-(LED42-Pad4)
- LED43 pad 1: GND -> VCC
- LED43 pad 2: Net-(LED24-Pad4) -> Net-(LED43-Pad2)
- LED43 pad 4: Net-(LED43-Pad4) -> Net-(LED29-Pad2)
- LED44 pad 1: GND -> VCC
- LED44 pad 2: Net-(LED44-Pad2) -> Net-(LED30-Pad4)
- LED44 pad 3: GND -> Net-(LED30-Pad3)
- LED44 pad 4: Net-(LED23-Pad2) -> Net-(LED44-Pad4)
- LED45 pad 1: GND -> VCC
- LED45 pad 2: Net-(LED22-Pad4) -> Net-(LED45-Pad2)
- LED45 pad 4: Net-(LED45-Pad4) -> Net-(LED31-Pad2)
- LED46 pad 1: Net-(LED46-Pad1) -> VCC
- LED46 pad 2: Net-(LED46-Pad2) -> Net-(LED32-Pad4)
- LED46 pad 4: Net-(LED21-Pad2) -> Net-(LED46-Pad4)
- LED47 pad 1: GND -> VCC
- LED47 pad 4: Net-(LED14-Pad2) -> Net-(LED33-Pad2)
- LED48 pad 1: Net-(LED48-Pad1) -> VCC
- LED48 pad 2: Net-(LED48-Pad2) -> Net-(LED34-Pad4)
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Other:
- board size 355.7 x 103.2 mm -> 383.4 x 103.2 mm
- rule pad_to_mask_clearance: 0 -> 0.2

Commit message: lined up rgb leds, WIP on adding bypass capacitors
Parts:
- added LED80: YS-SK6812MINI-E, kbd:YS-SK6812MINI-E_underglow, F.Cu at (400.4, 140.5)
- added LED81: YS-SK6812MINI-E, kbd:YS-SK6812MINI-E_underglow, F.Cu at (274.2, 140.5)
- added LED82: YS-SK6812MINI-E, kbd:YS-SK6812MINI-E_underglow, F.Cu at (170.2, 140.5)
- added LED83: YS-SK6812MINI-E, kbd:YS-SK6812MINI-E_underglow, F.Cu at (127.4, 140.5)
- added LED84: YS-SK6812MINI-E, kbd:YS-SK6812MINI-E_underglow, F.Cu at (360.0, 178.4)
- added LED85: YS-SK6812MINI-E, kbd:YS-SK6812MINI-E_underglow, F.Cu at (388.5, 178.6)
- added LED86: YS-SK6812MINI-E, kbd:YS-SK6812MINI-E_underglow, F.Cu at (170.2, 178.6)
- added LED87: YS-SK6812MINI-E, kbd:YS-SK6812MINI-E_underglow, F.Cu at (122.7, 178.6)
- added OL1: OLED, kbd:OLED_v2, F.Cu at (296.7, 95.8)
- added OL2: OLED, kbd:OLED_v2, F.Cu at (195.5, 95.8)
- added R1: 500, Resistor_SMD:R_0805_2012Metric_Pad1.20x1.40mm_HandSolder, B.Cu at (269.6, 120.7)
- added R2: 500, Resistor_SMD:R_0805_2012Metric_Pad1.20x1.40mm_HandSolder, B.Cu at (109.9, 120.3)
- D_1, D_10, D_11, D_12, D_13, D_14, D_15, D_16, D_17, D_18, D_19, D_2, D_20, D_21, D_22, D_23, D_24, D_25, D_26, D_27, D_28, D_29, D_3, D_30, D_31, D_32, D_33, D_34, D_35, D_36, D_37, D_38, D_39, D_4, D_40, D_41, D_42, D_43, D_44, D_45, D_46, D_47, D_48, D_49, D_5, D_50, D_51, D_52, D_53, D_55, D_56, D_57, D_58, D_59, D_6, D_60, D_61, D_62, D_63, D_7, D_8, D_9: footprint onigaku:D3_SMD_v2 -> kbd:D3_SMD_v2
- D_54: footprint onigaku:D3_SMD_v2 -> kbd:D3_SMD_v2; moved to B.Cu
- J1: footprint onigaku:MJ-4PP-9_1side -> kbd:MJ-4PP-9_1side; moved to B.Cu
- J2: footprint onigaku:MJ-4PP-9 -> kbd:MJ-4PP-9_1side; moved to B.Cu
- LED1, LED10, LED11, LED12, LED13, LED14, LED15, LED16, LED2, LED3, LED4, LED5, LED6, LED7, LED8, LED9: footprint onigaku:YS-SK6812MINI-E -> kbd:YS-SK6812MINI-E_underglow
- LED17, LED18, LED19, LED20, LED21, LED22, LED23, LED24, LED25, LED26, LED27, LED28, LED29, LED30, LED31, LED32, LED33, LED34, LED35, LED36, LED37, LED38, LED39, LED40, LED41, LED42, LED43, LED44, LED45, LED46, LED47, LED48, LED49, LED50, LED51, LED52, LED53, LED54, LED55, LED56, LED57, LED58, LED59, LED60, LED61, LED62, LED63, LED64, LED65, LED66, LED67, LED68, LED69, LED70, LED71, LED72, LED73, LED74, LED75, LED76, LED77, LED78, LED79: footprint onigaku:YS-SK6812MINI-E -> kbd:YS-SK6812MINI-E; moved to B.Cu
- RSW1: footprint onigaku:ResetSW -> Button_Switch_SMD:SW_SPST_TL3342
- RSW2: footprint onigaku:ResetSW_1side -> Button_Switch_SMD:SW_SPST_TL3342
- SW_1, SW_10, SW_11, SW_12, SW_13, SW_14, SW_15, SW_16, SW_17, SW_18, SW_19, SW_2, SW_20, SW_21, SW_24, SW_25, SW_26, SW_27, SW_28, SW_29, SW_3, SW_30, SW_31, SW_32, SW_33, SW_34, SW_37, SW_38, SW_39, SW_4, SW_40, SW_41, SW_42, SW_43, SW_44, SW_45, SW_46, SW_49, SW_5, SW_50, SW_51, SW_52, SW_53, SW_6, SW_8, SW_9: footprint onigaku:CherryMX_Hotswap -> kbd:CherryMX_Hotswap
- SW_22, SW_23: footprint onigaku:CherryMX_Hotswap -> kbd:CherryMX_Hotswap_1.5u
- SW_35: footprint onigaku:CherryMX_Hotswap -> kbd:CherryMX_Hotswap_2.25u_North
- SW_36: renamed from SW_e; footprint onigaku:CherryMX_Hotswap -> kbd:CherryMX_Hotswap_1.75u
- SW_47, SW_54: footprint onigaku:CherryMX_Hotswap_2.75u_North -> kbd:CherryMX_Hotswap_2.75u_North
- SW_48, SW_63: footprint onigaku:CherryMX_Hotswap_2.25u_North -> kbd:CherryMX_Hotswap_2.25u_North
- SW_55, SW_56, SW_57, SW_58, SW_59, SW_60, SW_61, SW_62: footprint onigaku:CherryMX_Hotswap_1.25u_North -> kbd:CherryMX_Hotswap_1.25u_North
- SW_7: footprint onigaku:CherryMX_Hotswap -> kbd:CherryMX_Hotswap_2u_North
- U1, U2: value elite-c -> Elite-C
- moved LED52 299.4 mm to (115.4, 145.3)
- moved LED75 293.2 mm to (110.6, 183.4)
- moved LED53 282.2 mm to (141.6, 145.3)
- moved LED76 281.5 mm to (134.5, 183.4)
- moved LED24 280.3 mm to (108.3, 107.2)
- moved LED39 274.3 mm to (113.0, 126.2)
- moved LED65 274.3 mm to (151.3, 164.3)
- moved LED77 268.3 mm to (158.2, 183.4)
- moved U1 260.0 mm to (89.3, 107.4), turned to 270 degrees
- moved LED41 258.2 mm to (156.0, 126.2)
- moved LED64 257.6 mm to (120.3, 164.3)
- moved LED13 254.8 mm to (125.1, 159.4)
- moved LED54 254.2 mm to (160.7, 145.3)
- moved LED40 242.6 mm to (136.8, 126.2)
- moved LED5 242.1 mm to (127.5, 121.2)
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Connections:
- D_54 pad 1: col0_R -> row4_R
- D_55 pad 1: col0_R -> row4_R
- D_56 pad 1: col0_R -> row4_R
- D_57 pad 1: col0_R -> row4_R
- D_58 pad 1: col0_R -> row4_R
- LED1 pad 1: GND -> VCC
- LED1 pad 3: VCC -> GND
- LED1 pad 4: BACKLIGHT_LED_R -> Net-(LED1-Pad4)
- LED10 pad 1: GND -> VCC
- LED10 pad 3: VCC -> GND
- LED11 pad 1: GND -> VCC
- LED11 pad 3: VCC -> GND
- LED12 pad 1: GND -> VCC
- LED12 pad 3: VCC -> GND
- LED13 pad 1: GND -> VCC
- LED13 pad 3: VCC -> GND
- LED14 pad 1: GND -> VCC
- LED14 pad 3: VCC -> GND
- LED15 pad 1: GND -> VCC
- LED15 pad 3: VCC -> GND
- LED16 pad 1: GND -> VCC
- LED16 pad 3: VCC -> GND
- LED2 pad 1: GND -> VCC
- LED2 pad 3: VCC -> GND
- LED3 pad 1: GND -> VCC
- LED3 pad 3: VCC -> GND
- LED4 pad 1: GND -> VCC
- LED4 pad 2: Net-(LED12-Pad4) -> Net-(LED4-Pad2)
- LED4 pad 3: VCC -> GND
- LED5 pad 1: GND -> VCC
- LED5 pad 3: VCC -> GND
- LED5 pad 4: BACKLIGHT_LED_L -> Net-(LED5-Pad4)
- LED6 pad 1: GND -> VCC
- LED6 pad 3: VCC -> GND
- LED7 pad 1: GND -> VCC
- LED7 pad 3: VCC -> GND
- LED8 pad 1: GND -> VCC
- LED8 pad 2: Net-(LED16-Pad4) -> Net-(LED8-Pad2)
- LED8 pad 3: VCC -> GND
- LED9 pad 1: GND -> VCC
- LED9 pad 3: VCC -> GND
- LED9 pad 4: Net-(LED9-Pad4) -> Net-(LED10-Pad2)
- SW_54 pad 1: Net-(SW_54-Pad1) -> col0_R
- U1 pad 1: Net-(U1-Pad1) -> data_L
- U1 pad 10: row3_L -> row4_L
- U1 pad 11: row4_L -> Net-(U1-Pad11)
- U1 pad 14: col6_L -> Net-(U1-Pad14)
- U1 pad 15: col5_L -> col6_L
- U1 pad 16: col4_L -> col5_L
- U1 pad 17: col3_L -> col4_L
- U1 pad 18: col2_L -> col3_L
- U1 pad 19: col1_L -> col2_L
- U1 pad 2: data_L -> GND
- U1 pad 20: col0_L -> col1_L
- U1 pad 21: VCC -> col0_L
- U1 pad 22: reset_L -> VCC
- U1 pad 23: GND -> reset_L
- U1 pad 24: Net-(U1-Pad24) -> GND
- U1 pad 25: (no net) -> Net-(U1-Pad25)
- U1 pad 26: (no net) -> Net-(U1-Pad26)
- U1 pad 27: (no net) -> Net-(U1-Pad27)
- U1 pad 28: (no net) -> Net-(U1-Pad28)
- U1 pad 29: (no net) -> Net-(U1-Pad29)
- U1 pad 4: GND -> SDA_L
- U1 pad 5: Net-(U1-Pad5) -> SCL_L
- U1 pad 6: Net-(U1-Pad6) -> row0_L
- U1 pad 7: row0_L -> row1_L
- U1 pad 8: row1_L -> row2_L
- U1 pad 9: row2_L -> row3_L
- U2 pad 1: Net-(U2-Pad1) -> data_R
- U2 pad 10: row3_R -> row4_R
- U2 pad 11: col0_R -> Net-(U2-Pad11)
- U2 pad 13: col7_R -> Net-(U2-Pad13)
- U2 pad 14: col6_R -> col7_R
- U2 pad 15: col5_R -> col6_R
- U2 pad 16: col4_R -> col5_R
- U2 pad 17: col3_R -> col4_R
- U2 pad 18: col2_R -> col3_R
- U2 pad 19: col1_R -> col2_R
- U2 pad 2: data_R -> GND
- U2 pad 20: col0_R -> col1_R
- U2 pad 21: VCC -> col0_R
- U2 pad 22: reset_R -> VCC
- U2 pad 23: GND -> reset_R
- U2 pad 24: Net-(U2-Pad24) -> GND
- U2 pad 25: (no net) -> Net-(U2-Pad25)
- U2 pad 26: (no net) -> Net-(U2-Pad26)
- U2 pad 27: (no net) -> Net-(U2-Pad27)
- U2 pad 28: (no net) -> Net-(U2-Pad28)
- U2 pad 29: (no net) -> Net-(U2-Pad29)
- U2 pad 4: GND -> SDA_R
- U2 pad 5: Net-(U2-Pad5) -> SCL_R
- U2 pad 6: Net-(U2-Pad6) -> row0_R
- U2 pad 7: row0_R -> row1_R
- U2 pad 8: row1_R -> row2_R
- U2 pad 9: row2_R -> row3_R
Other:
- board size 383.4 x 103.2 mm -> 351.3 x 110.1 mm
- net class Default: trace_width 0.25 -> 0.254
- net class Power added: clearance 0.2, trace_width 0.381, via_dia 0.8, via_drill 0.4

Commit message: rearranged leds, moved caps, adjusting size of keyboard
Parts:
- removed the LED10 at (400.4, 159.5)
- removed the U2 at (421.9, 107.4)
- added C1: 0.1uF, Capacitor_SMD:C_0603_1608Metric_Pad1.08x0.95mm_HandSolder, B.Cu at (322.1, 121.4)
- added C10: 0.1uF, Capacitor_SMD:C_0603_1608Metric_Pad1.08x0.95mm_HandSolder, B.Cu at (132.3, 140.4)
- added C11: 0.1uF, Capacitor_SMD:C_0603_1608Metric_Pad1.08x0.95mm_HandSolder, B.Cu at (393.4, 178.6)
- added C12: 0.1uF, Capacitor_SMD:C_0603_1608Metric_Pad1.08x0.95mm_HandSolder, B.Cu at (127.6, 178.6)
- added C13: 0.1uF, Capacitor_SMD:C_0603_1608Metric_Pad1.08x0.95mm_HandSolder, B.Cu at (279.1, 159.5)
- added C14: 0.1uF, Capacitor_SMD:C_0603_1608Metric_Pad1.08x0.95mm_HandSolder, B.Cu at (393.4, 159.5)
- added C15: 0.1uF, Capacitor_SMD:C_0603_1608Metric_Pad1.08x0.95mm_HandSolder, B.Cu at (288.7, 178.4)
- added C16: 0.1uF, Capacitor_SMD:C_0603_1608Metric_Pad1.08x0.95mm_HandSolder, B.Cu at (326.9, 178.4)
- added C17: 0.1uF, Capacitor_SMD:C_0603_1608Metric_Pad1.08x0.95mm_HandSolder, B.Cu at (365.0, 178.4)
- added C18: 0.1uF, Capacitor_SMD:C_0603_1608Metric_Pad1.08x0.95mm_HandSolder, B.Cu at (130.0, 159.4)
- added C19: 0.1uF, Capacitor_SMD:C_0603_1608Metric_Pad1.08x0.95mm_HandSolder, B.Cu at (175.3, 159.5)
- added C2: 0.1uF, Capacitor_SMD:C_0603_1608Metric_Pad1.08x0.95mm_HandSolder, B.Cu at (360.2, 121.3)
- added C20: 0.1uF, Capacitor_SMD:C_0603_1608Metric_Pad1.08x0.95mm_HandSolder, B.Cu at (213.4, 159.5)
- added C21: 0.1uF, Capacitor_SMD:C_0603_1608Metric_Pad1.08x0.95mm_HandSolder, B.Cu at (222.9, 178.6)
- added C22: 0.1uF, Capacitor_SMD:C_0603_1608Metric_Pad1.08x0.95mm_HandSolder, B.Cu at (175.1, 178.5)
- added C23: 0.1uF, Capacitor_SMD:C_0603_1608Metric_Pad1.08x0.95mm_HandSolder, B.Cu at (331.5, 107.2)
- added C24: 0.1uF, Capacitor_SMD:C_0603_1608Metric_Pad1.08x0.95mm_HandSolder, B.Cu at (350.6, 107.2)
- added C25: 0.1uF, Capacitor_SMD:C_0603_1608Metric_Pad1.08x0.95mm_HandSolder, B.Cu at (369.6, 107.2)
- added C26: 0.1uF, Capacitor_SMD:C_0603_1608Metric_Pad1.08x0.95mm_HandSolder, B.Cu at (312.4, 107.2)
- added C27: 0.1uF, Capacitor_SMD:C_0603_1608Metric_Pad1.08x0.95mm_HandSolder, B.Cu at (274.4, 107.2)
- added C28: 0.1uF, Capacitor_SMD:C_0603_1608Metric_Pad1.08x0.95mm_HandSolder, B.Cu at (293.4, 107.2)
- added C29: 0.1uF, Capacitor_SMD:C_0603_1608Metric_Pad1.08x0.95mm_HandSolder, B.Cu at (398.1, 107.2)
- added C3: 0.1uF, Capacitor_SMD:C_0603_1608Metric_Pad1.08x0.95mm_HandSolder, B.Cu at (393.4, 121.4)
- added C30: 0.1uF, Capacitor_SMD:C_0603_1608Metric_Pad1.08x0.95mm_HandSolder, B.Cu at (170.4, 107.2)
- added C31: 0.1uF, Capacitor_SMD:C_0603_1608Metric_Pad1.08x0.95mm_HandSolder, B.Cu at (189.5, 107.2)
- added C32: 0.1uF, Capacitor_SMD:C_0603_1608Metric_Pad1.08x0.95mm_HandSolder, B.Cu at (208.5, 107.2)
- added C33: 0.1uF, Capacitor_SMD:C_0603_1608Metric_Pad1.08x0.95mm_HandSolder, B.Cu at (227.6, 107.2)
- added C34: 0.1uF, Capacitor_SMD:C_0603_1608Metric_Pad1.08x0.95mm_HandSolder, B.Cu at (132.5, 107.2)
- added C35: 0.1uF, Capacitor_SMD:C_0603_1608Metric_Pad1.08x0.95mm_HandSolder, B.Cu at (151.4, 107.2)
- added C36: 0.1uF, Capacitor_SMD:C_0603_1608Metric_Pad1.08x0.95mm_HandSolder, B.Cu at (113.4, 107.2)
- added C37: 0.1uF, Capacitor_SMD:C_0603_1608Metric_Pad1.08x0.95mm_HandSolder, B.Cu at (264.8, 126.2)
- added C38: 0.1uF, Capacitor_SMD:C_0603_1608Metric_Pad1.08x0.95mm_HandSolder, B.Cu at (283.8, 126.3)
- added C39: 0.1uF, Capacitor_SMD:C_0603_1608Metric_Pad1.08x0.95mm_HandSolder, B.Cu at (302.9, 126.3)
- added C4: 0.1uF, Capacitor_SMD:C_0603_1608Metric_Pad1.08x0.95mm_HandSolder, B.Cu at (395.7, 140.9)
- added C40: 0.1uF, Capacitor_SMD:C_0603_1608Metric_Pad1.08x0.95mm_HandSolder, B.Cu at (321.9, 126.2)
- added C41: 0.1uF, Capacitor_SMD:C_0603_1608Metric_Pad1.08x0.95mm_HandSolder, B.Cu at (341.0, 126.3)
- added C42: 0.1uF, Capacitor_SMD:C_0603_1608Metric_Pad1.08x0.95mm_HandSolder, B.Cu at (360.2, 126.1)
- added C43: 0.1uF, Capacitor_SMD:C_0603_1608Metric_Pad1.08x0.95mm_HandSolder, B.Cu at (379.2, 126.1)
- added C44: 0.1uF, Capacitor_SMD:C_0603_1608Metric_Pad1.08x0.95mm_HandSolder, B.Cu at (403.0, 126.1)
- added C45: 0.1uF, Capacitor_SMD:C_0603_1608Metric_Pad1.08x0.95mm_HandSolder, B.Cu at (118.0, 126.2)
- added C46: 0.1uF, Capacitor_SMD:C_0603_1608Metric_Pad1.08x0.95mm_HandSolder, B.Cu at (217.9, 126.2)
- added C47: 0.1uF, Capacitor_SMD:C_0603_1608Metric_Pad1.08x0.95mm_HandSolder, B.Cu at (141.7, 126.2)
- added C48: 0.1uF, Capacitor_SMD:C_0603_1608Metric_Pad1.08x0.95mm_HandSolder, B.Cu at (161.0, 126.3)
- added C49: 0.1uF, Capacitor_SMD:C_0603_1608Metric_Pad1.08x0.95mm_HandSolder, B.Cu at (199.1, 126.3)
- added C5: 0.1uF, Capacitor_SMD:C_0603_1608Metric_Pad1.08x0.95mm_HandSolder, B.Cu at (279.1, 140.4)
- added C50: 0.1uF, Capacitor_SMD:C_0603_1608Metric_Pad1.08x0.95mm_HandSolder, B.Cu at (269.7, 145.3)
- added C51: 0.1uF, Capacitor_SMD:C_0603_1608Metric_Pad1.08x0.95mm_HandSolder, B.Cu at (288.7, 145.3)
- added C52: 0.1uF, Capacitor_SMD:C_0603_1608Metric_Pad1.08x0.95mm_HandSolder, B.Cu at (307.6, 145.3)
- added C53: 0.1uF, Capacitor_SMD:C_0603_1608Metric_Pad1.08x0.95mm_HandSolder, B.Cu at (326.8, 145.3)
- added C54: 0.1uF, Capacitor_SMD:C_0603_1608Metric_Pad1.08x0.95mm_HandSolder, B.Cu at (345.7, 145.3)
- added C55: 0.1uF, Capacitor_SMD:C_0603_1608Metric_Pad1.08x0.95mm_HandSolder, B.Cu at (364.7, 145.3)
- added C56: 0.1uF, Capacitor_SMD:C_0603_1608Metric_Pad1.08x0.95mm_HandSolder, B.Cu at (395.7, 145.3)
- added C57: 0.1uF, Capacitor_SMD:C_0603_1608Metric_Pad1.08x0.95mm_HandSolder, B.Cu at (120.4, 145.3)
- added C58: 0.1uF, Capacitor_SMD:C_0603_1608Metric_Pad1.08x0.95mm_HandSolder, B.Cu at (146.7, 145.3)
- added C59: 0.1uF, Capacitor_SMD:C_0603_1608Metric_Pad1.08x0.95mm_HandSolder, B.Cu at (165.6, 145.3)
- added C6: 0.1uF, Capacitor_SMD:C_0603_1608Metric_Pad1.08x0.95mm_HandSolder, B.Cu at (170.8, 121.2)
- added C60: 0.1uF, Capacitor_SMD:C_0603_1608Metric_Pad1.08x0.95mm_HandSolder, B.Cu at (203.8, 145.3)
- added C61: 0.1uF, Capacitor_SMD:C_0603_1608Metric_Pad1.08x0.95mm_HandSolder, B.Cu at (222.6, 145.3)
- added C62: 0.1uF, Capacitor_SMD:C_0603_1608Metric_Pad1.08x0.95mm_HandSolder, B.Cu at (336.3, 164.2)
- added C63: 0.1uF, Capacitor_SMD:C_0603_1608Metric_Pad1.08x0.95mm_HandSolder, B.Cu at (279.0, 164.2)
- added C64: 0.1uF, Capacitor_SMD:C_0603_1608Metric_Pad1.08x0.95mm_HandSolder, B.Cu at (298.1, 164.2)
- added C65: 0.1uF, Capacitor_SMD:C_0603_1608Metric_Pad1.08x0.95mm_HandSolder, B.Cu at (317.1, 164.3)
- added C66: 0.1uF, Capacitor_SMD:C_0603_1608Metric_Pad1.08x0.95mm_HandSolder, B.Cu at (355.2, 164.2)
- added C67: 0.1uF, Capacitor_SMD:C_0603_1608Metric_Pad1.08x0.95mm_HandSolder, B.Cu at (391.0, 164.4)
- added C68: 0.1uF, Capacitor_SMD:C_0603_1608Metric_Pad1.08x0.95mm_HandSolder, B.Cu at (213.2, 164.3)
- added C69: 0.1uF, Capacitor_SMD:C_0603_1608Metric_Pad1.08x0.95mm_HandSolder, B.Cu at (125.2, 164.3)
- added C7: 0.1uF, Capacitor_SMD:C_0603_1608Metric_Pad1.08x0.95mm_HandSolder, B.Cu at (208.7, 121.1)
- added C70: 0.1uF, Capacitor_SMD:C_0603_1608Metric_Pad1.08x0.95mm_HandSolder, B.Cu at (156.2, 164.3)
- added C71: 0.1uF, Capacitor_SMD:C_0603_1608Metric_Pad1.08x0.95mm_HandSolder, B.Cu at (175.1, 164.3)
- added C72: 0.1uF, Capacitor_SMD:C_0603_1608Metric_Pad1.08x0.95mm_HandSolder, B.Cu at (232.2, 164.3)
- added C73: 0.1uF, Capacitor_SMD:C_0603_1608Metric_Pad1.08x0.95mm_HandSolder, B.Cu at (295.8, 183.4)
- added C74: 0.1uF, Capacitor_SMD:C_0603_1608Metric_Pad1.08x0.95mm_HandSolder, B.Cu at (333.9, 183.4)
- added C75: 0.1uF, Capacitor_SMD:C_0603_1608Metric_Pad1.08x0.95mm_HandSolder, B.Cu at (357.6, 183.4)
- added C76: 0.1uF, Capacitor_SMD:C_0603_1608Metric_Pad1.08x0.95mm_HandSolder, B.Cu at (381.5, 183.4)
- added C77: 0.1uF, Capacitor_SMD:C_0603_1608Metric_Pad1.08x0.95mm_HandSolder, B.Cu at (405.4, 183.4)
- added C78: 0.1uF, Capacitor_SMD:C_0603_1608Metric_Pad1.08x0.95mm_HandSolder, B.Cu at (115.6, 183.4)
- added C79: 0.1uF, Capacitor_SMD:C_0603_1608Metric_Pad1.08x0.95mm_HandSolder, B.Cu at (139.4, 183.4)
- added C8: 0.1uF, Capacitor_SMD:C_0603_1608Metric_Pad1.08x0.95mm_HandSolder, B.Cu at (208.5, 140.4)
- added C80: 0.1uF, Capacitor_SMD:C_0603_1608Metric_Pad1.08x0.95mm_HandSolder, B.Cu at (163.2, 183.4)
- added C81: 0.1uF, Capacitor_SMD:C_0603_1608Metric_Pad1.08x0.95mm_HandSolder, B.Cu at (220.3, 183.4)
- added C82: 0.1uF, Capacitor_SMD:C_0603_1608Metric_Pad1.08x0.95mm_HandSolder, B.Cu at (186.9, 183.3)
- added C83: 0.1uF, Capacitor_SMD:C_0603_1608Metric_Pad1.08x0.95mm_HandSolder, B.Cu at (180.0, 126.2)
- added C84: 0.1uF, Capacitor_SMD:C_0603_1608Metric_Pad1.08x0.95mm_HandSolder, B.Cu at (184.7, 145.3)
- added C85: 0.1uF, Capacitor_SMD:C_0603_1608Metric_Pad1.08x0.95mm_HandSolder, B.Cu at (194.1, 164.3)
- added C86: 0.1uF, Capacitor_SMD:C_0603_1608Metric_Pad1.08x0.95mm_HandSolder, B.Cu at (284.0, 121.3)
- added C87: 0.1uF, Capacitor_SMD:C_0603_1608Metric_Pad1.08x0.95mm_HandSolder, B.Cu at (132.5, 121.1)
- added C9: 0.1uF, Capacitor_SMD:C_0603_1608Metric_Pad1.08x0.95mm_HandSolder, B.Cu at (175.1, 140.4)
- added LED14: YS-SK6812MINI-E, kbd:YS-SK6812MINI-E_underglow, F.Cu at (388.5, 159.5)
- added R3: 500, Resistor_SMD:R_0805_2012Metric_Pad1.20x1.40mm_HandSolder, B.Cu at (414.3, 180.3)
- added R4: 500, Resistor_SMD:R_0805_2012Metric_Pad1.20x1.40mm_HandSolder, B.Cu at (97.3, 183.1)
- added U1: Elite-C, keebio:Elite-C, F.Cu at (421.8, 120.3)
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- renumbered LED8 to LED10, LED82 to LED11, LED83 to LED12, LED9 to LED13, LED11 to LED15, LED12 to LED16, LED84 to LED17, LED85 to LED18, LED13 to LED19, LED14 to LED20, LED15 to LED21, LED16 to LED22, LED86 to LED23, LED87 to LED24, LED17 to LED25, LED18 to LED26, LED19 to LED27, LED20 to LED28, LED21 to LED29, LED22 to LED30, LED23 to LED31, LED24 to LED32, LED25 to LED33, LED26 to LED34, LED27 to LED35, LED28 to LED36, LED29 to LED37, LED30 to LED38, LED31 to LED39, LED32 to LED40, LED33 to LED41, LED34 to LED42, LED35 to LED43, LED36 to LED44, LED37 to LED45, LED38 to LED46, LED39 to LED47, LED40 to LED48, LED41 to LED49, LED80 to LED5, LED42 to LED50, LED43 to LED51, LED44 to LED52, LED45 to LED53, LED46 to LED54, LED47 to LED55, LED48 to LED56, LED49 to LED57, LED50 to LED58, LED51 to LED59, LED81 to LED6, LED52 to LED60, LED53 to LED61, LED54 to LED62, LED55 to LED63, LED56 to LED64, LED57 to LED65, LED58 to LED66, LED59 to LED67, LED60 to LED68, LED61 to LED69, LED5 to LED7, LED62 to LED70, LED63 to LED71, LED64 to LED72, LED65 to LED73, LED66 to LED74, LED67 to LED75, LED68 to LED76, LED69 to LED77, LED70 to LED78, LED71 to LED79, LED6 to LED8, LED72 to LED80, LED73 to LED81, LED74 to LED82, LED75 to LED83, LED76 to LED84, LED77 to LED85, LED78 to LED86, LED79 to LED87, LED7 to LED9, U1 to U2
Connections:
- J2 pad A: VCC -> VDD
- J2 pad B: GND -> GNDA
- LED1 pad 1: VCC -> VDD
- LED1 pad 3: GND -> GNDA
- LED11 pad 3: Net-(LED82-Pad3) -> GND
- LED12 pad 3: Net-(LED82-Pad3) -> GND
- LED13 pad 1: VCC -> VDD
- LED13 pad 2: Net-(LED74-Pad4) -> Net-(LED1-Pad4)
- LED13 pad 3: GND -> GNDA
- LED15 pad 1: VCC -> VDD
- LED15 pad 3: GND -> GNDA
- LED16 pad 1: VCC -> VDD
- LED16 pad 3: GND -> GNDA
- LED17 pad 1: VCC -> VDD
- LED17 pad 3: GND -> GNDA
- LED18 pad 1: VCC -> VDD
- LED18 pad 3: GND -> GNDA
- LED18 pad 4: Net-(LED81-Pad2) -> Net-(LED18-Pad4)
- LED19 pad 2: Net-(LED13-Pad2) -> Net-(LED19-Pad2)
- LED19 pad 4: Net-(LED13-Pad4) (its old number) -> Net-(LED19-Pad4)
- LED2 pad 1: VCC -> VDD
- LED2 pad 3: GND -> GNDA
- LED20 pad 2: Net-(LED14-Pad2) -> Net-(LED19-Pad4)
- LED23 pad 3: Net-(LED82-Pad3) -> GND
- LED24 pad 3: Net-(LED82-Pad3) -> GND
- LED25 pad 1: VCC -> VDD
- LED25 pad 3: GND -> GNDA
- LED26 pad 1: VCC -> VDD
- LED26 pad 3: GND -> GNDA
- LED27 pad 1: VCC -> VDD
- LED27 pad 3: GND -> GNDA
- LED28 pad 1: VCC -> VDD
- LED28 pad 3: GND -> GNDA
- LED29 pad 1: VCC -> VDD
- LED29 pad 3: GND -> GNDA
- LED3 pad 1: VCC -> VDD
- LED3 pad 3: GND -> GNDA
- LED30 pad 1: VCC -> VDD
- LED30 pad 3: GND -> GNDA
- LED31 pad 1: VCC -> VDD
- LED31 pad 3: Net-(LED23-Pad3) -> GNDA
- LED32 pad 2: Net-(LED24-Pad2) -> Net-(LED32-Pad2)
- LED33 pad 4: Net-(LED25-Pad4) (its old number) -> Net-(LED32-Pad2)
- LED34 pad 2: Net-(LED25-Pad4) (its old number) -> Net-(LED34-Pad2)
- LED35 pad 4: Net-(LED27-Pad4) (its old number) -> Net-(LED34-Pad2)
- LED36 pad 2: Net-(LED27-Pad4) (its old number) -> Net-(LED36-Pad2)
- LED37 pad 4: Net-(LED29-Pad4) (its old number) -> Net-(LED36-Pad2)
- LED38 pad 2: Net-(LED29-Pad4) (its old number) -> Net-(LED38-Pad2)
- LED38 pad 3: Net-(LED30-Pad3) -> GND
- LED39 pad 1: VCC -> VDD
- LED39 pad 3: GND -> GNDA
- LED4 pad 1: VCC -> VDD
- LED4 pad 3: GND -> GNDA
- LED40 pad 1: VCC -> VDD
- LED40 pad 3: GND -> GNDA
- LED41 pad 1: Net-(LED33-Pad1) -> VDD
- LED41 pad 3: Net-(LED33-Pad3) -> GNDA
- LED42 pad 1: VCC -> VDD
- LED42 pad 3: GND -> GNDA
- LED43 pad 1: VCC -> VDD
- LED43 pad 3: GND -> GNDA
- LED44 pad 1: VCC -> VDD
- LED44 pad 3: GND -> GNDA
- LED45 pad 1: VCC -> VDD
- LED45 pad 3: GND -> GNDA
- LED46 pad 1: VCC -> VDD
- LED46 pad 3: Net-(LED23-Pad3) -> GNDA
- LED5 pad 1: VCC -> VDD
- LED5 pad 3: GND -> GNDA
- LED52 pad 3: Net-(LED30-Pad3) -> GND
- LED53 pad 1: VCC -> VDD
- LED53 pad 3: GND -> GNDA
- LED54 pad 1: VCC -> VDD
- LED54 pad 3: GND -> GNDA
- LED55 pad 1: VCC -> VDD
- LED55 pad 3: GND -> GNDA
- LED56 pad 1: VCC -> VDD
- LED56 pad 3: GND -> GNDA
- LED57 pad 1: VCC -> VDD
- LED57 pad 3: GND -> GNDA
- LED58 pad 1: VCC -> VDD
- LED58 pad 3: GND -> GNDA
- LED58 pad 4: Net-(LED50-Pad4) (its old number) -> Net-(LED58-Pad4)
- LED59 pad 1: VCC -> VDD
- LED59 pad 3: GND -> GNDA
- LED6 pad 1: VCC -> VDD
- LED6 pad 2: Net-(LED81-Pad2) -> Net-(LED6-Pad2)
- LED6 pad 3: GND -> GNDA
- LED65 pad 3: Net-(LED30-Pad3) -> GND
- LED66 pad 1: VCC -> VDD
- LED66 pad 3: GND -> GNDA
- LED67 pad 1: VCC -> VDD
- LED67 pad 3: GND -> GNDA
- LED68 pad 1: VCC -> VDD
- LED68 pad 3: GND -> GNDA
- LED69 pad 1: VCC -> VDD
- LED69 pad 3: GND -> GNDA
- LED70 pad 1: VCC -> VDD
- LED70 pad 2: Net-(LED62-Pad2) (its old number) -> Net-(LED70-Pad2)
- LED70 pad 3: GND -> GNDA
- LED71 pad 1: VCC -> VDD
- LED71 pad 3: GND -> GNDA
- LED74 pad 2: Net-(LED66-Pad2) (its old number) -> Net-(LED74-Pad2)
- LED75 pad 4: Net-(LED67-Pad4) (its old number) -> Net-(LED75-Pad4)
- LED76 pad 2: Net-(LED67-Pad4) (its old number) -> Net-(LED76-Pad2)
- LED77 pad 3: Net-(LED30-Pad3) -> GND
- LED77 pad 4: Net-(LED69-Pad4) (its old number) -> Net-(LED77-Pad4)
- LED78 pad 1: VCC -> VDD
- LED78 pad 3: GND -> GNDA
- LED79 pad 1: VCC -> VDD
- LED79 pad 3: GND -> GNDA
- LED80 pad 1: VCC -> VDD
- LED80 pad 3: GND -> GNDA
- LED80 pad 4: Net-(LED72-Pad4) -> Net-(LED70-Pad2)
- LED81 pad 1: VCC -> VDD
- LED81 pad 2: Net-(LED73-Pad2) -> Net-(LED58-Pad4)
- LED81 pad 3: Net-(LED73-Pad3) -> GNDA
- LED82 pad 1: VCC -> VDD
- LED82 pad 3: Net-(LED23-Pad3) -> GNDA
- LED82 pad 4: Net-(LED74-Pad4) -> Net-(LED82-Pad4)
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Other:
- board size 351.3 x 110.1 mm -> 351.3 x 110.2 mm

Commit message: laying out traces on the right
Parts:
- moved RSW1 2.25 mm to (421.8, 142.1)
- moved RSW2 2.25 mm to (89.3, 142.1)
Routing:
- net col0_R: track 0.00 -> 274.4 mm, vias 0 -> 10
- net col1_R: track 0.00 -> 219.6 mm, vias 0 -> 8
- net col3_R: track 0.00 -> 203.5 mm, vias 0 -> 10
- net col2_R: track 0.00 -> 201.5 mm, vias 0 -> 8
- net col4_R: track 0.00 -> 185.1 mm, vias 0 -> 10
- net row2_R: track 0.00 -> 177.5 mm, vias 0 -> 18
- net row4_R: track 0.00 -> 175.9 mm, vias 0 -> 12
- net row1_R: track 0.00 -> 167.7 mm, vias 0 -> 18
- net row0_R: track 0.00 -> 161.8 mm, vias 0 -> 14
- net col7_R: track 0.00 -> 137.2 mm, vias 0 -> 2
- net col6_R: track 0.00 -> 133.7 mm, vias 0 -> 8
- net VDD: track 0.00 -> 129.4 mm
- net col5_R: track 0.00 -> 109.6 mm, vias 0 -> 5
- net Net-(LED46-Pad4): track 0.00 -> 59.2 mm
- net Net-(LED31-Pad2): track 0.00 -> 51.2 mm, vias 0 -> 4
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
Commit message: routing WIP
Routing:
- net GNDA: track 0.00 -> 652.7 mm, vias 0 -> 46
- net VDD: track 129.4 -> 706.8 mm, vias 0 -> 32
- net Net-(LED79-Pad4): track 0.00 -> 53.8 mm
- net Net-(LED29-Pad2): track 0.00 -> 47.6 mm, vias 0 -> 2
- net Net-(LED27-Pad2): track 0.00 -> 45.1 mm
- net Net-(LED25-Pad2): track 0.00 -> 39.1 mm, vias 0 -> 2
- net Net-(LED66-Pad2): track 0.00 -> 37.3 mm
- net Net-(LED27-Pad4): track 0.00 -> 35.6 mm
- net Net-(LED39-Pad2): track 0.00 -> 33.4 mm, vias 0 -> 2
- net Net-(LED25-Pad4): track 0.00 -> 32.4 mm
- net Net-(LED43-Pad2): track 0.00 -> 32.1 mm
- net Net-(LED70-Pad2): track 0.00 -> 31.4 mm
- net Net-(LED57-Pad2): track 0.00 -> 29.0 mm, vias 0 -> 2
- net Net-(LED67-Pad4): track 0.00 -> 29.0 mm, vias 0 -> 2
- net Net-(LED55-Pad2): track 0.00 -> 27.4 mm, vias 0 -> 2
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
Commit message: routing WIP
Routing:
- net col5_R: track 111.6 -> 114.4 mm, vias 5 -> 6

Commit message: right side routed
Parts:
- moved D_53 69.4 mm to (262.6, 223.6)
- moved C10 69.4 mm to (175.1, 195.0)
- moved C18 69.4 mm to (172.8, 214.0)
- moved C21 69.4 mm to (265.7, 233.2)
- moved C30 69.4 mm to (213.2, 161.8)
- moved C32 69.4 mm to (251.3, 161.8)
- moved C35 69.4 mm to (194.2, 161.8)
- moved C36 69.4 mm to (156.2, 161.8)
- moved C45 69.4 mm to (160.8, 180.8)
- moved C46 69.4 mm to (260.7, 180.8)
- moved C47 69.4 mm to (184.5, 180.8)
- moved C48 69.4 mm to (203.8, 180.9)
- moved C49 69.4 mm to (241.9, 180.9)
- moved C6 69.4 mm to (213.6, 175.8)
- moved C69 69.4 mm to (168.0, 218.9)
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Connections:
- LED13 pad 2: Net-(LED1-Pad4) -> Net-(LED13-Pad2)
- LED14 pad 2: Net-(LED13-Pad4) -> Net-(LED14-Pad2)
- LED15 pad 2: Net-(LED14-Pad4) -> Net-(LED13-Pad4)
- LED5 pad 2: Net-(LED5-Pad2) -> Net-(LED14-Pad4)
- LED6 pad 2: Net-(LED6-Pad2) -> Net-(LED1-Pad4)
- LED6 pad 4: Net-(LED5-Pad2) -> Net-(LED13-Pad2)
- U2 pad 25: Net-(U2-Pad25) -> BACKLIGHT_LED_L
- U2 pad 29: BACKLIGHT_LED_L -> Net-(U2-Pad29)
Routing:
- net GNDA: track 652.7 -> 1034.0 mm, vias 46 -> 63
- net VDD: track 706.8 -> 1072.4 mm, vias 32 -> 36
- net row3_R: track 0.00 -> 183.9 mm, vias 0 -> 12
- net Net-(LED16-Pad4): track 0.00 -> 48.7 mm, vias 0 -> 4
- net Net-(LED15-Pad4): track 0.00 -> 47.9 mm, vias 0 -> 2
- net Net-(LED17-Pad4): track 0.00 -> 39.3 mm, vias 0 -> 2
- net Net-(LED1-Pad2): track 0.00 -> 36.3 mm, vias 0 -> 4
- net Net-(LED2-Pad2): track 0.00 -> 35.8 mm, vias 0 -> 4
- net Net-(LED18-Pad4): track 0.00 -> 34.6 mm, vias 0 -> 2
- net Net-(LED13-Pad4): track 0.00 -> 34.6 mm, vias 0 -> 2
- net Net-(LED3-Pad2): track 0.00 -> 33.2 mm, vias 0 -> 2
- net Net-(LED1-Pad4): track 0.00 -> 31.1 mm, vias 0 -> 2
- net BACKLIGHT_LED_R: track 0.00 -> 28.9 mm, vias 0 -> 1
- net Net-(LED13-Pad2): track 0.00 -> 27.4 mm, vias 0 -> 4
- net Net-(LED14-Pad4): track 0.00 -> 26.6 mm, vias 0 -> 4
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Other:
- board size 351.3 x 110.2 mm -> 333.9 x 110.2 mm
