File: onigaku.kicad_pcb (KiCad board)
At the start: 2 copper layers, 333.9 x 110.2 mm, 312 parts, among them J1 MJ-4PP-9, J2 MJ-4PP-9, U1 Elite-C, U2 Elite-C

Commit message: wiring up oleds and trs. starting left side
Parts:
- moved C80 23.9 mm to (229.9, 238.0)
- moved D_62 23.9 mm to (217.4, 242.7)
- moved LED85 23.9 mm to (224.9, 238.0)
- moved SW_62 23.9 mm to (225.0, 242.7)
- moved C82 23.7 mm to (206.0, 237.9)
- moved D_61 23.7 mm to (193.5, 242.7)
- moved LED86 23.7 mm to (201.0, 237.9)
- moved SW_61 23.7 mm to (201.2, 242.7)
- moved R3 4.70 mm to (435.0, 234.9)
- moved R1 4.44 mm to (435.2, 217.8)
Connections:
- U2 pad 14: col6_L -> col0_L
- U2 pad 15: col5_L -> col1_L
- U2 pad 16: col4_L -> col2_L
- U2 pad 18: col2_L -> col4_L
- U2 pad 19: col1_L -> col5_L
- U2 pad 20: col0_L -> col6_L
Routing:
- net GND: track 0.00 -> 380.8 mm
- net VCC: track 0.00 -> 295.7 mm, vias 0 -> 1
- net col6_L: track 0.00 -> 250.4 mm, vias 0 -> 9
- net col5_L: track 0.00 -> 220.5 mm, vias 0 -> 7
- net col3_L: track 0.00 -> 199.0 mm, vias 0 -> 9
- net col4_L: track 0.00 -> 191.8 mm, vias 0 -> 8
- net VDD: track 1072.4 -> 1248.6 mm, vias 36 -> 38
- net col2_L: track 0.00 -> 171.8 mm, vias 0 -> 9
- net row4_L: track 0.00 -> 171.1 mm, vias 0 -> 17
- net GNDA: track 1034.0 -> 1201.6 mm
- net row3_L: track 0.00 -> 162.1 mm, vias 0 -> 13
- net data_R: track 0.00 -> 157.6 mm
- net data_L: track 0.00 -> 148.3 mm, vias 0 -> 1
- net row0_L: track 0.00 -> 141.4 mm, vias 0 -> 12
- net row2_L: track 0.00 -> 141.0 mm, vias 0 -> 11
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