File: onigaku.kicad_pcb (KiCad board)
At the start: 2 copper layers, 333.9 x 110.2 mm, 308 parts, among them J1 MJ-4PP-9, J2 MJ-4PP-9, U1 Elite-C, U2 Elite-C

Commit message: redid entire left side
Parts:
- added C19: 0.1uF, Capacitor_SMD:C_0603_1608Metric_Pad1.08x0.95mm_HandSolder, F.Cu at (477.6, 295.2)
- added C88: 0.1uF, Capacitor_SMD:C_0603_1608Metric_Pad1.08x0.95mm_HandSolder, F.Cu at (399.8, 267.8)
- added C89: 0.1uF, Capacitor_SMD:C_0603_1608Metric_Pad1.08x0.95mm_HandSolder, F.Cu at (399.8, 270.3)
- added C9: 0.1uF, Capacitor_SMD:C_0603_1608Metric_Pad1.08x0.95mm_HandSolder, B.Cu at (476.1, 238.0)
- added C90: 0.1uF, Capacitor_SMD:C_0603_1608Metric_Pad1.08x0.95mm_HandSolder, F.Cu at (404.1, 267.8)
- added C91: 0.1uF, Capacitor_SMD:C_0603_1608Metric_Pad1.08x0.95mm_HandSolder, F.Cu at (399.8, 272.8)
- added C92: 0.1uF, Capacitor_SMD:C_0603_1608Metric_Pad1.08x0.95mm_HandSolder, F.Cu at (404.1, 270.3)
- added C93: 0.1uF, Capacitor_SMD:C_0603_1608Metric_Pad1.08x0.95mm_HandSolder, F.Cu at (408.5, 267.8)
- added C94: 0.1uF, Capacitor_SMD:C_0603_1608Metric_Pad1.08x0.95mm_HandSolder, F.Cu at (404.1, 272.8)
- added C95: 0.1uF, Capacitor_SMD:C_0603_1608Metric_Pad1.08x0.95mm_HandSolder, F.Cu at (408.5, 270.3)
- added D_64: D, kbd:D3_SMD_v2, B.Cu at (444.2, 186.6)
- added D_65: D, kbd:D3_SMD_v2, F.Cu at (487.2, 278.9)
- added D_66: D, kbd:D3_SMD_v2, F.Cu at (478.3, 282.3)
- added D_67: D, kbd:D3_SMD_v2, F.Cu at (484.0, 282.3)
- added D_68: D, kbd:D3_SMD_v2, F.Cu at (489.8, 282.3)
- added D_69: D, kbd:D3_SMD_v2, F.Cu at (478.3, 285.6)
- added D_70: D, kbd:D3_SMD_v2, F.Cu at (484.0, 285.6)
- added D_71: D, kbd:D3_SMD_v2, F.Cu at (478.3, 289.0)
- added D_72: D, kbd:D3_SMD_v2, F.Cu at (484.0, 289.0)
- added D_73: D, kbd:D3_SMD_v2, F.Cu at (478.3, 292.3)
- added K_14: KEYSW, kbd:CherryMX_Hotswap, F.Cu at (452.0, 166.5)
- added K_15: KEYSW, kbd:CherryMX_Hotswap, F.Cu at (471.1, 166.5)
- added K_16: KEYSW, kbd:CherryMX_Hotswap, F.Cu at (490.2, 166.5)
- added K_31: KEYSW, kbd:CherryMX_Hotswap, F.Cu at (452.0, 185.5)
- added K_32: KEYSW, kbd:CherryMX_Hotswap, F.Cu at (471.1, 185.5)
- added K_33: KEYSW, kbd:CherryMX_Hotswap, F.Cu at (490.2, 185.5)
- added K_59: KEYSW, kbd:CherryMX_Hotswap, F.Cu at (471.0, 223.6)
- added K_68: KEYSW, kbd:CherryMX_Hotswap, F.Cu at (452.0, 242.7)
- added K_69: KEYSW, kbd:CherryMX_Hotswap, F.Cu at (471.0, 242.7)
- added K_70: KEYSW, kbd:CherryMX_Hotswap, F.Cu at (490.1, 242.7)
- added LED11: YS-SK6812MINI-E, kbd:YS-SK6812MINI-E, B.Cu at (452.1, 161.8)
- added LED20: YS-SK6812MINI-E, kbd:YS-SK6812MINI-E, B.Cu at (471.1, 161.7)
- added LED88: YS-SK6812MINI-E, kbd:YS-SK6812MINI-E, B.Cu at (490.2, 161.8)
- added LED89: YS-SK6812MINI-E, kbd:YS-SK6812MINI-E, B.Cu at (452.1, 180.8)
- added LED90: YS-SK6812MINI-E, kbd:YS-SK6812MINI-E, B.Cu at (471.2, 180.8)
- added LED91: YS-SK6812MINI-E, kbd:YS-SK6812MINI-E, B.Cu at (490.2, 180.8)
- added LED92: YS-SK6812MINI-E, kbd:YS-SK6812MINI-E, B.Cu at (471.2, 218.9)
- added LED93: YS-SK6812MINI-E, kbd:YS-SK6812MINI-E, B.Cu at (452.1, 238.0)
- added LED94: YS-SK6812MINI-E, kbd:YS-SK6812MINI-E, B.Cu at (471.2, 238.0)
- added LED95: YS-SK6812MINI-E, kbd:YS-SK6812MINI-E, B.Cu at (490.1, 238.0)
- moved RSW1 66.4 mm to (513.5, 196.6)
- moved U1 66.4 mm to (513.5, 174.8)
- moved R2 4.96 mm to (139.6, 196.7)
- moved U2 1.80 mm to (131.1, 176.3)
- moved C10 0.94 mm to (175.1, 196.0)
- moved C33 0.89 mm to (271.3, 161.8)
- moved LED12 0.82 mm to (170.2, 195.9)
- moved C87 0.46 mm to (175.0, 176.1)
- moved LED7 0.46 mm to (170.1, 176.1)
- turned C27 to 90 degrees
- turned C28 to 90 degrees
Connections:
- C23 pad 1: GNDA -> VCC
- C23 pad 2: VDD -> GND
- C24 pad 1: GNDA -> GND
- C24 pad 2: VDD -> VCC
- C25 pad 1: GNDA -> VCC
- C25 pad 2: VDD -> GND
- C26 pad 1: GNDA -> GND
- C26 pad 2: VDD -> VCC
- C27 pad 1: GNDA -> VCC
- C27 pad 2: VDD -> GND
- C28 pad 1: GNDA -> VCC
- C28 pad 2: VDD -> GND
- C29 pad 1: GNDA -> VCC
- C29 pad 2: VDD -> GND
- C37 pad 1: GNDA -> GND
- C37 pad 2: VDD -> VCC
- C38 pad 1: GNDA -> VCC
- C38 pad 2: VDD -> GND
- C39 pad 1: GNDA -> GND
- C39 pad 2: VDD -> VCC
- C40 pad 1: GNDA -> VCC
- C40 pad 2: VDD -> GND
- C41 pad 1: GNDA -> GND
- C41 pad 2: VDD -> VCC
- C42 pad 1: GNDA -> VCC
- C42 pad 2: VDD -> GND
- C43 pad 1: GNDA -> GND
- C43 pad 2: VDD -> VCC
- C44 pad 1: VDD -> GND
- C44 pad 2: GNDA -> VCC
- C50 pad 1: GNDA -> GND
- C50 pad 2: VDD -> VCC
- C51 pad 1: GNDA -> VCC
- C51 pad 2: VDD -> GND
- C52 pad 1: GNDA -> GND
- C52 pad 2: VDD -> VCC
- C53 pad 1: GNDA -> VCC
- C53 pad 2: VDD -> GND
- C54 pad 1: GNDA -> VCC
- C54 pad 2: VDD -> GND
- C55 pad 1: GNDA -> GND
- C55 pad 2: VDD -> VCC
- C56 pad 1: GNDA -> VCC
- C56 pad 2: VDD -> GND
- C62 pad 1: GNDA -> VCC
- C62 pad 2: VDD -> GND
- C63 pad 1: GNDA -> GND
- C63 pad 2: VDD -> VCC
- C64 pad 1: GNDA -> VCC
- C64 pad 2: VDD -> GND
- C65 pad 1: GNDA -> GND
- C65 pad 2: VDD -> VCC
- C66 pad 1: GNDA -> VCC
- C66 pad 2: VDD -> GND
- C67 pad 1: GNDA -> GND
- C67 pad 2: VDD -> VCC
- C73 pad 1: GNDA -> GND
- C73 pad 2: VDD -> VCC
- C74 pad 1: GNDA -> GND
- C74 pad 2: VDD -> VCC
- C75 pad 1: GNDA -> VCC
- C75 pad 2: VDD -> GND
- C76 pad 1: GNDA -> GND
- C76 pad 2: VDD -> VCC
- C77 pad 1: VDD -> GND
- C77 pad 2: GNDA -> VCC
- LED25 pad 1: VDD -> VCC
- LED25 pad 3: GNDA -> GND
- LED26 pad 1: VDD -> VCC
- LED26 pad 3: GNDA -> GND
- LED27 pad 1: VDD -> VCC
- LED27 pad 3: GNDA -> GND
- LED28 pad 1: VDD -> VCC
- LED28 pad 3: GNDA -> GND
- LED29 pad 1: VDD -> VCC
- LED29 pad 3: GNDA -> GND
- LED30 pad 1: VDD -> VCC
- LED30 pad 3: GNDA -> GND
- LED31 pad 1: VDD -> VCC
- LED31 pad 3: GNDA -> GND
- LED33 pad 4: Net-(LED32-Pad2) -> Net-(LED33-Pad4)
- LED35 pad 4: Net-(LED34-Pad2) -> Net-(LED35-Pad4)
- LED37 pad 4: Net-(LED36-Pad2) -> Net-(LED37-Pad4)
- LED39 pad 1: VDD -> VCC
- LED39 pad 3: GNDA -> GND
- LED40 pad 1: VDD -> VCC
- LED40 pad 3: GNDA -> GND
- LED41 pad 1: VDD -> GND
- LED41 pad 2: Net-(LED41-Pad2) -> Net-(LED27-Pad2)
- LED41 pad 3: GNDA -> VCC
- LED41 pad 4: Net-(LED27-Pad2) -> Net-(LED41-Pad4)
- LED42 pad 1: VDD -> VCC
- LED42 pad 3: GNDA -> GND
- LED43 pad 1: VDD -> VCC
- LED43 pad 3: GNDA -> GND
- LED44 pad 1: VDD -> VCC
- LED44 pad 3: GNDA -> GND
- LED45 pad 1: VDD -> VCC
- LED45 pad 3: GNDA -> GND
- LED46 pad 1: VDD -> VCC
- LED46 pad 3: GNDA -> GND
- LED47 pad 4: Net-(LED47-Pad4) -> Net-(LED32-Pad2)
- LED48 pad 2: Net-(LED47-Pad4) -> Net-(LED48-Pad2)
- LED48 pad 4: Net-(LED48-Pad4) -> Net-(LED34-Pad2)
- LED49 pad 2: Net-(LED48-Pad4) -> Net-(LED35-Pad4)
- LED50 pad 2: Net-(LED49-Pad4) -> Net-(LED50-Pad2)
- LED50 pad 4: Net-(LED50-Pad4) -> Net-(LED36-Pad2)
- LED51 pad 2: Net-(LED50-Pad4) -> Net-(LED37-Pad4)
- LED52 pad 2: Net-(LED51-Pad4) -> Net-(LED52-Pad2)
- LED53 pad 1: VDD -> VCC
- LED53 pad 3: GNDA -> GND
- LED54 pad 1: VDD -> VCC
- LED54 pad 3: GNDA -> GND
- LED55 pad 1: VDD -> VCC
- LED55 pad 3: GNDA -> GND
- LED55 pad 4: Net-(LED41-Pad2) -> Net-(LED41-Pad4)
- LED56 pad 1: VDD -> VCC
- LED56 pad 3: GNDA -> GND
- LED57 pad 1: VDD -> VCC
- LED57 pad 3: GNDA -> GND
- LED58 pad 1: VDD -> VCC
- LED58 pad 3: GNDA -> GND
- LED59 pad 1: VDD -> VCC
- LED59 pad 3: GNDA -> GND
- LED61 pad 4: Net-(LED60-Pad2) -> Net-(LED48-Pad2)
- LED62 pad 2: Net-(LED62-Pad2) -> Net-(LED49-Pad4)
- LED62 pad 4: Net-(LED61-Pad2) -> Net-(LED62-Pad4)
- LED63 pad 4: Net-(LED62-Pad2) -> Net-(LED50-Pad2)
- LED64 pad 2: Net-(LED64-Pad2) -> Net-(LED51-Pad4)
- LED64 pad 4: Net-(LED63-Pad2) -> Net-(LED64-Pad4)
- LED65 pad 4: Net-(LED64-Pad2) -> Net-(LED52-Pad2)
- LED66 pad 1: VDD -> VCC
- LED66 pad 3: GNDA -> GND
- LED67 pad 1: VDD -> VCC
- LED67 pad 3: GNDA -> GND
- LED68 pad 1: VDD -> VCC
- LED68 pad 3: GNDA -> GND
- LED69 pad 1: VDD -> VCC
- LED69 pad 3: GNDA -> GND
- LED70 pad 1: VDD -> VCC
- LED70 pad 3: GNDA -> GND
- LED71 pad 1: VDD -> VCC
- LED71 pad 3: GNDA -> GND
- LED72 pad 2: Net-(LED72-Pad2) -> Net-(LED33-Pad4)
- LED73 pad 2: Net-(LED72-Pad4) -> Net-(LED73-Pad2)
- LED73 pad 4: Net-(LED73-Pad4) -> Net-(LED61-Pad2)
- LED74 pad 2: Net-(LED73-Pad4) -> Net-(LED62-Pad4)
- LED75 pad 2: Net-(LED74-Pad4) -> Net-(LED75-Pad2)
- LED75 pad 4: Net-(LED75-Pad4) -> Net-(LED63-Pad2)
- LED76 pad 2: Net-(LED75-Pad4) -> Net-(LED64-Pad4)
- LED76 pad 4: Net-(LED76-Pad4) -> Net-(LED75-Pad2)
- LED77 pad 2: Net-(LED76-Pad4) -> Net-(LED77-Pad2)
- LED78 pad 1: VDD -> VCC
- LED78 pad 3: GNDA -> GND
- LED79 pad 1: VDD -> VCC
- LED79 pad 3: GNDA -> GND
- LED80 pad 1: VDD -> VCC
- LED80 pad 3: GNDA -> GND
- LED81 pad 1: VDD -> VCC
- LED81 pad 3: GNDA -> GND
- LED82 pad 1: VDD -> VCC
- LED82 pad 3: GNDA -> GND
- LED83 pad 4: Net-(LED72-Pad2) -> Net-(LED60-Pad2)
- LED84 pad 2: Net-(LED84-Pad2) -> Net-(LED72-Pad4)
- LED85 pad 2: Net-(LED85-Pad2) -> Net-(LED74-Pad4)
- LED86 pad 4: Net-(LED84-Pad2) -> Net-(LED73-Pad2)
- LED87 pad 4: Net-(LED85-Pad2) -> Net-(LED77-Pad2)
- R3 pad 1: Net-(LED82-Pad4) -> Net-(LED88-Pad4)
- U1 pad 27: Net-(U1-Pad27) -> col8_R
- U1 pad 28: Net-(U1-Pad28) -> col9_R
- U1 pad 29: Net-(U1-Pad29) -> col10_R
- U2 pad 14: col0_L -> col6_L
- U2 pad 15: col1_L -> col5_L
- U2 pad 16: col2_L -> col4_L
- U2 pad 18: col4_L -> col2_L
- U2 pad 19: col5_L -> col1_L
- U2 pad 20: col6_L -> col0_L
Routing:
- net GND: track 20.6 -> 1027.0 mm, vias 1 -> 9
- net VCC: track 1270.3 -> 1013.2 mm, vias 106 -> 22
- net row0_L: track 141.7 -> 223.1 mm, vias 15 -> 2
- net Net-(LED33-Pad4): track 0.00 -> 59.8 mm, vias 0 -> 2
- net GNDA: track 1072.3 -> 1023.2 mm, vias 24 -> 22
- net col6_L: track 250.4 -> 294.5 mm
- net row2_L: track 143.5 -> 186.6 mm, vias 11 -> 2
- net Net-(LED47-Pad4): track 39.8 -> 0.00 mm, vias 6 -> 0
- net row1_L: track 142.1 -> 181.3 mm, vias 15 -> 2
- net row3_L: track 172.7 -> 211.5 mm, vias 13 -> 2
- net Net-(LED72-Pad2): track 38.5 -> 0.00 mm, vias 4 -> 0
- net Net-(LED77-Pad2): track 0.00 -> 34.2 mm, vias 0 -> 2
- net Net-(LED76-Pad4): track 33.6 -> 0.00 mm, vias 4 -> 0
- net Net-(LED48-Pad4): track 33.3 -> 0.00 mm, vias 4 -> 0
- net Net-(LED50-Pad4): track 33.1 -> 0.00 mm, vias 4 -> 0
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- removed copper zone on B.Cu, net GND
- removed copper zone on B.Cu, net GNDA
Other:
- board size 333.9 x 110.2 mm -> 402.1 x 110.2 mm

Commit message: redoing right side, figuring out reset switch WIP
Parts:
- added C100: 0.1uF, Capacitor_SMD:C_0603_1608Metric_Pad1.08x0.95mm_HandSolder, B.Cu at (495.2, 233.2)
- added C101: 0.1uF, Capacitor_SMD:C_0603_1608Metric_Pad1.08x0.95mm_HandSolder, B.Cu at (495.3, 176.0)
- added C96: 0.1uF, Capacitor_SMD:C_0603_1608Metric_Pad1.08x0.95mm_HandSolder, B.Cu at (445.3, 233.1)
- added C97: 0.1uF, Capacitor_SMD:C_0603_1608Metric_Pad1.08x0.95mm_HandSolder, B.Cu at (495.6, 199.7)
- added C98: 0.1uF, Capacitor_SMD:C_0603_1608Metric_Pad1.08x0.95mm_HandSolder, B.Cu at (495.3, 217.8)
- added C99: 0.1uF, Capacitor_SMD:C_0603_1608Metric_Pad1.08x0.95mm_HandSolder, B.Cu at (469.8, 233.2)
- added LED100: YS-SK6812MINI-E, kbd:YS-SK6812MINI-E_underglow, F.Cu at (490.1, 233.2)
- added LED101: YS-SK6812MINI-E, kbd:YS-SK6812MINI-E_underglow, F.Cu at (490.2, 176.0)
- added LED96: YS-SK6812MINI-E, kbd:YS-SK6812MINI-E_underglow, F.Cu at (440.1, 233.2)
- added LED97: YS-SK6812MINI-E, kbd:YS-SK6812MINI-E_underglow, F.Cu at (490.5, 199.6)
- added LED98: YS-SK6812MINI-E, kbd:YS-SK6812MINI-E_underglow, F.Cu at (490.2, 217.9)
- added LED99: YS-SK6812MINI-E, kbd:YS-SK6812MINI-E_underglow, F.Cu at (464.7, 233.2)
- C19, C88, C89, C90, C91, C92, C93, C94, C95, D_65, D_66, D_67, D_68, D_69, D_70, D_71, D_72, D_73: moved to B.Cu
- RSW1, RSW2: footprint Button_Switch_SMD:SW_SPST_TL3342 -> kbd:ResetSW_1side
- moved C90 139.7 mm to (495.2, 161.8), turned to 270 degrees
- moved C89 132.7 mm to (476.1, 161.7), turned to 270 degrees
- moved C93 122.8 mm to (495.2, 180.7), turned to 270 degrees
- moved C88 120.6 mm to (457.1, 161.7), turned to 270 degrees
- moved D_66 115.6 mm to (482.6, 166.8), turned to 270 degrees
- moved C92 114.9 mm to (476.2, 180.8), turned to 270 degrees
- moved D_65 114.7 mm to (463.4, 166.8), turned to 270 degrees
- moved C91 108.3 mm to (457.1, 180.9), turned to 270 degrees
- moved D_67 104.4 mm to (444.5, 185.7), turned to 270 degrees
- moved D_68 100.1 mm to (463.6, 185.7), turned to 270 degrees
- moved D_69 100.0 mm to (482.6, 185.7), turned to 270 degrees
- moved R3 97.3 mm to (499.1, 161.8), turned to 270 degrees
- moved C94 89.9 mm to (476.1, 218.9), turned to 270 degrees
- moved R1 77.6 mm to (512.2, 208.2)
- moved LED14 66.0 mm to (467.7, 176.0)
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Connections:
- C1 pad 1: VDD -> VCC
- C1 pad 2: GNDA -> GND
- C11 pad 1: VDD -> VCC
- C11 pad 2: GNDA -> GND
- C13 pad 1: VDD -> VCC
- C13 pad 2: GNDA -> GND
- C14 pad 1: VDD -> VCC
- C14 pad 2: GNDA -> GND
- C15 pad 1: VDD -> VCC
- C15 pad 2: GNDA -> GND
- C16 pad 1: VDD -> VCC
- C16 pad 2: GNDA -> GND
- C17 pad 1: VDD -> VCC
- C17 pad 2: GNDA -> GND
- C2 pad 1: VDD -> VCC
- C2 pad 2: GNDA -> GND
- C3 pad 1: VDD -> VCC
- C3 pad 2: GNDA -> GND
- C4 pad 1: VDD -> VCC
- C4 pad 2: GNDA -> GND
- C5 pad 1: VDD -> VCC
- C5 pad 2: GNDA -> GND
- C86 pad 1: VDD -> VCC
- C86 pad 2: GNDA -> GND
- J2 pad A: VDD -> VCC
- J2 pad B: GNDA -> GND
- LED1 pad 1: VDD -> VCC
- LED1 pad 3: GNDA -> GND
- LED13 pad 1: VDD -> VCC
- LED13 pad 3: GNDA -> GND
- LED14 pad 1: VDD -> VCC
- LED14 pad 3: GNDA -> GND
- LED15 pad 1: VDD -> VCC
- LED15 pad 3: GNDA -> GND
- LED16 pad 1: VDD -> VCC
- LED16 pad 3: GNDA -> GND
- LED17 pad 1: VDD -> VCC
- LED17 pad 3: GNDA -> GND
- LED18 pad 1: VDD -> VCC
- LED18 pad 3: GNDA -> GND
- LED2 pad 1: VDD -> VCC
- LED2 pad 3: GNDA -> GND
- LED3 pad 1: VDD -> VCC
- LED3 pad 3: GNDA -> GND
- LED4 pad 1: VDD -> VCC
- LED4 pad 3: GNDA -> GND
- LED41 pad 1: GND -> VCC
- LED41 pad 2: Net-(LED27-Pad2) -> Net-(LED41-Pad2)
- LED41 pad 3: VCC -> GND
- LED41 pad 4: Net-(LED41-Pad4) -> Net-(LED27-Pad2)
- LED5 pad 1: VDD -> VCC
- LED5 pad 3: GNDA -> GND
- LED55 pad 4: Net-(LED41-Pad4) -> Net-(LED41-Pad2)
- LED6 pad 1: VDD -> VCC
- LED6 pad 3: GNDA -> GND
- OL1 pad 3: VDD -> VCC
- OL1 pad 4: GNDA -> GND
- R1 pad 2: Net-(LED18-Pad4) -> Net-(LED100-Pad4)
- RSW1 pad 2: GNDA -> GND
- U1 pad 21: VDD -> VCC
- U1 pad 23: GNDA -> GND
- U1 pad 3: GNDA -> GND
- U1 pad 4: GNDA -> GND
Routing:
- net VDD: track 1247.7 -> 0.00 mm, vias 56 -> 0
- net GND: track 1027.0 -> 2191.6 mm, vias 9 -> 12
- net VCC: track 1013.2 -> 2097.1 mm, vias 22 -> 29
- net GNDA: track 1023.2 -> 0.00 mm, vias 22 -> 0
- net col0_R: track 273.0 -> 104.5 mm, vias 10 -> 8
- net data_R: track 157.1 -> 0.00 mm
- net col1_R: track 225.9 -> 70.7 mm, vias 8 -> 6
- net row1_R: track 168.1 -> 317.5 mm, vias 18 -> 0
- net SCL_R: track 135.0 -> 0.00 mm, vias 3 -> 0
- net col2_R: track 203.3 -> 68.6 mm, vias 8 -> 6
- net col6_R: track 134.3 -> 0.00 mm, vias 10 -> 0
- net row0_R: track 161.4 -> 295.5 mm, vias 13 -> 0
- net SDA_R: track 131.2 -> 0.00 mm, vias 6 -> 0
- net row2_R: track 178.8 -> 301.9 mm, vias 18 -> 2
- net col3_R: track 206.6 -> 89.2 mm, vias 10 -> 8
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Other:
- board size 402.1 x 110.2 mm -> 402.1 x 110.3 mm

Commit message: wiring done, added more leds, figuring out best place for oled
Parts:
- added C102: 0.1uF, Capacitor_SMD:C_0603_1608Metric_Pad1.08x0.95mm_HandSolder, B.Cu at (160.9, 176.0)
- added C103: 0.1uF, Capacitor_SMD:C_0603_1608Metric_Pad1.08x0.95mm_HandSolder, B.Cu at (170.4, 233.3)
- added LED102: YS-SK6812MINI-E, kbd:YS-SK6812MINI-E_underglow, F.Cu at (155.9, 176.1)
- added LED103: YS-SK6812MINI-E, kbd:YS-SK6812MINI-E_underglow, F.Cu at (165.4, 233.2)
- moved OL2 61.4 mm to (281.8, 193.7), turned to 0 degrees
- moved OL1 47.5 mm to (302.8, 193.8), turned to 0 degrees
- moved RSW1 35.4 mm to (547.5, 206.5)
- moved C101 35.3 mm to (525.0, 195.1)
- moved LED101 35.2 mm to (519.8, 195.1)
- moved C19 33.3 mm to (528.3, 238.0)
- moved K_16 33.3 mm to (523.4, 166.5)
- moved K_33 33.3 mm to (523.4, 185.5)
- moved LED91 33.3 mm to (523.5, 180.8)
- moved C1 33.3 mm to (380.7, 176.0)
- moved C13 33.3 mm to (337.8, 214.1)
- moved C14 33.3 mm to (506.0, 176.0)
- moved C15 33.3 mm to (347.3, 233.0)
- moved C2 33.3 mm to (418.8, 175.9)
- moved C23 33.3 mm to (390.1, 161.8)
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Connections:
- C101 pad 2: Net-(C101-Pad2) -> GND
- LED19 pad 4: Net-(LED19-Pad4) -> Net-(LED103-Pad2)
- LED24 pad 2: Net-(LED19-Pad4) -> Net-(LED103-Pad4)
- LED7 pad 4: Net-(LED7-Pad4) -> Net-(LED102-Pad2)
- R2 pad 2: Net-(LED7-Pad4) -> Net-(LED102-Pad4)
- U1 pad 27: col8_R -> col10_R
- U1 pad 29: col10_R -> col8_R
Routing:
- net VCC: track 2097.1 -> 2609.7 mm, vias 29 -> 65
- net col2_R: track 68.6 -> 326.7 mm, vias 6 -> 8
- net col0_R: track 104.5 -> 334.1 mm, vias 8 -> 11
- net col3_R: track 89.2 -> 307.6 mm, vias 8 -> 10
- net col1_R: track 70.7 -> 289.2 mm, vias 6 -> 9
- net GND: track 2191.6 -> 2397.7 mm
- net col4_R: track 95.1 -> 287.3 mm, vias 8 -> 11
- net col6_R: track 0.00 -> 179.7 mm, vias 0 -> 9
- net col5_R: track 43.5 -> 195.4 mm, vias 4 -> 6
- net col8_R: track 0.00 -> 141.1 mm, vias 0 -> 6
- net col9_R: track 0.00 -> 112.9 mm, vias 0 -> 7
- net col7_R: track 58.5 -> 166.3 mm, vias 2 -> 6
- net col10_R: track 0.00 -> 94.4 mm, vias 0 -> 4
- net Net-(LED14-Pad2): track 0.00 -> 49.4 mm, vias 0 -> 2
- net BACKLIGHT_LED_R: track 0.00 -> 46.6 mm, vias 0 -> 1
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Other:
- board size 402.1 x 110.3 mm -> 435.4 x 110.3 mm

Commit message: wired up and still thinking
Parts:
- J1, J2: footprint kbd:MJ-4PP-9_1side -> mj-4pp-9:MJ-4PP-9; moved to F.Cu
- RSW1, RSW2: footprint kbd:ResetSW_1side -> Button_Switch_SMD:SW_SPST_TL3342
- moved OL1 221.1 mm to (521.2, 159.4), turned to 180 degrees
- moved OL2 176.3 mm to (108.8, 159.4), turned to 180 degrees
- moved J2 73.4 mm to (256.5, 112.6), turned to 270 degrees
- moved RSW1 65.6 mm to (521.2, 146.4)
- moved RSW2 59.4 mm to (108.9, 146.4)
- moved U2 57.0 mm to (108.9, 123.8)
- moved U1 56.9 mm to (521.5, 123.8)
- moved K_16 55.9 mm to (501.2, 115.2)
- moved C18 55.9 mm to (141.2, 162.8)
- moved C38 55.9 mm to (320.3, 129.6)
- moved C39 55.9 mm to (339.3, 129.6)
- moved C45 55.9 mm to (138.6, 129.5)
- moved C65 55.9 mm to (353.6, 167.6)
- moved C83 55.9 mm to (200.5, 129.5)
- moved C92 55.9 mm to (487.3, 129.5)
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Routing:
- net data_R: track 0.00 -> 233.8 mm, vias 0 -> 2
- net SCL_L: track 132.6 -> 47.5 mm, vias 0 -> 1
- net SDA_L: track 131.1 -> 53.9 mm, vias 0 -> 1
- net row4_R: track 225.0 -> 301.3 mm, vias 0 -> 2
- net GND: track 2397.7 -> 2473.5 mm, vias 12 -> 14
- net SDA_R: track 0.00 -> 57.6 mm, vias 0 -> 1
- net SCL_R: track 0.00 -> 55.9 mm, vias 0 -> 1
- net col2_R: track 326.7 -> 274.8 mm, vias 8 -> 9
- net VCC: track 2609.7 -> 2655.9 mm, vias 65 -> 64
- net reset_L: track 0.00 -> 42.3 mm
- net data_L: track 150.0 -> 170.4 mm, vias 1 -> 2
- net reset_R: track 0.00 -> 6.30 mm
- net row4_L: track 194.7 -> 200.1 mm
- net col0_R: track 334.1 -> 338.0 mm
- net row2_L: track 186.6 -> 190.2 mm
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Other:
- board size 435.4 x 110.3 mm -> 432.9 x 98.3 mm
