File: bakekujira.kicad_pcb (KiCad board)
At the start: 2 copper layers, 405.8 x 120.8 mm, 370 parts, among them J1 MJ-4PP-9, J2 MJ-4PP-9, U1 proton_c, U2 proton_c

Commit message: added images, readme, added holes for acrylic to cover the proton-c
Parts:
- added G***: LOGO, bake-kujira:bakekujira-kana, F.Cu at (228.4, 86.2)
- added G***: LOGO, bake-kujira:bakekujira-logo-large, F.Cu at (291.2, 87.7)
- added REF**: Breakaway_Tabs, kbd:Breakaway_Tabs, F.Cu at (44.5, 132.2)
- added REF**: Breakaway_Tabs, kbd:Breakaway_Tabs, F.Cu at (134.5, 132.2)
- added REF**: Breakaway_Tabs, kbd:Breakaway_Tabs, F.Cu at (248.7, 132.2)
- added REF**: Breakaway_Tabs, kbd:Breakaway_Tabs, F.Cu at (403.4, 132.2)
- added Ref**: Val**, kbd:M2_HOLE_v2, F.Cu at (409.2, 100.9)
- added Ref**: Val**, kbd:M2_HOLE_v2, F.Cu at (388.3, 40.2)
- added Ref**: Val**, kbd:M2_HOLE_v2, F.Cu at (416.8, 123.6)
- added Ref**: Val**, kbd:M2_HOLE_v2, F.Cu at (346.5, 125.2)
- added Ref**: Val**, kbd:M2_HOLE_v2, F.Cu at (344.1, 46.0)
- added Ref**: Val**, kbd:M2_HOLE_v2, F.Cu at (68.8, 55.9)
- added Ref**: Val**, kbd:M2_HOLE_v2, F.Cu at (173.9, 122.9)
- added Ref**: Val**, kbd:M2_HOLE_v2, F.Cu at (202.6, 123.0)
- added Ref**: Val**, kbd:M2_HOLE_v2, F.Cu at (216.1, 93.3)
- added Ref**: Val**, kbd:M2_HOLE_v2, F.Cu at (207.3, 74.3)
- added Ref**: Val**, kbd:M2_HOLE_v2, F.Cu at (191.6, 55.2)
- added Ref**: Val**, kbd:M2_HOLE_v2, F.Cu at (424.4, 101.0)
- added Ref**: Val**, kbd:M2_HOLE_v2, F.Cu at (156.2, 54.4)
- added Ref**: Val**, kbd:M2_HOLE_v2, F.Cu at (39.0, 101.0)
- added Ref**: Val**, kbd:M2_HOLE_v2, F.Cu at (23.8, 101.0)
- added Ref**: Val**, kbd:M2_HOLE_v2, F.Cu at (159.7, 74.2)
- added Ref**: Val**, kbd:M2_HOLE_v2, F.Cu at (387.0, 81.4)
- added Ref**: Val**, kbd:M2_HOLE_v2, F.Cu at (296.7, 125.2)
- added Ref**: Val**, kbd:M2_HOLE_v2, F.Cu at (89.0, 118.6)
- added Ref**: Val**, kbd:M2_HOLE_v2, F.Cu at (31.4, 123.6)
Routing:
- net reset_R: track 64.9 -> 57.9 mm
- net row4_R: track 308.8 -> 314.6 mm
- net VCC: track 1084.1 -> 1087.3 mm
- net Net-(LED7-Pad4): track 39.6 -> 41.6 mm
- net col9_R: track 102.6 -> 104.4 mm
- net Net-(LED47-Pad2): track 33.5 -> 34.8 mm
- net Net-(LED60-Pad2): track 26.9 -> 25.7 mm
- net col6_L: track 310.8 -> 309.6 mm
- net GNDA: track 1502.4 -> 1503.2 mm
- net Net-(LED31-Pad2): track 33.1 -> 33.8 mm
- net VDD: track 1623.0 -> 1622.3 mm
- net GND: track 968.9 -> 969.4 mm

Commit message: fixing split and rgb source
Parts:
- removed G***: LOGO, bake-kujira:bakekujira-kana
- removed G***: LOGO, bake-kujira:bakekujira-logo-large
- removed REF** (x7), REF1: Breakaway_Tabs, kbd:Breakaway_Tabs
- removed Ref** (x20): Val**, kbd:M2_HOLE_v2
- moved R1 20.0 mm to (404.3, 77.8)
Connections:
- U1 pad 5V: Net-(U1-Pad5V) -> VDD
- U1 pad A3|5v: VDD -> LED_R
- U1 pad B0: LED_R -> Net-(U1-PadB0)
- U2 pad 5V: Net-(U2-Pad5V) -> VCC
- U2 pad A3|5v: VCC -> LED_L
- U2 pad B0: LED_L -> Net-(U2-PadB0)
Routing:
- net LED_R: track 2.83 -> 38.2 mm, vias 0 -> 1
- net LED_L: track 14.4 -> 47.0 mm, vias 0 -> 1
- net Net-(LED25-Pad4): track 38.5 -> 16.7 mm
- net VCC: track 1087.3 -> 1097.1 mm, vias 29 -> 31
- net row4_R: track 314.6 -> 323.6 mm
- net SDA_L: track 44.2 -> 50.2 mm, vias 0 -> 1
- net SCL_L: track 42.9 -> 47.7 mm, vias 0 -> 1
- net row3_R: track 319.1 -> 321.9 mm
- net reset_L: track 58.2 -> 57.0 mm
- net VDD: track 1622.3 -> 1623.1 mm, vias 38 -> 39
- net Net-(U2-PadB0): track 0.00 -> 0.73 mm

Commit message: updated readme
Parts:
- added G***: LOGO, bake-kujira:bakekujira-logo-large, F.Cu at (290.2, 87.0)
- added G***: LOGO, bake-kujira:onigakuen-keylab-square_15mmx15mm, F.Cu at (31.4, 126.0)
- added G***: LOGO, bake-kujira:onigakuen-keylab-square_15mmx15mm, F.Cu at (416.8, 126.0)
- added G***: LOGO, bake-kujira:bakekujira-kana, F.Cu at (228.4, 85.7)
- added REF**: Breakaway_Tabs, onigaku:Breakaway_Tabs, F.Cu at (44.4, 132.2)
- added REF**: Breakaway_Tabs, onigaku:Breakaway_Tabs, F.Cu at (134.5, 132.2)
- added REF**: Breakaway_Tabs, onigaku:Breakaway_Tabs, F.Cu at (248.7, 132.3)
- added REF**: Breakaway_Tabs, onigaku:Breakaway_Tabs, F.Cu at (403.3, 132.2)
- added REF**: Breakaway_Tabs, onigaku:Breakaway_Tabs, F.Cu at (403.5, 35.1)
- added REF**: Breakaway_Tabs, onigaku:Breakaway_Tabs, F.Cu at (199.3, 35.1)
- added REF**: Breakaway_Tabs, onigaku:Breakaway_Tabs, F.Cu at (166.6, 35.1)
- added REF**: Breakaway_Tabs, onigaku:Breakaway_Tabs, F.Cu at (44.5, 35.1)
Other:
- board text removed: "bake kujira v1.0 papadakko alfredy@gmail.com"

Commit message: readme and small udpates
Parts:
- removed G***: LOGO, bake-kujira:bakekujira-logo-large
- removed G*** (x2): LOGO, bake-kujira:onigakuen-keylab-square_15mmx15mm
- removed G***: LOGO, bake-kujira:bakekujira-kana
- removed REF** (x8): Breakaway_Tabs, onigaku:Breakaway_Tabs
- SW_1, SW_10, SW_11, SW_12, SW_13, SW_14, SW_15, SW_16, SW_17, SW_18, SW_19, SW_2, SW_20, SW_21, SW_22, SW_23, SW_24, SW_26, SW_27, SW_28, SW_3, SW_30, SW_31, SW_32, SW_33, SW_34, SW_35, SW_36, SW_37, SW_38, SW_39, SW_4, SW_40, SW_43, SW_44, SW_45, SW_46, SW_47, SW_48, SW_49, SW_5, SW_50, SW_51, SW_52, SW_54, SW_56, SW_57, SW_58, SW_59, SW_6, SW_60, SW_66, SW_67, SW_68, SW_8, SW_9: footprint kbd:CherryMX_Hotswap -> onigaku:CherryMX_Hotswap
- SW_25, SW_29: footprint kbd:CherryMX_Hotswap_1.5u -> onigaku:CherryMX_Hotswap_1.5u
- SW_41, SW_55: footprint kbd:CherryMX_Hotswap_2.25u_North -> onigaku:CherryMX_Hotswap_2.25u_North
- SW_42: footprint kbd:CherryMX_Hotswap_1.75u -> onigaku:CherryMX_Hotswap_1.75u
- SW_53: footprint kbd:CherryMX_Hotswap_2.75u_North -> onigaku:CherryMX_Hotswap_2.75u_North
- SW_61: footprint kbd:CherryMX_Hotswap_2.75u_North_reversed_stabilizers -> onigaku:CherryMX_Hotswap_2.75u_North_reversed_stabilizers
- SW_62, SW_63, SW_64, SW_65, SW_69, SW_70, SW_71, SW_72: footprint kbd:CherryMX_Hotswap_1.25u_North -> onigaku:CherryMX_Hotswap_1.25u_North
- SW_7: footprint kbd:CherryMX_Hotswap_2u_North -> onigaku:CherryMX_Hotswap_2u_North
- SW_73: footprint kbd:CherryMX_Hotswap_2.25u_North_reversed_stabilizers -> onigaku:CherryMX_Hotswap_2.25u_North_reversed_stabilizers
