File: bakekujira.sch (KiCad schematic (older format))
At the start: 366 parts, among them J1 MJ-4PP-9, J2 MJ-4PP-9, U1 proton_c, U2 proton_c

Commit message: added images, readme, added holes for acrylic to cover the proton-c
Parts:
- LED1, LED10, LED100, LED101, LED102, LED103, LED104, LED11, LED12, LED13, LED14, LED15, LED16, LED17, LED18, LED19, LED2, LED20, LED21, LED22, LED23, LED24, LED25, LED26, LED27, LED28, LED29, LED3, LED30, LED31, LED32, LED33, LED34, LED35, LED36, LED37, LED38, LED39, LED4, LED40, LED41, LED42, LED43, LED44, LED45, LED46, LED47, LED48, LED49, LED5, LED50, LED51, LED52, LED53, LED54, LED55, LED56, LED57, LED58, LED59, LED6, LED60, LED61, LED62, LED63, LED64, LED65, LED66, LED67, LED68, LED69, LED7, LED70, LED71, LED72, LED73, LED74, LED75, LED76, LED77, LED78, LED79, LED8, LED80, LED81, LED82, LED83, LED84, LED85, LED86, LED87, LED88, LED89, LED9, LED90, LED91, LED92, LED93, LED94, LED95, LED96, LED97, LED98, LED99: symbol kbd:YS-SK6812MINI-E -> bakekujira-rescue:YS-SK6812MINI-E-kbd
- OL1, OL2: symbol kbd:OLED -> bakekujira-rescue:OLED-kbd
- RSW1, RSW2: symbol kbd:SW_PUSH -> bakekujira-rescue:SW_PUSH-kbd
Connections:
- wire segments 703 -> 702

Commit message: fixing split and rgb source
Connections:
- net LED_L: now also U2.A3|5v (A3(5v_shifted)); no longer U2.B0 (PB0)
- net LED_R: now also U1.A3|5v (A3(5v_shifted)); no longer U1.B0 (PB0)
- net VCC: now also U2.5V (VBUS(5V_RAW)); no longer U2.A3|5v (A3(5v_shifted))
- net VDD: now also U1.5V (VBUS(5V_RAW)); no longer U1.A3|5v (A3(5v_shifted))
- no-connect marks 11 -> 7
Other:
- moved on the sheet: C73, LED73
Changed lines of the file:
@@
 	1    0    0    -1
 $EndComp
-Text GLabel 13425 2275 0    50   Input ~ 0
+Text GLabel 14625 875  1    50   Input ~ 0
 LED_R
-Text GLabel 9925 2300 0    50   Input ~ 0
+Text GLabel 11125 900  1    50   Input ~ 0
 LED_L
 Text GLabel 1475 9050 0    50   Input ~ 0
@@
 Text GLabel 15475 1875 2    47   Input ~ 0
 col7_R
-NoConn ~ 11975 1200
 NoConn ~ 9925 1300
 NoConn ~ 13425 1275
-NoConn ~ 15475 1175
 Text GLabel 14300 4925 2    50   Input ~ 0
 data_R
@@
 L power:VCC #PWR05
 U 1 1 604F807F
-P 11125 900
-F 0 "#PWR05" H 11125 750 50  0001 C CNN
-F 1 "VCC" H 11125 1050 50  0000 C CNN
-F 2 "" H 11125 900 50  0001 C CNN
-F 3 "" H 11125 900 50  0001 C CNN
-	1    11125 900
-	1    0    0    -1
+P 11975 1200
+F 0 "#PWR05" H 11975 1050 50  0001 C CNN
+F 1 "VCC" H 11975 1350 50  0000 C CNN
+F 2 "" H 11975 1200 50  0001 C CNN
+F 3 "" H 11975 1200 50  0001 C CNN
+	1    11975 1200
+	0    1    1    0
 $EndComp
 $Comp
@@
 $EndComp
 Connection ~ 2775 10425
-Connection ~ 2975 12075
+Connection ~ 2975 12975
 $Comp
 L power:VCC #PWR0106
 U 1 1 604F8167
-P 2975 12075
-F 0 "#PWR0106" H 2975 11925 50  0001 C CNN
-F 1 "VCC" H 2975 12225 50  0000 C CNN
-F 2 "" H 2975 12075 50  0001 C CNN
-F 3 "" H 2975 12075 50  0001 C CNN
-	1    2975 12075
+P 2975 12975
+F 0 "#PWR0106" H 2975 12825 50  0001 C CNN
+F 1 "VCC" H 2975 13125 50  0000 C CNN
+F 2 "" H 2975 12975 50  0001 C CNN
+F 3 "" H 2975 12975 50  0001 C CNN
+	1    2975 12975
 	1    0    0    -1
 $EndComp
@@
 L power:GND #PWR0113
 U 1 1 6ED98F0A
-P 2975 12275
-F 0 "#PWR0113" H 2975 12025 50  0001 C CNN
-F 1 "GND" H 2975 12125 50  0000 C CNN
-F 2 "" H 2975 12275 50  0001 C CNN
-F 3 "" H 2975 12275 50  0001 C CNN
-	1    2975 12275
+P 2975 13175
+F 0 "#PWR0113" H 2975 12925 50  0001 C CNN
+F 1 "GND" H 2975 13025 50  0000 C CNN
+F 2 "" H 2975 13175 50  0001 C CNN
+F 3 "" H 2975 13175 50  0001 C CNN
+	1    2975 13175
 	1    0    0    -1
 $EndComp
@@
 L bakekujira-rescue:YS-SK6812MINI-E-kbd LED73
 U 1 1 604F8069
-P 3275 12075
-F 0 "LED73" H 3619 12105 29  0000 L CNN
-F 1 "YS-SK6812MINI-E" H 3619 12046 29  0000 L CNN
-F 2 "kbd:YS-SK6812MINI-E" H 3375 11825 50  0001 C CNN
-F 3 "" H 3375 11825 50  0001 C CNN
-	1    3275 12075
+P 3275 12975
+F 0 "LED73" H 3619 13005 29  0000 L CNN
+F 1 "YS-SK6812MINI-E" H 3619 12946 29  0000 L CNN
+F 2 "kbd:YS-SK6812MINI-E" H 3375 12725 50  0001 C CNN
+F 3 "" H 3375 12725 50  0001 C CNN
+	1    3275 12975
 	0    -1   -1   0
 $EndComp
@@
 L Device:C_Small C73
 U 1 1 62E67A22
-P 2975 12175
-F 0 "C73" H 2985 12245 50  0000 L CNN
-F 1 "0.1uF" H 2985 12095 50  0000 L CNN
-F 2 "Capacitor_SMD:C_0603_1608Metric_Pad1.08x0.95mm_HandSolder" H 2975 12175 50  0001 C CNN
-F 3 "~" H 2975 12175 50  0001 C CNN
-	1    2975 12175
+P 2975 13075
+F 0 "C73" H 2985 13145 50  0000 L CNN
+F 1 "0.1uF" H 2985 12995 50  0000 L CNN
+F 2 "Capacitor_SMD:C_0603_1608Metric_Pad1.08x0.95mm_HandSolder" H 2975 13075 50  0001 C CNN
+F 3 "~" H 2975 13075 50  0001 C CNN
+	1    2975 13075
 	1    0    0    -1
 $EndComp
@@
 Connection ~ 2175 11250
 Wire Wire Line
-	3275 13550 3275 12375
+	3275 13550 3275 13275
 Wire Wire Line
-	3275 10725 3275 11775
+	3275 10725 3275 12675
 Wire Wire Line
 	3275 9875 3275 10125
@@
 	2175 13850 2175 14525
 Wire Wire Line
-	3575 13850 3575 12075
-Connection ~ 3575 12075
+	3575 13850 3575 12975
+Connection ~ 3575 12975
 Wire Wire Line
 	2475 12375 2475 13550
@@
 	2175 12025 2175 12075
 Wire Wire Line
-	3575 12025 3575 12075
-Wire Wire Line
 	2175 11250 2175 12075
-Wire Wire Line
-	3575 10425 3575 12075
 Connection ~ 3575 13850
 Wire Wire Line
@@
 	-1   0    0    1
 $EndComp
-Wire Wire Line
-	10625 5150 10925 5150
 NoConn ~ 10925 4900
 Wire Wire Line
@@
 L power:VDD #PWR04
 U 1 1 60DB99D7
-P 14625 875
-F 0 "#PWR04" H 14625 725 50  0001 C CNN
-F 1 "VDD" H 14625 1025 50  0000 C CNN
-F 2 "" H 14625 875 50  0001 C CNN
-F 3 "" H 14625 875 50  0001 C CNN
-	1    14625 875
-	1    0    0    -1
+P 15475 1175
+F 0 "#PWR04" H 15475 1025 50  0001 C CNN
+F 1 "VDD" H 15475 1325 50  0000 C CNN
+F 2 "" H 15475 1175 50  0001 C CNN
+F 3 "" H 15475 1175 50  0001 C CNN
+	1    15475 1175
+	0    1    1    0
 $EndComp
 $Comp
@@
 $EndComp
 $Comp
-L power:VCC #PWR0179
-U 1 1 608116AC
-P 10625 5150
-F 0 "#PWR0179" H 10625 5000 50  0001 C CNN
-F 1 "VCC" H 10625 5300 50  0000 C CNN
-F 2 "" H 10625 5150 50  0001 C CNN
-F 3 "" H 10625 5150 50  0001 C CNN
-	1    10625 5150
-	0    -1   -1   0
-$EndComp
-$Comp
-L power:VDD #PWR0180
-U 1 1 60AA1A07
-P 14300 4775
-F 0 "#PWR0180" H 14300 4625 50  0001 C CNN
-F 1 "VDD" H 14300 4925 50  0000 C CNN
-F 2 "" H 14300 4775 50  0001 C CNN
-F 3 "" H 14300 4775 50  0001 C CNN
-	1    14300 4775
-	0    1    1    0
-$EndComp
-$Comp
 L proton_c:proton_c U1
 U 1 1 60CC6B5A
@@
 Text GLabel 12675 6000 3    50   Input ~ 0
 data_R
-NoConn ~ 11975 1500
-NoConn ~ 15475 1475
 Text GLabel 15475 1775 2    50   Input ~ 0
 col8_R
+Wire Wire Line
+	3575 12925 3575 12975
+Wire Wire Line
+	3575 10425 3575 12975
+Wire Wire Line
+	11975 1500 12275 1500
+Wire Wire Line
+	10425 5150 10925 5150
+Wire Wire Line
+	15900 1475 15475 1475
+$Comp
+L power:VCC #PWR0179
+U 1 1 609B34A3
+P 10425 5150
+F 0 "#PWR0179" H 10425 5000 50  0001 C CNN
+F 1 "VCC" H 10425 5300 50  0000 C CNN
+F 2 "" H 10425 5150 50  0001 C CNN
+F 3 "" H 10425 5150 50  0001 C CNN
+	1    10425 5150
+	0    -1   -1   0
+$EndComp
+$Comp
+L power:VDD #PWR0180
+U 1 1 609B3DC1
+P 14300 4775
+F 0 "#PWR0180" H 14300 4625 50  0001 C CNN
+F 1 "VDD" H 14300 4925 50  0000 C CNN
+F 2 "" H 14300 4775 50  0001 C CNN
+F 3 "" H 14300 4775 50  0001 C CNN
+	1    14300 4775
+	0    1    1    0
+$EndComp
 $EndSCHEMATC

Commit message: updated readme
Changed lines of the file:
@@
 	3575 10425 3575 12975
 Wire Wire Line
-	11975 1500 12275 1500
-Wire Wire Line
 	10425 5150 10925 5150
-Wire Wire Line
-	15900 1475 15475 1475
 $Comp
 L power:VCC #PWR0179

Commit message: readme and small udpates
Parts:
- SW_1, SW_10, SW_11, SW_12, SW_13, SW_14, SW_15, SW_16, SW_17, SW_18, SW_19, SW_2, SW_20, SW_21, SW_22, SW_23, SW_24, SW_26, SW_27, SW_28, SW_3, SW_30, SW_31, SW_32, SW_33, SW_34, SW_35, SW_36, SW_37, SW_38, SW_39, SW_4, SW_40, SW_43, SW_44, SW_45, SW_46, SW_47, SW_48, SW_49, SW_5, SW_50, SW_51, SW_52, SW_54, SW_56, SW_57, SW_58, SW_59, SW_6, SW_60, SW_66, SW_67, SW_68, SW_8, SW_9: footprint kbd:CherryMX_Hotswap -> onigaku:CherryMX_Hotswap
- SW_25, SW_29: footprint kbd:CherryMX_Hotswap_1.5u -> onigaku:CherryMX_Hotswap_1.5u
- SW_41, SW_55: footprint kbd:CherryMX_Hotswap_2.25u_North -> onigaku:CherryMX_Hotswap_2.25u_North
- SW_42: footprint kbd:CherryMX_Hotswap_1.75u -> onigaku:CherryMX_Hotswap_1.75u
- SW_53: footprint kbd:CherryMX_Hotswap_2.75u_North -> onigaku:CherryMX_Hotswap_2.75u_North
- SW_61: footprint kbd:CherryMX_Hotswap_2.75u_North_reversed_stabilizers -> onigaku:CherryMX_Hotswap_2.75u_North_reversed_stabilizers
- SW_62, SW_63, SW_64, SW_65, SW_69, SW_70, SW_71, SW_72: footprint kbd:CherryMX_Hotswap_1.25u_North -> onigaku:CherryMX_Hotswap_1.25u_North
- SW_7: footprint kbd:CherryMX_Hotswap_2u_North -> onigaku:CherryMX_Hotswap_2u_North
- SW_73: footprint kbd:CherryMX_Hotswap_2.25u_North_reversed_stabilizers -> onigaku:CherryMX_Hotswap_2.25u_North_reversed_stabilizers
