File: kujira/kujira.kicad_pcb (KiCad board)
At the start: 2 copper layers, 405.8 x 111.6 mm, 372 parts, among them J1 MJ-4PP-9, J2 MJ-4PP-9, U1 Elite-C, U2 Elite-C

Commit message: tabs increased width, double checked schematic with keyboard layout dxf/svg
Other:
- board size 405.8 x 111.6 mm -> 405.8 x 119.1 mm

Commit message: moved some leds around, re arranged some traces
Parts:
- removed REF** (x8): Breakaway_Tabs, kbd:Breakaway_Tabs
- SW_54: footprint kbd:CherryMX_Hotswap_2.75u_North -> kbd:CherryMX_Hotswap_2.75u_North_reversed_stabilizers
- SW_63: footprint kbd:CherryMX_Hotswap_2.25u_North -> kbd:CherryMX_Hotswap_2.25u_North_reversed_stabilizers
- moved C19 18.4 mm to (401.4, 117.2)
- moved C4 18.4 mm to (351.3, 55.3)
- moved C67 18.4 mm to (322.8, 98.2)
- moved C75 18.4 mm to (289.4, 117.2)
- moved C77 18.4 mm to (337.1, 117.2)
- moved C9 18.4 mm to (382.5, 117.2)
- moved C94 18.4 mm to (382.5, 98.2)
- moved D_56 18.4 mm to (276.9, 121.9)
- moved D_57 18.4 mm to (300.7, 121.9)
- moved D_58 18.4 mm to (324.5, 121.9)
- moved LED45 18.4 mm to (306.0, 59.9)
- moved LED81 18.4 mm to (308.3, 117.2)
- moved C41 18.4 mm to (272.7, 60.1)
- moved C44 18.4 mm to (334.7, 59.9)
- moved C89 18.4 mm to (382.5, 40.9)
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Routing:
- net VDD: track 1608.0 -> 1631.5 mm
- net GNDA: track 1498.7 -> 1520.4 mm
- net Net-(LED15-Pad4): track 37.8 -> 52.8 mm, vias 2 -> 3
- net col2_R: track 275.3 -> 261.8 mm
- net Net-(LED13-Pad2): track 26.4 -> 35.4 mm
- net Net-(LED13-Pad4): track 32.5 -> 25.5 mm
- net col0_R: track 337.9 -> 343.3 mm
- net col1_R: track 291.4 -> 296.7 mm
- net col10_R: track 95.1 -> 97.2 mm
- net col9_R: track 113.7 -> 115.6 mm
- net col7_R: track 168.2 -> 169.9 mm
- net col5_R: track 188.7 -> 190.3 mm
- net reset_R: track 42.1 -> 43.7 mm
- net col6_L: track 295.7 -> 297.2 mm
- net Net-(LED1-Pad4): track 31.1 -> 29.6 mm
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Other:
- board size 405.8 x 119.1 mm -> 405.8 x 120.8 mm

Commit message: updated rgb lighting based on restrictive pin requirement for underglow and maatrix
Parts:
- removed R1, R2: 500, Resistor_SMD:R_0805_2012Metric_Pad1.20x1.40mm_HandSolder
- moved R4 34.4 mm to (51.1, 73.5), turned to 180 degrees
- moved R3 30.0 mm to (408.4, 70.9), turned to 0 degrees
Connections:
- LED19 pad 2: Net-(LED12-Pad4) -> Net-(LED103-Pad4)
- LED19 pad 4: Net-(LED103-Pad2) -> Net-(LED12-Pad2)
- LED21 pad 2: Net-(LED21-Pad2) -> Net-(LED10-Pad4)
- LED21 pad 4: Net-(LED10-Pad2) -> Net-(LED21-Pad4)
- LED22 pad 2: Net-(LED22-Pad2) -> Net-(LED21-Pad4)
- LED22 pad 4: Net-(LED21-Pad2) -> Net-(LED22-Pad4)
- LED23 pad 2: Net-(LED23-Pad2) -> Net-(LED22-Pad4)
- LED23 pad 4: Net-(LED22-Pad2) -> Net-(LED23-Pad4)
- LED24 pad 2: Net-(LED103-Pad4) -> Net-(LED23-Pad4)
- LED24 pad 4: Net-(LED23-Pad2) -> Net-(LED103-Pad2)
- LED32 pad 4: Net-(LED32-Pad4) -> Net-(LED102-Pad2)
- LED7 pad 2: Net-(LED7-Pad2) -> Net-(LED102-Pad4)
- LED7 pad 4: Net-(LED102-Pad2) -> Net-(LED7-Pad4)
- LED8 pad 2: Net-(LED8-Pad2) -> Net-(LED7-Pad4)
- LED8 pad 4: Net-(LED7-Pad2) -> Net-(LED8-Pad4)
- LED88 pad 4: Net-(LED88-Pad4) -> Net-(LED14-Pad2)
- LED9 pad 2: Net-(LED10-Pad4) -> Net-(LED8-Pad4)
- LED9 pad 4: Net-(LED8-Pad2) -> Net-(LED10-Pad2)
- LED97 pad 4: Net-(LED14-Pad2) -> Net-(LED101-Pad2)
- LED98 pad 2: Net-(LED101-Pad4) -> Net-(LED100-Pad4)
- R3 pad 1: Net-(LED88-Pad4) -> Net-(LED101-Pad4)
- R4 pad 1: Net-(LED32-Pad4) -> Net-(LED12-Pad4)
- U1 pad 25: BACKLIGHT_LED_R -> Net-(U1-Pad25)
- U2 pad 25: BACKLIGHT_LED_L -> Net-(U2-Pad25)
Routing:
- net Net-(U1-Pad25): track 0.00 -> 47.3 mm, vias 0 -> 1
- net BACKLIGHT_LED_R: track 47.3 -> 0.00 mm, vias 1 -> 0
- net Net-(LED23-Pad2): track 46.4 -> 0.00 mm, vias 2 -> 0
- net Net-(LED23-Pad4): track 0.00 -> 37.7 mm, vias 0 -> 2
- net Net-(LED21-Pad4): track 0.00 -> 36.4 mm, vias 0 -> 2
- net Net-(LED22-Pad2): track 35.4 -> 0.00 mm
- net Net-(LED8-Pad4): track 0.00 -> 35.2 mm, vias 0 -> 4
- net Net-(LED7-Pad4): track 0.00 -> 34.5 mm, vias 0 -> 4
- net Net-(LED8-Pad2): track 28.5 -> 0.00 mm, vias 2 -> 0
- net Net-(LED7-Pad2): track 27.5 -> 0.00 mm, vias 2 -> 0
- net LED_R: track 29.9 -> 2.76 mm, vias 1 -> 0
- net Net-(LED22-Pad4): track 0.00 -> 27.0 mm, vias 0 -> 2
- net Net-(LED12-Pad2): track 0.00 -> 25.1 mm, vias 0 -> 2
- net Net-(LED12-Pad4): track 26.6 -> 3.85 mm, vias 2 -> 0
- net Net-(LED103-Pad4): track 39.8 -> 19.6 mm
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