File: kujira/kujira.kicad_pcb (KiCad board)
At the start: 2 copper layers, 405.8 x 120.8 mm, 362 parts, among them J1 MJ-4PP-9, J2 MJ-4PP-9, U1 Elite-C, U2 Elite-C

Commit message: reannotated everything using auto
Parts:
- renumbered C86 to C1, C7 to C10, C79 to C100, C80 to C101, C82 to C102, C81 to C103, C8 to C11, C20 to C12, C21 to C13, C11 to C14, C10 to C15, C18 to C16, C103 to C17, C12 to C18, C22 to C19, C1 to C2, C13 to C20, C14 to C21, C15 to C22, C16 to C23, C17 to C24, C96 to C25, C99 to C26, C100 to C27, C98 to C28, C97 to C29, C2 to C3, C101 to C30, C27 to C31, C28 to C32, C26 to C33, C23 to C34, C24 to C35, C25 to C36, C29 to C37, C88 to C38, C89 to C39, C3 to C4, C90 to C40, C36 to C41, C34 to C42, C35 to C43, C30 to C44, C31 to C45, C32 to C46, C33 to C47, C37 to C48, C38 to C49, C4 to C5, C39 to C50, C40 to C51, C41 to C52, C42 to C53, C43 to C54, C44 to C55, C91 to C56, C92 to C57, C93 to C58, C45 to C59, C5 to C6, C47 to C60, C48 to C61, C83 to C62, C49 to C63, C46 to C64, C50 to C65, C51 to C66, C52 to C67, C53 to C68, C54 to C69, C102 to C7, C55 to C70, C56 to C71, C57 to C72, C69 to C73, C58 to C74, C59 to C75, C84 to C76, C60 to C77, C61 to C78, C63 to C79, C87 to C8, C64 to C80, C65 to C81, C62 to C82, C66 to C83, C67 to C84, C94 to C85, C70 to C86, C71 to C87, C85 to C88, C68 to C89, C6 to C9, C72 to C90, C73 to C91, C74 to C92, C75 to C93, C76 to C94, C77 to C95, C95 to C96, C9 to C97, C19 to C98, C78 to C99, D_66 to D_10, D_8 to D_11, D_9 to D_12, D_10 to D_13, D_11 to D_14, D_12 to D_15, D_13 to D_16, D_14 to D_17, D_15 to D_18, D_16 to D_19, D_17 to D_20, D_18 to D_21, D_19 to D_22, D_20 to D_23, D_21 to D_24, D_22 to D_25, D_67 to D_26, D_68 to D_27, D_69 to D_28, D_23 to D_29, D_24 to D_30, D_25 to D_31, D_26 to D_32, D_27 to D_33, D_28 to D_34, D_29 to D_35, D_30 to D_36, D_31 to D_37, D_32 to D_38, D_33 to D_39, D_34 to D_40, D_35 to D_41, D_36 to D_42, D_37 to D_43, D_38 to D_44, D_39 to D_45, D_40 to D_46, D_41 to D_47, D_42 to D_48, D_43 to D_49, D_44 to D_50, D_45 to D_51, D_46 to D_52, D_47 to D_53, D_70 to D_54, D_48 to D_55, D_49 to D_56, D_50 to D_57, D_51 to D_58, D_52 to D_59, D_53 to D_60, D_54 to D_61, D_55 to D_62, D_56 to D_63, D_57 to D_64, D_58 to D_65, D_71 to D_66, D_72 to D_67, D_73 to D_68, D_59 to D_69, D_60 to D_70, D_61 to D_71, D_62 to D_72, D_63 to D_73, D_64 to D_8, D_65 to D_9, LED9 to LED10, LED84 to LED100, LED86 to LED101, LED85 to LED102, LED87 to LED103, LED10 to LED11, LED21 to LED12, LED22 to LED13, LED6 to LED14, LED13 to LED15, LED15 to LED16, LED16 to LED17, LED17 to LED18, LED18 to LED19, LED96 to LED20, LED99 to LED21, LED100 to LED22, LED98 to LED23, LED97 to LED24, LED101 to LED25, LED12 to LED26, LED19 to LED27, LED103 to LED28, LED24 to LED29, LED23 to LED30, LED25 to LED31, LED26 to LED32, LED27 to LED33, LED28 to LED34, LED29 to LED35, LED30 to LED36, LED31 to LED37, LED11 to LED38, LED20 to LED39, LED88 to LED40, LED32 to LED41, LED33 to LED42, LED34 to LED43, LED35 to LED44, LED36 to LED45, LED37 to LED46, LED38 to LED47, LED39 to LED48, LED40 to LED49, LED41 to LED50, LED42 to LED51, LED43 to LED52, LED44 to LED53, LED45 to LED54, LED46 to LED55, LED89 to LED56, LED90 to LED57, LED91 to LED58, LED47 to LED59, LED14 to LED6, LED48 to LED60, LED49 to LED61, LED50 to LED62, LED51 to LED63, LED52 to LED64, LED53 to LED65, LED54 to LED66, LED55 to LED67, LED56 to LED68, LED57 to LED69, LED102 to LED7, LED58 to LED70, LED59 to LED71, LED60 to LED72, LED72 to LED73, LED61 to LED74, LED62 to LED75, LED63 to LED76, LED64 to LED77, LED65 to LED78, LED66 to LED79, LED7 to LED8, LED67 to LED80, LED68 to LED81, LED69 to LED82, LED70 to LED83, LED71 to LED84, LED92 to LED85, LED73 to LED86, LED74 to LED87, LED75 to LED88, LED76 to LED89, LED8 to LED9, LED77 to LED90, LED78 to LED91, LED79 to LED92, LED80 to LED93, LED81 to LED94, LED82 to LED95, LED93 to LED96, LED94 to LED97, LED95 to LED98, LED83 to LED99, R3 to R1, R4 to R2, K_16 to SW_10, SW_8 to SW_11, SW_9 to SW_12, SW_10 to SW_13, SW_11 to SW_14, SW_12 to SW_15, SW_13 to SW_16, SW_14 to SW_17, SW_15 to SW_18, SW_16 to SW_19, SW_17 to SW_20, SW_18 to SW_21, SW_19 to SW_22, SW_20 to SW_23, SW_21 to SW_24, SW_22 to SW_25, K_31 to SW_26, K_32 to SW_27, K_33 to SW_28, SW_23 to SW_29, SW_24 to SW_30, SW_25 to SW_31, SW_26 to SW_32, SW_27 to SW_33, SW_28 to SW_34, SW_29 to SW_35, SW_30 to SW_36, SW_31 to SW_37, SW_32 to SW_38, SW_33 to SW_39, SW_34 to SW_40, SW_35 to SW_41, SW_36 to SW_42, SW_37 to SW_43, SW_38 to SW_44, SW_39 to SW_45, SW_40 to SW_46, SW_41 to SW_47, SW_42 to SW_48, SW_43 to SW_49, SW_44 to SW_50, SW_45 to SW_51, SW_46 to SW_52, SW_47 to SW_53, K_59 to SW_54, SW_48 to SW_55, SW_49 to SW_56, SW_50 to SW_57, SW_51 to SW_58, SW_52 to SW_59, SW_53 to SW_60, SW_54 to SW_61, SW_55 to SW_62, SW_56 to SW_63, SW_57 to SW_64, SW_58 to SW_65, K_68 to SW_66, K_69 to SW_67, K_70 to SW_68, SW_59 to SW_69, SW_60 to SW_70, SW_61 to SW_71, SW_62 to SW_72, SW_63 to SW_73, K_14 to SW_8, K_15 to SW_9

Commit message: flipped elite-cs, added extra LED
Parts:
- added C104: 0.1uF, Capacitor_SMD:C_0603_1608Metric_Pad1.08x0.95mm_HandSolder, B.Cu at (238.3, 55.3)
- added LED104: YS-SK6812MINI-E, kbd:YS-SK6812MINI-E_underglow, F.Cu at (233.0, 55.3)
- U1, U2: moved to B.Cu
- moved C22 15.1 mm to (222.1, 112.4)
- moved LED16 15.1 mm to (217.1, 112.4)
- moved R1 14.7 mm to (423.2, 71.1)
- moved LED2 12.4 mm to (261.3, 55.2)
- moved C2 12.4 mm to (266.3, 55.3)
- moved C1 9.52 mm to (206.2, 55.1)
- moved LED1 9.52 mm to (201.2, 55.2)
- moved C3 4.06 mm to (296.0, 55.1)
- moved LED3 4.06 mm to (291.0, 55.2)
Connections:
- LED2 pad 4: Net-(LED1-Pad2) -> Net-(LED104-Pad2)
Routing:
- net Net-(U1-Pad25): track 47.3 -> 0.00 mm, vias 1 -> 0
- net row0_L: track 223.7 -> 182.1 mm, vias 2 -> 1
- net Net-(LED104-Pad2): track 0.00 -> 28.1 mm, vias 0 -> 2
- net row1_L: track 180.2 -> 154.5 mm, vias 2 -> 1
- net col5_L: track 245.7 -> 265.3 mm, vias 8 -> 10
- net col6_L: track 297.2 -> 314.4 mm, vias 9 -> 11
- net Net-(LED16-Pad4): track 52.8 -> 36.1 mm, vias 3 -> 2
- net col2_L: track 152.3 -> 168.6 mm
- net col1_L: track 126.2 -> 142.4 mm
- net row3_R: track 304.4 -> 320.6 mm
- net row2_R: track 297.1 -> 312.8 mm
- net VCC: track 1056.3 -> 1071.9 mm
- net Net-(LED15-Pad4): track 25.5 -> 41.0 mm
- net LED_L: track 29.7 -> 14.4 mm, vias 1 -> 0
- net col0_L: track 106.2 -> 121.4 mm
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
Commit message: why are my breakaway tabs missing
Parts:
- added REF**: Breakaway_Tabs, kbd:Breakaway_Tabs, F.Cu at (44.5, 132.2)
- added REF**: Breakaway_Tabs, kbd:Breakaway_Tabs, F.Cu at (134.5, 132.2)
- added REF**: Breakaway_Tabs, kbd:Breakaway_Tabs, F.Cu at (248.7, 132.2)
- added REF**: Breakaway_Tabs, kbd:Breakaway_Tabs, F.Cu at (403.4, 132.2)
- added REF**: Breakaway_Tabs, kbd:Breakaway_Tabs, F.Cu at (403.5, 35.1)
- added REF**: Breakaway_Tabs, kbd:Breakaway_Tabs, F.Cu at (199.3, 35.1)
- added REF**: Breakaway_Tabs, kbd:Breakaway_Tabs, F.Cu at (166.6, 35.1)
- added REF**: Breakaway_Tabs, kbd:Breakaway_Tabs, F.Cu at (44.6, 35.1)
- moved C12 9.40 mm to (165.9, 93.4)
- moved LED12 9.40 mm to (160.9, 93.5)
Routing:
- net Net-(LED11-Pad4): track 31.1 -> 42.1 mm, vias 2 -> 4
- net VCC: track 1071.9 -> 1080.7 mm
- net Net-(LED12-Pad4): track 36.4 -> 39.7 mm
- net col6_R: track 170.7 -> 172.1 mm
- net GND: track 980.7 -> 979.6 mm
- net Net-(LED77-Pad4): track 28.6 -> 29.3 mm
