File: bakekujira/bakekujira.kicad_pcb (KiCad board)
At the start: 2 copper layers, 405.8 x 120.8 mm, 372 parts, among them J1 MJ-4PP-9, J2 MJ-4PP-9, U1 Elite-C, U2 Elite-C

Commit message: renamed to bakekujira (may still change), added graphics, moved oled up to cover up elite-c
Parts:
- removed REF** (x8): Breakaway_Tabs, kbd:Breakaway_Tabs
- added G***: LOGO, bake-kujira:bake_kujira_flipped, F.Cu at (416.1, 108.0)
- added G***: LOGO, bake-kujira:bake_kujira, F.Cu at (31.4, 108.0)
- added REF1: Breakaway_Tabs, kbd:Breakaway_Tabs, F.Cu at (44.6, 35.1)
- added REF2: Breakaway_Tabs, kbd:Breakaway_Tabs, F.Cu at (166.6, 35.1)
- added REF3: Breakaway_Tabs, kbd:Breakaway_Tabs, F.Cu at (199.3, 35.1)
- added REF4: Breakaway_Tabs, kbd:Breakaway_Tabs, F.Cu at (403.5, 35.1)
- added REF5: Breakaway_Tabs, kbd:Breakaway_Tabs, F.Cu at (403.4, 132.2)
- added REF6: Breakaway_Tabs, kbd:Breakaway_Tabs, F.Cu at (248.7, 132.2)
- added REF7: Breakaway_Tabs, kbd:Breakaway_Tabs, F.Cu at (134.5, 132.2)
- added REF8: Breakaway_Tabs, kbd:Breakaway_Tabs, F.Cu at (44.5, 132.2)
- moved OL1 14.1 mm to (416.8, 75.8), turned to 0 degrees
- moved OL2 14.1 mm to (31.4, 75.8), turned to 0 degrees
- moved RSW1 7.56 mm to (416.8, 84.5)
- moved RSW2 7.56 mm to (31.4, 84.5), turned to 0 degrees
- turned C10 to 90 degrees
- turned C103 to 90 degrees
- turned C11 to 90 degrees
- turned C13 to 90 degrees
- turned C15 to 90 degrees
- turned C16 to 90 degrees
- turned C17 to 90 degrees
- turned C18 to 90 degrees
- turned C19 to 90 degrees
- turned C20 to 90 degrees
- turned C22 to 90 degrees
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Connections:
- C10 pad 1: VCC -> GND
- C10 pad 2: GND -> VCC
- C103 pad 1: GND -> VCC
- C103 pad 2: VCC -> GND
- C11 pad 1: VCC -> GND
- C11 pad 2: GND -> VCC
- C13 pad 1: VCC -> GND
- C13 pad 2: GND -> VCC
- C15 pad 1: VCC -> GND
- C15 pad 2: GND -> VCC
- C16 pad 1: VCC -> GND
- C16 pad 2: GND -> VCC
- C17 pad 1: VCC -> GND
- C17 pad 2: GND -> VCC
- C18 pad 1: VCC -> GND
- C18 pad 2: GND -> VCC
- C19 pad 1: VCC -> GND
- C19 pad 2: GND -> VCC
- C20 pad 1: VDD -> GNDA
- C20 pad 2: GNDA -> VDD
- C22 pad 1: VDD -> GNDA
- C22 pad 2: GNDA -> VDD
- C23 pad 1: VDD -> GNDA
- C23 pad 2: GNDA -> VDD
- C25 pad 1: VDD -> GNDA
- C25 pad 2: GNDA -> VDD
- C28 pad 1: VDD -> GNDA
- C28 pad 2: GNDA -> VDD
- C29 pad 1: VDD -> GNDA
- C29 pad 2: GNDA -> VDD
- C30 pad 1: VDD -> GNDA
- C30 pad 2: GNDA -> VDD
- C33 pad 1: GNDA -> VDD
- C33 pad 2: VDD -> GNDA
- C35 pad 1: GNDA -> VDD
- C35 pad 2: VDD -> GNDA
- C38 pad 1: GNDA -> VDD
- C38 pad 2: VDD -> GNDA
- C39 pad 1: GNDA -> VDD
- C39 pad 2: VDD -> GNDA
- C40 pad 1: GNDA -> VDD
- C40 pad 2: VDD -> GNDA
- C46 pad 1: GND -> VCC
- C46 pad 2: VCC -> GND
- C47 pad 1: GND -> VCC
- C47 pad 2: VCC -> GND
- C48 pad 1: GNDA -> VDD
- C48 pad 2: VDD -> GNDA
- C50 pad 1: GNDA -> VDD
- C50 pad 2: VDD -> GNDA
- C52 pad 1: GNDA -> VDD
- C52 pad 2: VDD -> GNDA
- C54 pad 1: GNDA -> VDD
- C54 pad 2: VDD -> GNDA
- C55 pad 1: GNDA -> VDD
- C55 pad 2: VDD -> GNDA
- C56 pad 1: GNDA -> VDD
- C56 pad 2: VDD -> GNDA
- C57 pad 1: GNDA -> VDD
- C57 pad 2: VDD -> GNDA
- C58 pad 1: GNDA -> VDD
- C58 pad 2: VDD -> GNDA
- C59 pad 1: GND -> VCC
- C59 pad 2: VCC -> GND
- C60 pad 1: GND -> VCC
- C60 pad 2: VCC -> GND
- C61 pad 1: GND -> VCC
- C61 pad 2: VCC -> GND
- C62 pad 1: GND -> VCC
- C62 pad 2: VCC -> GND
- C63 pad 1: GND -> VCC
- C63 pad 2: VCC -> GND
- C64 pad 1: GND -> VCC
- C64 pad 2: VCC -> GND
- C65 pad 1: GNDA -> VDD
- C65 pad 2: VDD -> GNDA
- C67 pad 1: GNDA -> VDD
- C67 pad 2: VDD -> GNDA
- C7 pad 1: VCC -> GND
- C7 pad 2: GND -> VCC
- C70 pad 1: GNDA -> VDD
- C70 pad 2: VDD -> GNDA
- C79 pad 1: GNDA -> VDD
- C79 pad 2: VDD -> GNDA
- C8 pad 1: VCC -> GND
- C8 pad 2: GND -> VCC
- C81 pad 1: GNDA -> VDD
- C81 pad 2: VDD -> GNDA
- C84 pad 1: GNDA -> VDD
- C84 pad 2: VDD -> GNDA
- C85 pad 1: GNDA -> VDD
- C85 pad 2: VDD -> GNDA
- C9 pad 1: VCC -> GND
- C9 pad 2: GND -> VCC
- C91 pad 1: GNDA -> VDD
- C91 pad 2: VDD -> GNDA
- C92 pad 1: GNDA -> VDD
- C92 pad 2: VDD -> GNDA
- C94 pad 1: GNDA -> VDD
- C94 pad 2: VDD -> GNDA
- C95 pad 1: GNDA -> VDD
- C95 pad 2: VDD -> GNDA
- C96 pad 1: GNDA -> VDD
- C96 pad 2: VDD -> GNDA
- C97 pad 1: GNDA -> VDD
- C97 pad 2: VDD -> GNDA
- C98 pad 1: GNDA -> VDD
- C98 pad 2: VDD -> GNDA
- C99 pad 1: GND -> VCC
- C99 pad 2: VCC -> GND
Routing:
- net SCL_L: track 44.6 -> 26.5 mm
- net SDA_L: track 44.7 -> 30.1 mm
- net VDD: track 1634.3 -> 1619.9 mm, vias 37 -> 38
- net GND: track 979.6 -> 969.0 mm, vias 7 -> 6
- net SCL_R: track 40.8 -> 31.4 mm, vias 0 -> 1
- net reset_R: track 40.9 -> 48.6 mm
- net reset_L: track 42.1 -> 46.6 mm
- net VCC: track 1080.7 -> 1076.3 mm, vias 29 -> 28
- net SDA_R: track 42.7 -> 39.1 mm, vias 0 -> 1
- net Net-(LED25-Pad4): track 42.1 -> 39.8 mm, vias 2 -> 4
- net col5_L: track 265.7 -> 264.2 mm
- net col6_R: track 172.1 -> 170.8 mm
- net col7_R: track 159.5 -> 158.8 mm
- net col4_R: track 250.8 -> 251.5 mm
- net col3_R: track 261.2 -> 261.9 mm
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Other:
- board text added: "Backside facing up"
- board text added: "bake kujira alfredy@gmail.com"
