File: bakekujira/bakekujira.kicad_pcb (KiCad board)
At the start: 2 copper layers, 405.8 x 120.8 mm, 374 parts, among them J1 MJ-4PP-9, J2 MJ-4PP-9, U1 Elite-C, U2 Elite-C

Commit message: switched over to protonc, rewired a bunch of shit, moved oled down to fit
Parts:
- removed G***: LOGO, bake-kujira:bake_kujira_flipped
- removed G***: LOGO, bake-kujira:bake_kujira
- removed REF1, REF2, REF3, REF4, REF5, REF6, REF7, REF8: Breakaway_Tabs, kbd:Breakaway_Tabs
- added R3: 4.7k, Resistor_SMD:R_0805_2012Metric_Pad1.20x1.40mm_HandSolder, B.Cu at (180.1, 50.4)
- added R4: 4.7k, Resistor_SMD:R_0805_2012Metric_Pad1.20x1.40mm_HandSolder, B.Cu at (189.2, 50.3)
- U1, U2: value Elite-C -> proton_c; footprint keebio:Elite-C -> proton_c:proton_c
- moved OL1 14.2 mm to (416.8, 90.0)
- moved OL2 14.2 mm to (31.4, 90.0)
- moved RSW1 11.5 mm to (416.8, 96.0)
- moved RSW2 11.5 mm to (31.4, 96.0)
- moved U2 1.44 mm to (31.4, 55.8), turned to 180 degrees
- moved U1 1.44 mm to (416.8, 55.8), turned to 180 degrees
Routing:
- net col2_R: track 256.8 -> 301.7 mm, vias 9 -> 6
- net col1_R: track 284.1 -> 312.4 mm, vias 10 -> 6
- net col3_R: track 261.9 -> 287.8 mm, vias 10 -> 8
- net col4_R: track 251.5 -> 269.0 mm, vias 10 -> 8
- net SCL_L: track 26.5 -> 42.9 mm
- net reset_R: track 48.6 -> 64.9 mm
- net Net-(LED80-Pad4): track 49.6 -> 35.4 mm, vias 2 -> 4
- net SDA_L: track 30.1 -> 44.2 mm
- net reset_L: track 46.6 -> 58.2 mm
- net col10_R: track 97.0 -> 87.1 mm, vias 5 -> 4
- net SCL_R: track 31.4 -> 40.5 mm, vias 1 -> 0
- net col9_R: track 110.6 -> 102.6 mm, vias 8 -> 7
- net VCC: track 1076.3 -> 1084.1 mm, vias 28 -> 29
- net row4_R: track 316.1 -> 308.8 mm, vias 2 -> 1
- net col5_L: track 264.2 -> 258.0 mm, vias 10 -> 9
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Other:
- outline, holes or cut-outs redrawn
- board text removed: "Backside facing up"

Commit message: cleanup, sanity checkin for missing breakaway tabs
Parts:
- added REF**: Breakaway_Tabs, kbd:Breakaway_Tabs, F.Cu at (403.5, 35.1)
- added REF**: Breakaway_Tabs, kbd:Breakaway_Tabs, F.Cu at (199.3, 35.1)
- added REF**: Breakaway_Tabs, kbd:Breakaway_Tabs, F.Cu at (166.6, 35.1)
- added REF1: Breakaway_Tabs, kbd:Breakaway_Tabs, F.Cu at (44.6, 35.1)
Other:
- rule pad_to_mask_clearance: 0 -> 0.2
- board text added: "bake kujira v1.0 papadakko alfredy@gmail.com"
- board text removed: "bake kujira alfredy@gmail.com"
